Commit message: tuned up and working a lot better

File: rotors_description/urdf/component_snippets.xacro (robot description, xacro)
@@ -230,45 +230,4 @@
         <imuSubTopic>${imu_sub_topic}</imuSubTopic>
         <motorSpeedCommandPubTopic>gazebo/command/motor_speed</motorSpeedCommandPubTopic>
-      </plugin>
-    </gazebo>
-  </xacro:macro>
-  <!-- Macro to add an IMU. -->
-  <xacro:macro name="imu_plugin_macro"
-    params="namespace imu_suffix parent_link imu_topic
-      mass_imu_sensor gyroscope_noise_density gyroscopoe_random_walk
-      gyroscope_bias_correlation_time gyroscope_turn_on_bias_sigma
-      accelerometer_noise_density accelerometer_random_walk
-      accelerometer_bias_correlation_time accelerometer_turn_on_bias_sigma
-      *inertia *origin">
-    <!-- IMU link -->
-    <link name="${namespace}/imu${imu_suffix}_link">
-      <inertial>
-        <xacro:insert_block name="inertia" />
-        <mass value="${mass_imu_sensor}" />  <!-- [kg] -->
-        <origin xyz="0 0 0" rpy="0 0 0" />
-      </inertial>
-    </link>
-    <!-- IMU joint -->
-    <joint name="${namespace}/imu${imu_suffix}_joint" type="revolute">
-      <xacro:insert_block name="origin" />
-      <parent link="${parent_link}" />
-      <child link="${namespace}/imu${imu_suffix}_link" />
-      <limit upper="0" lower="0" effort="0" velocity="0" />
-    </joint>
-    <gazebo>
-      <plugin filename="librotors_gazebo_imu_plugin.so" name="rotors_gazebo_imu${imu_suffix}_plugin">
-      <!-- A good description of the IMU parameters can be found in the kalibr documentation:
-           https://github.com/ethz-asl/kalibr/wiki/IMU-Noise-Model-and-Intrinsics -->
-        <robotNamespace>${namespace}</robotNamespace> <!-- (string, required): ros namespace in which the messages are published -->
-        <linkName>${namespace}/imu${imu_suffix}_link</linkName> <!-- (string, required): name of the body which holds the IMU sensor -->
-        <imuTopic>${imu_topic}</imuTopic> <!-- (string): name of the sensor output topic and prefix of service names (defaults to imu) -->
-        <gyroscopeNoiseDensity>${gyroscope_noise_density}</gyroscopeNoiseDensity> <!-- Gyroscope noise density (two-sided spectrum) [rad/s/sqrt(Hz)] -->
-        <gyroscopeRandomWalk>${gyroscopoe_random_walk}</gyroscopeRandomWalk> <!-- Gyroscope bias random walk [rad/s/s/sqrt(Hz)] -->
-        <gyroscopeBiasCorrelationTime>${gyroscope_bias_correlation_time}</gyroscopeBiasCorrelationTime> <!-- Gyroscope bias correlation time constant [s] -->
-        <gyroscopeTurnOnBiasSigma>${gyroscope_turn_on_bias_sigma}</gyroscopeTurnOnBiasSigma> <!-- Gyroscope turn on bias standard deviation [rad/s] -->
-        <accelerometerNoiseDensity>${accelerometer_noise_density}</accelerometerNoiseDensity> <!-- Accelerometer noise density (two-sided spectrum) [m/s^2/sqrt(Hz)] -->
-        <accelerometerRandomWalk>${accelerometer_random_walk}</accelerometerRandomWalk> <!-- Accelerometer bias random walk. [m/s^2/s/sqrt(Hz)] -->
-        <accelerometerBiasCorrelationTime>${accelerometer_bias_correlation_time}</accelerometerBiasCorrelationTime> <!-- Accelerometer bias correlation time constant [s] -->
-        <accelerometerTurnOnBiasSigma>${accelerometer_turn_on_bias_sigma}</accelerometerTurnOnBiasSigma> <!-- Accelerometer turn on bias standard deviation [m/s^2] -->
       </plugin>
     </gazebo>
@@ -605,23 +564,3 @@
     </xacro:odometry_plugin_macro>
   </xacro:macro>
-  <xacro:macro name="default_imu" params="namespace parent_link">
-    <!-- ADIS16448 IMU. -->
-    <xacro:imu_plugin_macro
-      namespace="${namespace}"
-      imu_suffix=""
-      parent_link="${parent_link}"
-      imu_topic="imu"
-      mass_imu_sensor="0.015"
-      gyroscope_noise_density="0.0003394"
-      gyroscopoe_random_walk="0.000038785"
-      gyroscope_bias_correlation_time="1000.0"
-      gyroscope_turn_on_bias_sigma="0.0087"
-      accelerometer_noise_density="0.004"
-      accelerometer_random_walk="0.006"
-      accelerometer_bias_correlation_time="300.0"
-      accelerometer_turn_on_bias_sigma="0.1960">
-      <inertia ixx="0.00001" ixy="0.0" ixz="0.0" iyy="0.00001" iyz="0.0" izz="0.00001" />
-      <origin xyz="0 0 0" rpy="0 0 0" />
-    </xacro:imu_plugin_macro>
-  </xacro:macro>
 </robot>

File: rotors_description/urdf/shredder_base.xacro (robot description, xacro)
@@ -17,11 +17,31 @@
 -->
 <robot name="shredder" xmlns:xacro="http://ros.org/wiki/xacro">
+  <!-- Plugin Macro Locations -->
   <xacro:include filename="$(find rotors_description)/urdf/component_snippets.xacro" />
-  <!-- Instantiate shredder "mechanics" -->
-  <xacro:include filename="$(find rotors_description)/urdf/shredder.xacro" />
+  <!-- Instantiate shredder mechanics -->
+  <xacro:include filename="$(find rotors_description)/urdf/shredder_mechanics.xacro" />
   <!-- Instantiate a controller. -->
   <xacro:controller_plugin_macro namespace="${namespace}" imu_sub_topic="imu" />
-  <!-- Mount an ADIS16448 IMU. -->
-  <xacro:default_imu namespace="${namespace}" parent_link="${namespace}/base_link" />
+  <!-- Mount an IMU. -->
+  <xacro:include filename="$(find rotors_gazebo_plugins)/xacro/imu.xacro"/>
+  <xacro:IMU_ADIS16448
+    namespace="${namespace}"
+    parent_link="${namespace}/base_link"
+    imu_topic="imu"/>
+  <!-- Mount an Altimeter -->
+  <xacro:include filename="$(find rotors_gazebo_plugins)/xacro/altimeter.xacro"/>
+  <xacro:Sonar_MB1030
+    namespace="${namespace}"
+    parent_link="${namespace}/base_link"
+    altimeter_topic="altimeter"/>
+  <!-- Publish Global State and Mocap for Relative Nav -->
+  <xacro:include filename="$(find rotors_gazebo_plugins)/xacro/global_state_plugin.xacro"/>
+  <xacro:global_state_publisher
+    namespace="${namespace}"
+    parent_link="${namespace}/base_link"
+    mocap_topic="mocap"
+    global_state_topic="global_state"
+    global_state_suffix=""/>
+  <!-- Enable Ground Truth -->
   <xacro:if value="$(arg enable_ground_truth)">
     <xacro:ground_truth_imu_and_odometry namespace="${namespace}" parent_link="${namespace}/base_link" />
