Commit message: various fixes

File: rotor_gazebo/urdf/shredder_base.xacro (robot description, xacro)
@@ -28,12 +28,4 @@
     <xacro:ground_truth namespace="${namespace}" parent_link="${namespace}/base_link" />
   </xacro:if>
-  <!-- Publish Global State and Mocap for Relative Nav -->
-  <xacro:include filename="$(find rotor_gazebo_plugins)/xacro/global_state_plugin.xacro"/>
-  <xacro:global_state_publisher
-    namespace=""
-    parent_link="${namespace}/base_link"
-    mocap_topic="mocap"
-    global_state_topic="global_state"
-    global_state_suffix=""/>
   <!-- Mount an IMU. -->
   <xacro:include filename="$(find rotor_gazebo_plugins)/xacro/imu.xacro"/>
@@ -58,5 +50,5 @@
     namespace=""
     parent_link="${namespace}/base_link"
-    visualize="false"/>
+    visualize="true"/>
   <!-- Instantiate a logger - haven't yet tried this, but left functionality just in case -->
   <xacro:if value="$(arg enable_logging)">

File: rotor_gazebo/urdf/shredder_mechanics.xacro (robot description, xacro)
@@ -20,5 +20,5 @@
   <!-- Properties -->
   <xacro:property name="namespace" value="$(arg mav_name)" />
-  <xacro:property name="rotor_velocity_slowdown_sim" value="50" />
+  <xacro:property name="rotor_velocity_slowdown_sim" value="10" />
   <xacro:property name="use_mesh_file" value="true" />
   <xacro:property name="mesh_file" value="package://rotor_gazebo/meshes/firefly.dae" />

File: rotor_gazebo_plugins/xacro/laser_scanner.xacro (robot description, xacro)
@@ -19,5 +19,5 @@
       max_angle="pi/2"
       update_rate="40">
-      <origin xyz="0 0 0" rpy="0 0 0" />
+      <origin xyz="0.09525 0 -0.0127" rpy="0 0 0" />
     </xacro:laser_scanner>
   </xacro:macro>

File: rotor_gazebo_plugins/xacro/rgbd.xacro (robot description, xacro)
@@ -19,5 +19,5 @@
       depth_camera_info_topic="/camera/depth/camera_info"
       pointcloud_topic="/camera/pointcloud">
-      <origin xyz="0 0 0" rpy="0 0 0" />
+      <origin xyz="0.127 0 -0.0889" rpy="0 0 0" /> <!-- for shredder -->
     </xacro:depth_camera>
   </xacro:macro>
@@ -39,5 +39,5 @@
     <link name="${namespace}/camera_link">
       <collision>
-        <origin xyz="0 0 0" rpy="0 0 0" />
+        <xacro:insert_block name="origin" />
         <geometry>
           <cylinder length="0.01" radius="0.007" />
