Commit message: laser, rgbd, imu and altimiter

File: rotor_gazebo/urdf/component_snippets.xacro (robot description, xacro)
@@ -233,57 +233,4 @@
     </gazebo>
   </xacro:macro>
-<!-- Macro to add a generic odometry sensor. -->
-  <xacro:macro name="odometry_plugin_macro"
-    params="
-      namespace odometry_sensor_suffix parent_link pose_topic pose_with_covariance_topic
-      position_topic transform_topic odometry_topic parent_frame_id
-      mass_odometry_sensor measurement_divisor measurement_delay unknown_delay
-      noise_normal_position noise_normal_quaternion noise_normal_linear_velocity
-      noise_normal_angular_velocity noise_uniform_position
-      noise_uniform_quaternion noise_uniform_linear_velocity
-      noise_uniform_angular_velocity enable_odometry_map odometry_map
-      image_scale *inertia *origin">
-    <!-- odometry link -->
-    <link name="${namespace}/odometry_sensor${odometry_sensor_suffix}_link">
-      <inertial>
-        <xacro:insert_block name="inertia" />
-        <mass value="${mass_odometry_sensor}" />  <!-- [kg] -->
-      </inertial>
-    </link>
-    <!-- odometry joint -->
-    <joint name="${namespace}/odometry_sensor${odometry_sensor_suffix}_joint" type="revolute">
-      <parent link="${parent_link}" />
-      <xacro:insert_block name="origin" />
-      <child link="${namespace}/odometry_sensor${odometry_sensor_suffix}_link" />
-      <limit upper="0" lower="0" effort="0" velocity="0" />
-    </joint>
-    <gazebo>
-      <plugin filename="librotor_gazebo_odometry_plugin.so" name="odometry_sensor${odometry_sensor_suffix}">
-        <linkName>${namespace}/odometry_sensor${odometry_sensor_suffix}_link</linkName>
-        <robotNamespace>${namespace}</robotNamespace>
-        <poseTopic>${pose_topic}</poseTopic>
-        <poseWithCovarianceTopic>${pose_with_covariance_topic}</poseWithCovarianceTopic>
-        <positionTopic>${position_topic}</positionTopic>
-        <transformTopic>${transform_topic}</transformTopic>
-        <odometryTopic>${odometry_topic}</odometryTopic>
-        <parentFrameId>${parent_frame_id}</parentFrameId> <!-- Use the scoped link name here. e.g. Model::link. -->
-        <measurementDivisor>${measurement_divisor}</measurementDivisor> <!-- only every (seq % measurementDivisor) == 0 measurement is published [int] -->
-        <measurementDelay>${measurement_delay}</measurementDelay> <!-- time that measurement gets held back before it's published in [simulation cycles (int)] -->
-        <unknownDelay>${unknown_delay}</unknownDelay> <!-- additional delay, that just gets added to the timestamp [s] -->
-        <noiseNormalPosition>${noise_normal_position}</noiseNormalPosition> <!-- standard deviation of additive white gaussian noise [m] -->
-        <noiseNormalQuaternion>${noise_normal_quaternion}</noiseNormalQuaternion> <!-- standard deviation white gaussian noise [rad]: q_m = q*quaternionFromSmallAngleApproximation(noiseNormalQ) -->
-        <noiseNormalLinearVelocity>${noise_normal_linear_velocity}</noiseNormalLinearVelocity> <!-- standard deviation of additive white gaussian noise [m/s] -->
-        <noiseNormalAngularVelocity>${noise_normal_angular_velocity}</noiseNormalAngularVelocity> <!-- standard deviation of additive white gaussian noise [rad/s] -->
-        <noiseUniformPosition>${noise_uniform_position}</noiseUniformPosition> <!-- symmetric bounds of uniform noise [m] -->
-        <noiseUniformQuaternion>${noise_uniform_quaternion}</noiseUniformQuaternion> <!-- symmetric bounds of uniform noise [rad], computation see above -->
-        <noiseUniformLinearVelocity>${noise_uniform_linear_velocity}</noiseUniformLinearVelocity> <!-- symmetric bounds of uniform noise [m/s] -->
-        <noiseUniformAngularVelocity>${noise_uniform_angular_velocity}</noiseUniformAngularVelocity> <!-- symmetric bounds of uniform noise [rad/s] -->
-        <xacro:if value="${enable_odometry_map}">
-          <covarianceImage>package://rotor_gazebo/resource/${odometry_map}</covarianceImage> <!-- a bitmap image describing where the sensor works (white), and where not (black) -->
-          <covarianceImageScale>${image_scale}</covarianceImageScale> <!-- the scale of the image in the gazebo world, if set to 1.0, 1 pixel in the image corresponds to 1 meter in the world -->
-        </xacro:if>
-      </plugin>
-    </gazebo>
-  </xacro:macro>
   <!-- Macro to add the wind plugin. -->
   <xacro:macro name="wind_plugin_macro"
@@ -464,36 +411,4 @@
       </xacro:vi_sensor_depth_macro>
     </xacro:if>
-    <!-- Groundtruth -->
-    <xacro:if value="${enable_ground_truth}">
-      <!-- Odometry Sensor -->
-      <xacro:odometry_plugin_macro
-        namespace="${namespace}/ground_truth"
-        odometry_sensor_suffix=""
-        parent_link="${namespace}/vi_sensor_link"
-        pose_topic="pose"
-        pose_with_covariance_topic="pose_with_covariance"
-        position_topic="position"
-        transform_topic="transform"
-        odometry_topic="odometry"
-        parent_frame_id="world"
-        mass_odometry_sensor="0.00001"
-        measurement_divisor="1"
-        measurement_delay="0"
-        unknown_delay="0.0"
-        noise_normal_position="0 0 0"
-        noise_normal_quaternion="0 0 0"
-        noise_normal_linear_velocity="0 0 0"
-        noise_normal_angular_velocity="0 0 0"
-        noise_uniform_position="0 0 0"
-        noise_uniform_quaternion="0 0 0"
-        noise_uniform_linear_velocity="0 0 0"
-        noise_uniform_angular_velocity="0 0 0"
-        enable_odometry_map="false"
-        odometry_map=""
-        image_scale="">
-        <inertia ixx="0.00001" ixy="0.0" ixz="0.0" iyy="0.00001" iyz="0.0" izz="0.00001" /> <!-- [kg m^2] [kg m^2] [kg m^2] [kg m^2] [kg m^2] [kg m^2] -->
-        <origin xyz="0.0 0.0 0.0" rpy="0.0 0.0 0.0" />
-      </xacro:odometry_plugin_macro>
-    </xacro:if>
     <!-- ADIS16448 IMU. -->
     <xacro:imu_plugin_macro
@@ -515,52 +430,3 @@
     </xacro:imu_plugin_macro>
   </xacro:macro>
-  <xacro:macro name="ground_truth_imu_and_odometry" params="namespace parent_link">
-    <!-- Mount an IMU providing ground truth. -->
-    <xacro:imu_plugin_macro
-      namespace="${namespace}"
-      imu_suffix="gt"
-      parent_link="${parent_link}"
-      imu_topic="ground_truth/imu"
-      mass_imu_sensor="0.00001"
-      gyroscope_noise_density="0.0"
-      gyroscopoe_random_walk="0.0"
-      gyroscope_bias_correlation_time="1000.0"
-      gyroscope_turn_on_bias_sigma="0.0"
-      accelerometer_noise_density="0.0"
-      accelerometer_random_walk="0.0"
-      accelerometer_bias_correlation_time="300.0"
-      accelerometer_turn_on_bias_sigma="0.0">
-      <inertia ixx="0.00001" ixy="0.0" ixz="0.0" iyy="0.00001" iyz="0.0" izz="0.00001" />
-      <origin xyz="0 0 0" rpy="0 0 0" />
-    </xacro:imu_plugin_macro>
-    <!-- Mount a generic odometry sensor providing ground truth. -->
-    <xacro:odometry_plugin_macro
-      namespace="${namespace}/ground_truth"
-      odometry_sensor_suffix="gt"
-      parent_link="${parent_link}"
-      pose_topic="pose"
-      pose_with_covariance_topic="pose_with_covariance"
-      position_topic="position"
-      transform_topic="transform"
-      odometry_topic="odometry"
-      parent_frame_id="world"
-      mass_odometry_sensor="0.00001"
-      measurement_divisor="1"
-      measurement_delay="0"
-      unknown_delay="0.0"
-      noise_normal_position="0 0 0"
-      noise_normal_quaternion="0 0 0"
-      noise_normal_linear_velocity="0 0 0"
-      noise_normal_angular_velocity="0 0 0"
-      noise_uniform_position="0 0 0"
-      noise_uniform_quaternion="0 0 0"
-      noise_uniform_linear_velocity="0 0 0"
-      noise_uniform_angular_velocity="0 0 0"
-      enable_odometry_map="false"
-      odometry_map=""
-      image_scale="">
-      <inertia ixx="0.00001" ixy="0.0" ixz="0.0" iyy="0.00001" iyz="0.0" izz="0.00001" /> <!-- [kg m^2] [kg m^2] [kg m^2] [kg m^2] [kg m^2] [kg m^2] -->
-      <origin xyz="0.0 0.0 0.0" rpy="0.0 0.0 0.0" />
-    </xacro:odometry_plugin_macro>
-  </xacro:macro>
 </robot>

File: rotor_gazebo/urdf/shredder_base.xacro (robot description, xacro)
@@ -45,35 +45,18 @@
   <!-- Enable Ground Truth -->
   <xacro:if value="$(arg enable_ground_truth)">
-    <xacro:ground_truth_imu_and_odometry namespace="${namespace}" parent_link="${namespace}/base_link" />
+    <xacro:include filename="$(find rotor_gazebo_plugins)/xacro/odometry_sensor.xacro"/>
+    <xacro:ground_truth namespace="${namespace}" parent_link="${namespace}/base_link" />
   </xacro:if>
-  <!-- Mount a generic odometry sensor without odometry map - used by attitude_controller -->
-  <xacro:odometry_plugin_macro
-    namespace="${namespace}/odometry_sensor1"
-    odometry_sensor_suffix="1"
+  <!-- Mount an RGBD Camera -->
+  <xacro:include filename="$(find rotor_gazebo_plugins)/xacro/rgbd.xacro"/>
+  <xacro:xtion
+    namespace="${namespace}"
+    parent_link="${namespace}/base_link"/>
+  <!-- Laser Scanner -->
+  <xacro:include filename="$(find rotor_gazebo_plugins)/xacro/laser_scanner.xacro"/>
+  <xacro:hokuyo_UTM-30LX
+    namespace="${namespace}"
     parent_link="${namespace}/base_link"
-    pose_topic="pose"
-    pose_with_covariance_topic="pose_with_covariance"
-    position_topic="position"
-    transform_topic="transform"
-    odometry_topic="odometry"
-    parent_frame_id="world"
-    mass_odometry_sensor="0.00001"
-    measurement_divisor="1"
-    measurement_delay="0"
-    unknown_delay="0.0"
-    noise_normal_position="0 0 0"
-    noise_normal_quaternion="0 0 0"
-    noise_normal_linear_velocity="0 0 0"
-    noise_normal_angular_velocity="0 0 0"
-    noise_uniform_position="0 0 0"
-    noise_uniform_quaternion="0 0 0"
-    noise_uniform_linear_velocity="0 0 0"
-    noise_uniform_angular_velocity="0 0 0"
-    enable_odometry_map="false"
-    odometry_map=""
-    image_scale="">
-    <inertia ixx="0.00001" ixy="0.0" ixz="0.0" iyy="0.00001" iyz="0.0" izz="0.00001" />
-    <origin xyz="0.0 0.0 0.0" rpy="0.0 0.0 0.0" />
-  </xacro:odometry_plugin_macro>
+    visualize="true"/>
   <xacro:if value="$(arg enable_logging)">
     <!-- Instantiate a logger -->

Commit message: cleaned up code

File: rotor_gazebo/urdf/component_snippets.xacro (robot description, xacro)
@@ -18,17 +18,4 @@
 <robot xmlns:xacro="http://ros.org/wiki/xacro">
   <xacro:property name="pi" value="3.14159265359" />
-  <!-- Macro to add logging to a bag file. -->
-  <xacro:macro name="bag_plugin_macro"
-    params="namespace bag_file rotor_velocity_slowdown_sim">
-    <gazebo>
-      <plugin filename="librotor_gazebo_bag_plugin.so" name="rosbag">
-        <robotNamespace>${namespace}</robotNamespace>
-        <bagFileName>${bag_file}</bagFileName>
-        <linkName>${namespace}/base_link</linkName>
-        <frameId>${namespace}/base_link</frameId>
-        <rotorVelocitySlowdownSim>${rotor_velocity_slowdown_sim}</rotorVelocitySlowdownSim>
-      </plugin>
-    </gazebo>
-  </xacro:macro>
   <!-- Macro to add a camera. -->
   <xacro:macro name="camera_macro"
@@ -221,16 +208,16 @@
   </xacro:macro>
   <!-- Macro to add the controller interface. -->
-  <xacro:macro name="controller_plugin_macro" params="namespace imu_sub_topic">
-    <gazebo>
-      <plugin name="controller_interface" filename="librotor_gazebo_controller_interface.so">
-        <robotNamespace>${namespace}</robotNamespace>
-        <commandAttitudeThrustSubTopic>command/attitude</commandAttitudeThrustSubTopic>
-        <commandRateThrustSubTopic>command/rate</commandRateThrustSubTopic>
-        <commandMotorSpeedSubTopic>command/motor_speed</commandMotorSpeedSubTopic>
-        <imuSubTopic>${imu_sub_topic}</imuSubTopic>
-        <motorSpeedCommandPubTopic>gazebo/command/motor_speed</motorSpeedCommandPubTopic>
-      </plugin>
-    </gazebo>
-  </xacro:macro>
+  <!-- <xacro:macro name="controller_plugin_macro" params="namespace imu_sub_topic"> -->
+    <!-- <gazebo> -->
+      <!-- <plugin name="controller_interface" filename="librotor_gazebo_controller_interface.so"> -->
+        <!-- <robotNamespace>${namespace}</robotNamespace> -->
+        <!-- <commandAttitudeThrustSubTopic>command/attitude</commandAttitudeThrustSubTopic> -->
+        <!-- <commandRateThrustSubTopic>command/rate</commandRateThrustSubTopic> -->
+        <!-- <commandMotorSpeedSubTopic>command/motor_speed</commandMotorSpeedSubTopic> -->
+        <!-- <imuSubTopic>${imu_sub_topic}</imuSubTopic> -->
+        <!-- <motorSpeedCommandPubTopic>gazebo/command/motor_speed</motorSpeedCommandPubTopic> -->
+      <!-- </plugin> -->
+    <!-- </gazebo> -->
+  <!-- </xacro:macro> -->
   <!-- Macro to add the wind plugin. -->
   <xacro:macro name="wind_plugin_macro"

File: rotor_gazebo/urdf/shredder/shredder_base.xacro (robot description, xacro)
@@ -17,9 +17,8 @@
 -->
 <robot name="shredder" xmlns:xacro="http://ros.org/wiki/xacro">
-  <!-- Plugin Macro Locations -->
-  <xacro:include filename="$(find rotor_gazebo)/urdf/component_snippets.xacro" />
   <!-- Instantiate shredder mechanics -->
-  <xacro:include filename="$(find rotor_gazebo)/urdf/shredder_mechanics.xacro" />
+  <xacro:include filename="$(find rotor_gazebo)/urdf/shredder/shredder_mechanics.xacro" />
   <!-- Instantiate a controller for the motors. -->
+  <xacro:include filename="$(find rotor_gazebo_plugins)/xacro/controller_interface.xacro"/>
   <xacro:controller_plugin_macro namespace="${namespace}" imu_sub_topic="imu" />
   <!-- Enable Ground Truth - Used by attitude_controller -->
@@ -57,10 +56,3 @@
     parent_link="${namespace}/base_link"
     visualize="false"/>
-  <!-- Instantiate a logger - haven't yet tried this, but left functionality just in case -->
-  <xacro:if value="$(arg enable_logging)">
-    <xacro:bag_plugin_macro
-      namespace=""
-      bag_file="$(arg log_file)"
-      rotor_velocity_slowdown_sim="${rotor_velocity_slowdown_sim}" />
-  </xacro:if>
 </robot>
