Commit message: cleaned up a lot in the multirotor files

File: rotor_gazebo/urdf/hummingbird/hummingbird_base.xacro (robot description, xacro)
@@ -1,36 +1,158 @@
 <?xml version="1.0"?>
 <!--
-  Copyright 2015 Fadri Furrer, ASL, ETH Zurich, Switzerland
-  Copyright 2015 Michael Burri, ASL, ETH Zurich, Switzerland
-  Copyright 2015 Mina Kamel, ASL, ETH Zurich, Switzerland
-  Copyright 2015 Janosch Nikolic, ASL, ETH Zurich, Switzerland
-  Copyright 2015 Markus Achtelik, ASL, ETH Zurich, Switzerland
-  Licensed under the Apache License, Version 2.0 (the "License");
-  you may not use this file except in compliance with the License.
-  You may obtain a copy of the License at
-  http://www.apache.org/licenses/LICENSE-2.0
-  Unless required by applicable law or agreed to in writing, software
-  distributed under the License is distributed on an "AS IS" BASIS,
-  WITHOUT WARRANTIES OR CONDITIONS OF ANY KIND, either express or implied.
-  See the License for the specific language governing permissions and
-  limitations under the License.
+Gazebo Hummingbird Definition File
+Author: James Jackson
 -->
 <robot name="hummingbird" xmlns:xacro="http://ros.org/wiki/xacro">
-  <xacro:include filename="$(find rotor_gazebo)/urdf/component_snippets.xacro" />
-  <!-- Instantiate hummingbird "mechanics" -->
-  <xacro:include filename="$(find rotor_gazebo)/urdf/hummingbird/hummingbird_mechanics.xacro" />
-  <!-- Instantiate a controller. -->
-  <xacro:controller_plugin_macro namespace="${namespace}" imu_sub_topic="imu" />
+  <!-- Properties -->
+  <xacro:property name="namespace" value="$(arg mav_name)" />
+  <xacro:property name="rotor_velocity_slowdown_sim" value="10" />
+  <xacro:property name="use_mesh_file" value="true" />
+  <xacro:property name="mesh_file" value="package://rotor_gazebo/meshes/hummingbird.dae" />
+  <xacro:property name="mass" value="0.5755" /> <!-- [kg] -->
+  <xacro:property name="body_width" value="0.1" /> <!-- [m] -->
+  <xacro:property name="body_height" value="0.12" /> <!-- [m] -->
+  <xacro:property name="mass_rotor" value="0.009" /> <!-- [kg] -->
+  <xacro:property name="arm_length" value="0.17" /> <!-- [m] -->
+  <xacro:property name="rotor_offset_top" value="0.01" /> <!-- [m] -->
+  <xacro:property name="radius_rotor" value="0.1" /> <!-- [m] -->
+  <xacro:property name="motor_constant" value="8.54858e-06" /> <!-- [kg m/s^2] -->
+  <xacro:property name="moment_constant" value="0.016" /> <!-- [m] -->
+  <xacro:property name="time_constant_up" value="0.0025" /> <!-- [s] -->
+  <xacro:property name="time_constant_down" value="0.0025" /> <!-- [s] -->
+  <xacro:property name="max_rot_velocity" value="838" /> <!-- [rad/s] -->
+  <xacro:property name="rotor_drag_coefficient" value="8.06428e-05" />
+  <xacro:property name="rolling_moment_coefficient" value="0.000001" />
+  <xacro:property name="body_inertia">
+    <inertia ixx="0.007" ixy="0.0" ixz="0.0" iyy="0.007" iyz="0.0" izz="0.012" />
+  </xacro:property>
+  <xacro:property name="rotor_inertia">
+    <xacro:box_inertia x="${radius_rotor}" y="0.015" z="0.003" mass="${mass_rotor*rotor_velocity_slowdown_sim}" />
+  </xacro:property>
+  <!-- *********************** GAZEBO ROBOT DEFINITION ******************* -->
+  <link name="${namespace}/base_link">
+    <inertial>
+      <mass value="${mass}" />  <!-- [kg] -->
+      <origin xyz="0 0 0" />
+      <xacro:insert_block name="body_inertia" />
+    </inertial>
+    <visual>
+      <origin xyz="0 0 0" rpy="0 0 .785" />
+      <geometry>
+        <xacro:if value="${use_mesh_file}">
+          <mesh filename="${mesh_file}" scale="1 1 1" />
+        </xacro:if>
+        <xacro:unless value="${use_mesh_file}">
+          <box size="${body_width} ${body_width} ${body_height}"/>
+        </xacro:unless>
+      </geometry>
+    </visual>
+    <collision>
+      <origin xyz="0 0 0" rpy="0 0 0" />
+      <geometry>
+        <box size="${body_width} ${body_width} ${body_height}" />
+      </geometry>
+    </collision>
+  </link>
+  <!-- ************************* ROTOR DYNAMICS ********************** -->
+  <gazebo>
+    <plugin filename="librotor_gazebo_multirotor_base_plugin.so" name="multirotor_base_plugin">
+      <robotNamespace>${namespace}</robotNamespace>
+      <linkName>${namespace}/base_link</linkName>
+      <rotorVelocitySlowdownSim>${rotor_velocity_slowdown_sim}</rotorVelocitySlowdownSim>
+    </plugin>
+  </gazebo>
+  <!-- **************** ROTORS ***************** -->
+  <xacro:include filename="$(find rotor_gazebo_plugins)/xacro/rotor.xacro"/>
+  <xacro:vertical_rotor
+    robot_namespace="${namespace}"
+    suffix="front_right"
+    direction="cw"
+    motor_constant="${motor_constant}"
+    moment_constant="${moment_constant}"
+    parent="${namespace}/base_link"
+    mass_rotor="${mass_rotor}"
+    radius_rotor="${radius_rotor}"
+    time_constant_up="${time_constant_up}"
+    time_constant_down="${time_constant_down}"
+    max_rot_velocity="${max_rot_velocity}"
+    motor_number="0"
+    rotor_drag_coefficient="${rotor_drag_coefficient}"
+    rolling_moment_coefficient="${rolling_moment_coefficient}"
+    color="Red"
+    use_own_mesh="false"
+    mesh="">
+    <origin xyz="${.707*arm_length} -${.707*arm_length} ${rotor_offset_top}" rpy="0 0 0" />
+    <xacro:insert_block name="rotor_inertia" />
+  </xacro:vertical_rotor>
+  <xacro:vertical_rotor
+    robot_namespace="${namespace}"
+    suffix="front_left"
+    direction="ccw"
+    motor_constant="${motor_constant}"
+    moment_constant="${moment_constant}"
+    parent="${namespace}/base_link"
+    mass_rotor="${mass_rotor}"
+    radius_rotor="${radius_rotor}"
+    time_constant_up="${time_constant_up}"
+    time_constant_down="${time_constant_down}"
+    max_rot_velocity="${max_rot_velocity}"
+    motor_number="1"
+    rotor_drag_coefficient="${rotor_drag_coefficient}"
+    rolling_moment_coefficient="${rolling_moment_coefficient}"
+    color="Red"
+    use_own_mesh="false"
+    mesh="">
+    <origin xyz="${.707*arm_length} ${.707*arm_length} ${rotor_offset_top}" rpy="0 0 0" />
+    <xacro:insert_block name="rotor_inertia" />
+  </xacro:vertical_rotor>
+  <xacro:vertical_rotor
+    robot_namespace="${namespace}"
+    suffix="back_left"
+    direction="cw"
+    motor_constant="${motor_constant}"
+    moment_constant="${moment_constant}"
+    parent="${namespace}/base_link"
+    mass_rotor="${mass_rotor}"
+    radius_rotor="${radius_rotor}"
+    time_constant_up="${time_constant_up}"
+    time_constant_down="${time_constant_down}"
+    max_rot_velocity="${max_rot_velocity}"
+    motor_number="2"
+    rotor_drag_coefficient="${rotor_drag_coefficient}"
+    rolling_moment_coefficient="${rolling_moment_coefficient}"
+    color="Black"
+    use_own_mesh="false"
+    mesh="">
+    <origin xyz="-${.707*arm_length} ${.707*arm_length} ${rotor_offset_top}" rpy="0 0 0" />
+    <xacro:insert_block name="rotor_inertia" />
+  </xacro:vertical_rotor>
+  <xacro:vertical_rotor
+    robot_namespace="${namespace}"
+    suffix="back_right"
+    direction="ccw"
+    motor_constant="${motor_constant}"
+    moment_constant="${moment_constant}"
+    parent="${namespace}/base_link"
+    mass_rotor="${mass_rotor}"
+    radius_rotor="${radius_rotor}"
+    time_constant_up="${time_constant_up}"
+    time_constant_down="${time_constant_down}"
+    max_rot_velocity="${max_rot_velocity}"
+    motor_number="3"
+    rotor_drag_coefficient="${rotor_drag_coefficient}"
+    rolling_moment_coefficient="${rolling_moment_coefficient}"
+    color="Black"
+    use_own_mesh="false"
+    mesh="">
+    <origin xyz="-${.707*arm_length} -${.707*arm_length} ${rotor_offset_top}" rpy="0 0 0" />
+    <xacro:insert_block name="rotor_inertia" />
+  </xacro:vertical_rotor>
+  <!-- ***************** SENSORS ******************* -->
   <!-- Mount an ADIS16448 IMU. -->
+  <xacro:include filename="$(find rotor_gazebo_plugins)/xacro/imu.xacro"/>
   <xacro:default_imu namespace="${namespace}" parent_link="${namespace}/base_link" />
-  <!-- Enable Ground Truth - Used by attitude_controller -->
+  <!-- Enable Ground Truth -->
   <xacro:include filename="$(find rotor_gazebo_plugins)/xacro/odometry_sensor.xacro"/>
   <xacro:ground_truth namespace="${namespace}" parent_link="${namespace}/base_link" />
-  <xacro:if value="$(arg enable_logging)">
-    <!-- Instantiate a logger -->
-    <xacro:bag_plugin_macro
-      namespace="${namespace}"
-      bag_file="$(arg log_file)"
-      rotor_velocity_slowdown_sim="${rotor_velocity_slowdown_sim}" />
-  </xacro:if>
 </robot>

File: rotor_gazebo/urdf/shredder/shredder_base.xacro (robot description, xacro)
@@ -1,31 +1,201 @@
 <?xml version="1.0"?>
 <!--
-  Copyright 2015 Fadri Furrer, ASL, ETH Zurich, Switzerland
-  Copyright 2015 Michael Burri, ASL, ETH Zurich, Switzerland
-  Copyright 2015 Mina Kamel, ASL, ETH Zurich, Switzerland
-  Copyright 2015 Janosch Nikolic, ASL, ETH Zurich, Switzerland
-  Copyright 2015 Markus Achtelik, ASL, ETH Zurich, Switzerland
-  Licensed under the Apache License, Version 2.0 (the "License");
-  you may not use this file except in compliance with the License.
-  You may obtain a copy of the License at
-  http://www.apache.org/licenses/LICENSE-2.0
-  Unless required by applicable law or agreed to in writing, software
-  distributed under the License is distributed on an "AS IS" BASIS,
-  WITHOUT WARRANTIES OR CONDITIONS OF ANY KIND, either express or implied.
-  See the License for the specific language governing permissions and
-  limitations under the License.
+Gazebo Shredder Definition File
+Author: James Jackson
 -->
 <robot name="shredder" xmlns:xacro="http://ros.org/wiki/xacro">
-  <!-- Instantiate shredder mechanics -->
-  <xacro:include filename="$(find rotor_gazebo)/urdf/shredder/shredder_mechanics.xacro" />
-  <!-- Instantiate a controller for the motors. -->
-  <xacro:include filename="$(find rotor_gazebo_plugins)/xacro/controller_interface.xacro"/>
-  <xacro:controller_plugin_macro namespace="${namespace}" imu_sub_topic="imu" />
-  <!-- Enable Ground Truth - Used by attitude_controller -->
+  <!-- Properties -->
+  <xacro:property name="namespace" value="$(arg mav_name)" />
+  <xacro:property name="rotor_velocity_slowdown_sim" value="10" />
+  <xacro:property name="use_mesh_file" value="true" />
+  <xacro:property name="mesh_file" value="package://rotor_gazebo/meshes/firefly.dae" />
+  <xacro:property name="mass" value="3.81" /> <!-- [kg] -->
+  <xacro:property name="body_width" value="0.1" /> <!-- [m] -->
+  <xacro:property name="body_height" value="0.16" /> <!-- [m] -->
+  <xacro:property name="mass_rotor" value="0.005" /> <!-- [kg] -->
+  <xacro:property name="arm_length" value="0.3429" /> <!-- [m] -->
+  <xacro:property name="rotor_offset_top" value="0.06985" /> <!-- [m] -->
+  <xacro:property name="radius_rotor" value="0.1524" /> <!-- [m] -->
+  <xacro:property name="motor_constant" value="1.426e-5" /> <!-- [N-s/rad] -->
+  <xacro:property name="moment_constant" value="0.055" /> <!-- [m] -->
+  <xacro:property name="time_constant_up" value="0.0215" /> <!-- [s] -->
+  <xacro:property name="time_constant_down" value="0.0375" /> <!-- [s] -->
+  <xacro:property name="max_rot_velocity" value="1177.89" /> <!-- [rad/s] -->
+  <xacro:property name="sin30" value="0.5" />
+  <xacro:property name="cos30" value="0.866025403784" />
+  <xacro:property name="rotor_drag_coefficient" value="8.06428e-05" />
+  <xacro:property name="rolling_moment_coefficient" value="0.000001" />
+  <xacro:property name="body_inertia">
+    <inertia ixx="0.0347563" ixy="0.0" ixz="0.0" iyy="0.0458929" iyz="0.0" izz="0.0977" />
+  </xacro:property>
+  <xacro:property name="rotor_inertia">
+    <xacro:box_inertia x="${radius_rotor}" y="0.015" z="0.003" mass="${mass_rotor*rotor_velocity_slowdown_sim}" />
+  </xacro:property>
+  <!-- *********************** GAZEBO ROBOT DEFINITION ******************* -->
+  <link name="${namespace}/base_link">
+    <inertial>
+      <mass value="${mass}" />  <!-- [kg] -->
+      <origin xyz="0 0 0" />
+      <xacro:insert_block name="body_inertia" />
+    </inertial>
+    <visual>
+      <origin xyz="0 0 0" rpy="0 0 0" />
+      <geometry>
+        <xacro:if value="${use_mesh_file}">
+          <mesh filename="${mesh_file}" scale="1 1 1" />
+        </xacro:if>
+        <xacro:unless value="${use_mesh_file}">
+          <box size="${body_width} ${body_width} ${body_height}"/> <!-- [m] [m] [m] -->
+        </xacro:unless>
+      </geometry>
+    </visual>
+    <collision>
+      <origin xyz="0 0 0" rpy="0 0 0" />
+      <geometry>
+        <box size="${body_width} ${body_width} ${body_height}" /> <!-- [m] [m] [m] -->
+      </geometry>
+    </collision>
+  </link>
+  <!-- ************************* ROTOR DYNAMICS ********************** -->
+  <gazebo>
+    <plugin filename="librotor_gazebo_multirotor_base_plugin.so" name="multirotor_base_plugin">
+      <robotNamespace>${namespace}</robotNamespace>
+      <linkName>${namespace}/base_link</linkName>
+      <rotorVelocitySlowdownSim>${rotor_velocity_slowdown_sim}</rotorVelocitySlowdownSim>
+    </plugin>
+  </gazebo>
+  <!-- **************** ROTORS ***************** -->
+  <xacro:include filename="$(find rotor_gazebo_plugins)/xacro/rotor.xacro" />
+  <xacro:vertical_rotor
+    robot_namespace="${namespace}"
+    suffix="front"
+    direction="cw"
+    motor_constant="${motor_constant}"
+    moment_constant="${moment_constant}"
+    parent="${namespace}/base_link"
+    mass_rotor="${mass_rotor}"
+    radius_rotor="${radius_rotor}"
+    time_constant_up="${time_constant_up}"
+    time_constant_down="${time_constant_down}"
+    max_rot_velocity="${max_rot_velocity}"
+    motor_number="0"
+    rotor_drag_coefficient="${rotor_drag_coefficient}"
+    rolling_moment_coefficient="${rolling_moment_coefficient}"
+    color="Red"
+    use_own_mesh="false"
+    mesh="">
+    <origin xyz="${arm_length} 0 ${rotor_offset_top}" rpy="0 0 0" />
+    <xacro:insert_block name="rotor_inertia" />
+  </xacro:vertical_rotor>
+  <xacro:vertical_rotor
+    robot_namespace="${namespace}"
+    suffix="front_left"
+    direction="ccw"
+    motor_constant="${motor_constant}"
+    moment_constant="${moment_constant}"
+    parent="${namespace}/base_link"
+    mass_rotor="${mass_rotor}"
+    radius_rotor="${radius_rotor}"
+    time_constant_up="${time_constant_up}"
+    time_constant_down="${time_constant_down}"
+    max_rot_velocity="${max_rot_velocity}"
+    motor_number="1"
+    rotor_drag_coefficient="${rotor_drag_coefficient}"
+    rolling_moment_coefficient="${rolling_moment_coefficient}"
+    color="Black"
+    use_own_mesh="false"
+    mesh="">
+    <origin xyz="${sin30*arm_length} ${cos30*arm_length} ${rotor_offset_top}" rpy="0 0 0" />
+    <xacro:insert_block name="rotor_inertia" />
+  </xacro:vertical_rotor>
+  <xacro:vertical_rotor robot_namespace="${namespace}"
+    suffix="back_left"
+    direction="cw"
+    motor_constant="${motor_constant}"
+    moment_constant="${moment_constant}"
+    parent="${namespace}/base_link"
+    mass_rotor="${mass_rotor}"
+    radius_rotor="${radius_rotor}"
+    time_constant_up="${time_constant_up}"
+    time_constant_down="${time_constant_down}"
+    max_rot_velocity="${max_rot_velocity}"
+    motor_number="2"
+    rotor_drag_coefficient="${rotor_drag_coefficient}"
+    rolling_moment_coefficient="${rolling_moment_coefficient}"
+    color="Black"
+    use_own_mesh="false"
+    mesh="">
+    <origin xyz="-${sin30*arm_length} ${cos30*arm_length} ${rotor_offset_top}" rpy="0 0 0" />
+    <xacro:insert_block name="rotor_inertia" />
+  </xacro:vertical_rotor>
+  <xacro:vertical_rotor robot_namespace="${namespace}"
+    suffix="back"
+    direction="ccw"
+    motor_constant="${motor_constant}"
+    moment_constant="${moment_constant}"
+    parent="${namespace}/base_link"
+    mass_rotor="${mass_rotor}"
+    radius_rotor="${radius_rotor}"
+    time_constant_up="${time_constant_up}"
+    time_constant_down="${time_constant_down}"
+    max_rot_velocity="${max_rot_velocity}"
+    motor_number="3"
+    rotor_drag_coefficient="${rotor_drag_coefficient}"
+    rolling_moment_coefficient="${rolling_moment_coefficient}"
+    color="Black"
+    use_own_mesh="false"
+    mesh="">
+    <origin xyz="-${arm_length} 0 ${rotor_offset_top}" rpy="0 0 0" />
+    <xacro:insert_block name="rotor_inertia" />
+  </xacro:vertical_rotor>
+  <xacro:vertical_rotor
+    robot_namespace="${namespace}"
+    suffix="right"
+    direction="cw"
+    motor_constant="${motor_constant}"
+    moment_constant="${moment_constant}"
+    parent="${namespace}/base_link"
+    mass_rotor="${mass_rotor}"
+    radius_rotor="${radius_rotor}"
+    time_constant_up="${time_constant_up}"
+    time_constant_down="${time_constant_down}"
+    max_rot_velocity="${max_rot_velocity}"
+    motor_number="4"
+    rotor_drag_coefficient="${rotor_drag_coefficient}"
+    rolling_moment_coefficient="${rolling_moment_coefficient}"
+    color="Black"
+    use_own_mesh="false"
+    mesh="">
+    <origin xyz="-${sin30*arm_length} -${cos30*arm_length} ${rotor_offset_top}" rpy="0 0 0" />
+    <xacro:insert_block name="rotor_inertia" />
+  </xacro:vertical_rotor>
+  <xacro:vertical_rotor
+    robot_namespace="${namespace}"
+    suffix="front_right"
+    direction="ccw"
+    motor_constant="${motor_constant}"
+    moment_constant="${moment_constant}"
+    parent="${namespace}/base_link"
+    mass_rotor="${mass_rotor}"
+    radius_rotor="${radius_rotor}"
+    time_constant_up="${time_constant_up}"
+    time_constant_down="${time_constant_down}"
+    max_rot_velocity="${max_rot_velocity}"
+    motor_number="5"
+    rotor_drag_coefficient="${rotor_drag_coefficient}"
+    rolling_moment_coefficient="${rolling_moment_coefficient}"
+    color="Black"
+    use_own_mesh="false"
+    mesh="">
+    <origin xyz="${sin30*arm_length} -${cos30*arm_length} ${rotor_offset_top}" rpy="0 0 0" />
+    <xacro:insert_block name="rotor_inertia" />
+  </xacro:vertical_rotor>
+  <!-- ***************** SENSORS ******************* -->
+  <!-- Ground Truth -->
   <xacro:if value="$(arg enable_ground_truth)">
     <xacro:include filename="$(find rotor_gazebo_plugins)/xacro/odometry_sensor.xacro"/>
     <xacro:ground_truth namespace="${namespace}" parent_link="${namespace}/base_link" />
   </xacro:if>
-  <!-- Mount an IMU. -->
+  <!-- Mount an IMU -->
   <xacro:include filename="$(find rotor_gazebo_plugins)/xacro/imu.xacro"/>
   <xacro:IMU_ADIS16448
@@ -34,9 +204,9 @@
     imu_topic="imu"/>
   <!--Enable Wind -->
-  <xacro:include filename="$(find rotor_gazebo_plugins)/xacro/wind.xacro"/>
+<!--   <xacro:include filename="$(find rotor_gazebo_plugins)/xacro/wind.xacro"/>
   <xacro:wind_param
     namespace=""
     link_name="${namespace}/base_link"
-    wind_pub_topic="wind"/>
+    wind_pub_topic="wind"/> -->
   <!-- Mount an Altimeter -->
   <xacro:include filename="$(find rotor_gazebo_plugins)/xacro/altimeter.xacro"/>

Commit message: updated moments of inertia

File: rotor_gazebo/urdf/hummingbird/hummingbird_base.xacro (robot description, xacro)
@@ -25,5 +25,5 @@
   <xacro:property name="rolling_moment_coefficient" value="0.000001" />
   <xacro:property name="body_inertia">
-    <inertia ixx="0.007" ixy="0.0" ixz="0.0" iyy="0.007" iyz="0.0" izz="0.012" />
+    <inertia ixx="0.182" ixy="0.0" ixz="0.0" iyy="0.179" iyz="0.0" izz="0.3258" />
   </xacro:property>
   <xacro:property name="rotor_inertia">
