Commit message: removed the last of rotor_gazebo, fixed a bug and added the first dependancy to fcu_common

File: fcu_sim/urdf/hummingbird/hummingbird_base.xacro (robot description, xacro)
@@ -57,5 +57,5 @@
   <!-- ************************* ROTOR DYNAMICS ********************** -->
   <gazebo>
-    <plugin filename="librotor_gazebo_multirotor_base_plugin.so" name="multirotor_base_plugin">
+    <plugin filename="libfcu_sim_multirotor_base_plugin.so" name="multirotor_base_plugin">
       <robotNamespace>${namespace}</robotNamespace>
       <linkName>${namespace}/base_link</linkName>

File: fcu_sim/urdf/junker/junker_base.xacro (robot description, xacro)
@@ -4,5 +4,5 @@
   <xacro:property name="namespace" value="junker"/>
   <xacro:property name="wind_speed_topic" value="gazebo/wind_speed"/>
-  <xacro:property name="command_topic" value="/command/FWCommand"/>
+  <xacro:property name="command_topic" value="/command"/>
   <xacro:property name="use_mesh_file" value="true" />
   <xacro:property name="mesh_file" value="package://fcu_sim/meshes/ju-87.dae"/>
@@ -145,5 +145,5 @@
   <!-- Add Aerodynamics -->
   <gazebo>
-    <plugin filename="librotor_gazebo_aircraft_forces_and_moments_plugin.so" name="aircraft_forces_and_moments_plugin">
+    <plugin filename="libfcu_sim_aircraft_forces_and_moments_plugin.so" name="aircraft_forces_and_moments_plugin">
       <namespace>${namespace}</namespace>
       <linkName>${namespace}/base_link</linkName>
@@ -224,3 +224,9 @@
     </plugin>
   </gazebo>
+  <!-- Odometry Sensor -->
+  <xacro:include filename="$(find fcu_sim_plugins)/xacro/odometry_sensor.xacro"/>
+  <xacro:ground_truth
+    namespace="${namespace}"
+    parent_link="${namespace}/base_link">
+  </xacro:ground_truth>
 </robot>

File: fcu_sim/urdf/shredder/shredder_base.xacro (robot description, xacro)
@@ -59,5 +59,5 @@
   <!-- ************************* ROTOR DYNAMICS ********************** -->
 <!--   <gazebo>
-    <plugin filename="librotor_gazebo_multirotor_base_plugin.so" name="multirotor_base_plugin">
+    <plugin filename="libfcu_sim_multirotor_base_plugin.so" name="multirotor_base_plugin">
       <robotNamespace>${namespace}</robotNamespace>
       <linkName>${namespace}/base_link</linkName>

File: fcu_sim_plugins/xacro/aircraft_forces_and_moments.xacro (robot description, xacro)
@@ -107,5 +107,5 @@
     </joint>
     <gazebo>
-      <plugin filename="librotor_gazebo_aircraft_and_moments_plugin.so" name="aircraft_forces_and_moments">
+      <plugin filename="libfcu_sim_aircraft_and_moments_plugin.so" name="aircraft_forces_and_moments">
         <linkName>${namespace}/aircraft_forces_and_moments_link</linkName>
         <robotNamespace>${namespace}</robotNamespace>

File: fcu_sim_plugins/xacro/altimeter.xacro (robot description, xacro)
@@ -45,5 +45,5 @@
     </joint>
     <gazebo>
-      <plugin filename="librotor_gazebo_altimeter_plugin.so" name="rotor_gazebo_altimeter${altimeter_suffix}_plugin">
+      <plugin filename="libfcu_sim_altimeter_plugin.so" name="fcu_sim_altimeter${altimeter_suffix}_plugin">
       <!-- A good description of the altimeter parameters can be found in the kalibr documentation:
            https://github.com/ethz-asl/kalibr/wiki/altimeter-Noise-Model-and-Intrinsics -->

File: fcu_sim_plugins/xacro/controller_interface.xacro (robot description, xacro)
@@ -4,5 +4,5 @@
   <xacro:macro name="controller_plugin_macro" params="namespace imu_sub_topic">
     <gazebo>
-      <plugin name="controller_interface" filename="librotor_gazebo_controller_interface.so">
+      <plugin name="controller_interface" filename="libfcu_sim_controller_interface.so">
         <robotNamespace>${namespace}</robotNamespace>
         <commandAttitudeThrustSubTopic>command/attitude</commandAttitudeThrustSubTopic>

File: fcu_sim_plugins/xacro/imu.xacro (robot description, xacro)
@@ -49,5 +49,5 @@
     </joint>
     <gazebo>
-      <plugin filename="librotor_gazebo_imu_plugin.so" name="rotor_gazebo_imu${imu_suffix}_plugin">
+      <plugin filename="libfcu_sim_imu_plugin.so" name="fcu_sim_imu${imu_suffix}_plugin">
       <!-- A good description of the IMU parameters can be found in the kalibr documentation:
            https://github.com/ethz-asl/kalibr/wiki/IMU-Noise-Model-and-Intrinsics -->

File: fcu_sim_plugins/xacro/odometry_sensor.xacro (robot description, xacro)
@@ -61,5 +61,5 @@
     </joint>
     <gazebo>
-      <plugin filename="librotor_gazebo_odometry_plugin.so" name="odometry_sensor${odometry_sensor_suffix}">
+      <plugin filename="libfcu_sim_odometry_plugin.so" name="odometry_sensor${odometry_sensor_suffix}">
         <linkName>${namespace}/odometry_sensor${odometry_sensor_suffix}_link</linkName>
         <robotNamespace>${namespace}</robotNamespace>

File: fcu_sim_plugins/xacro/rotor.xacro (robot description, xacro)
@@ -66,5 +66,5 @@
     </link>
     <gazebo>
-      <plugin name="${robot_namespace}_${suffix}_motor_model" filename="librotor_gazebo_motor_model.so">
+      <plugin name="${robot_namespace}_${suffix}_motor_model" filename="libfcu_sim_motor_model.so">
         <robotNamespace>${robot_namespace}</robotNamespace>
         <jointName>${robot_namespace}/rotor_${motor_number}_joint</jointName>

File: fcu_sim_plugins/xacro/wind.xacro (robot description, xacro)
@@ -27,5 +27,5 @@
           wind_gust_force_variance wind_gust_direction">
     <gazebo>
-      <plugin filename="librotor_gazebo_wind_plugin.so" name="gazebo_wind_plugin">
+      <plugin filename="libfcu_sim_wind_plugin.so" name="gazebo_wind_plugin">
         <robotNamespace>${namespace}</robotNamespace> <!-- (string, required): ros namespace in which the messages are published -->
         <xyzOffset>${xyz_offset}</xyzOffset> <!-- (Vector3, required): -->

Commit message: added the attitude controller back in

File: fcu_sim/urdf/hummingbird/hummingbird_base.xacro (robot description, xacro)
@@ -6,5 +6,5 @@
 <robot name="hummingbird" xmlns:xacro="http://ros.org/wiki/xacro">
   <!-- Properties -->
-  <xacro:property name="namespace" value="$(arg mav_name)" />
+  <xacro:property name="namespace" value="" />
   <xacro:property name="rotor_velocity_slowdown_sim" value="10" />
   <xacro:property name="use_mesh_file" value="true" />
@@ -158,4 +158,23 @@
   <!-- Enable Ground Truth -->
   <xacro:include filename="$(find fcu_sim_plugins)/xacro/odometry_sensor.xacro"/>
-  <xacro:ground_truth namespace="${namespace}" parent_link="${namespace}/base_link" />
+  <xacro:ground_truth
+    namespace="${namespace}"
+    parent_link="${namespace}/base_link" />
+  <!-- Altimeter -->
+  <xacro:include filename="$(find fcu_sim_plugins)/xacro/altimeter.xacro"/>
+  <xacro:Sonar_HC-SR04
+    namespace="${namespace}"
+    parent_link="${namespace}/base_link"
+    altimeter_topic="alt/data"/>
+    <!-- Downward Pointing Camera -->
+    <xacro:include filename="$(find fcu_sim_plugins)/xacro/camera.xacro"/>
+    <xacro:simple_camera
+      namespace="${namespace}"
+      frame_rate="30"
+      rgb_range=""
+      parent_link="${namespace}/base_link"
+      image_topic="rgb"
+      image_camera_info_topic="camera_info">
+      <origin xyz="0.0 0.0 -0.2" rpy="0 1.516 0"/>
+    </xacro:simple_camera>
 </robot>

Commit message: fixing multi-agent stuff

File: fcu_sim/urdf/hummingbird/hummingbird_base.xacro (robot description, xacro)
@@ -6,5 +6,5 @@
 <robot name="hummingbird" xmlns:xacro="http://ros.org/wiki/xacro">
   <!-- Properties -->
-  <xacro:property name="namespace" value="" />
+  <xacro:property name="namespace" value="hummingbird" />
   <xacro:property name="rotor_velocity_slowdown_sim" value="10" />
   <xacro:property name="use_mesh_file" value="true" />
@@ -161,4 +161,10 @@
     namespace="${namespace}"
     parent_link="${namespace}/base_link" />
+  <!-- Add Laser Scanner -->
+  <xacro:include filename="$(find fcu_sim_plugins)/xacro/laser_scanner.xacro"/>
+  <xacro:hokuyo_UTM-30LX
+    namespace="${namespace}"
+    parent_link="${namespace}/base_link"
+    visualize="true"/>
   <!-- Altimeter -->
   <xacro:include filename="$(find fcu_sim_plugins)/xacro/altimeter.xacro"/>

File: fcu_sim/urdf/shredder/shredder_base.xacro (robot description, xacro)
@@ -226,4 +226,4 @@
     namespace="${namespace}"
     parent_link="${namespace}/base_link"
-    visualize="false"/>
+    visualize="true"/>
 </robot>

File: fcu_sim_plugins/xacro/camera.xacro (robot description, xacro)
@@ -20,10 +20,10 @@
         <xacro:insert_block name="empty_inertia"/>
       </inertial>
-      <visual name="${namespace}/camera_visual">
+      <!-- <visual name="${namespace}/camera_visual">
         <xacro:insert_block name="origin"/>
         <geometry>
           <sphere radius="0.05"/>
         </geometry>
-      </visual>
+      </visual> -->
     </link>
     <joint name="${namespace}/camera_joint" type="fixed">
