Commit message: added ROSflight2, gazebo plugin, and simplified multirotor dynamics

File: fcu_sim/urdf/mikey_simple/mikey_simple_base.xacro (robot description, xacro)
@@ -9,21 +9,10 @@
   <xacro:property name="rotor_velocity_slowdown_sim" value="10" />
   <xacro:property name="use_mesh_file" value="true" />
-  <xacro:property name="mesh_file" value="package://fcu_sim/meshes/firefly.dae" />
-  <xacro:property name="mass" value="3.562" /> <!-- [kg] -->
+  <xacro:property name="mesh_file" value="package://fcu_sim/meshes/pelican.dae" />
+  <xacro:property name="mass" value="3.856" /> <!-- [kg] -->
   <xacro:property name="body_width" value="0.505" /> <!-- [m] -->
   <xacro:property name="body_height" value="0.1" /> <!-- [m] -->
-  <xacro:property name="mass_rotor" value="0.005" /> <!-- [kg] -->
-  <xacro:property name="arm_length" value="0.3429" /> <!-- [m] -->
-  <xacro:property name="rotor_offset_top" value="0.06985" /> <!-- [m] -->
-  <xacro:property name="radius_rotor" value="0.1524" /> <!-- [m] -->
-  <xacro:property name="motor_constant" value="1.426e-5" /> <!-- [N-s/rad] -->
-  <xacro:property name="moment_constant" value="0.055" /> <!-- [m] -->
-  <xacro:property name="time_constant_up" value="0.0215" /> <!-- [s] -->
-  <xacro:property name="time_constant_down" value="0.0375" /> <!-- [s] -->
-  <xacro:property name="max_rot_velocity" value="1177.89" /> <!-- [rad/s] -->
   <xacro:property name="sin30" value="0.5" />
   <xacro:property name="cos30" value="0.866025403784" />
-  <xacro:property name="rotor_drag_coefficient" value="8.06428e-05" />
-  <xacro:property name="rolling_moment_coefficient" value="0.000001" />
   <xacro:property name="body_inertia">
     <inertia ixx="0.0347563" ixy="0.0" ixz="0.0" iyy="0.0458929" iyz="0.0" izz="0.0977" />
@@ -47,4 +36,5 @@
       </geometry>
     </visual>
+    <!-- Prop guard -->
     <collision>
       <origin xyz="0 0 0" rpy="0 0 0" />
@@ -57,5 +47,5 @@
     <material>Gazebo/$(arg color)</material>
   </gazebo>
-  <!-- ************************* ROTOR DYNAMICS ********************** -->
+  <!-- ******************  FORCES AND MOMENTS **************** -->
   <xacro:include filename="$(find fcu_sim_plugins)/xacro/ROSflight_SIL.xacro"/>
   <xacro:mikey_ROSflight_SIL namespace="${namespace}" parent_link="${namespace}/base_link"/>
@@ -71,15 +61,15 @@
     imu_topic="imu/data"/>
   <!--Enable Wind -->
-  <!-- <xacro:include filename="$(find fcu_sim_plugins)/xacro/wind.xacro"/>
+  <xacro:include filename="$(find fcu_sim_plugins)/xacro/wind.xacro"/>
   <xacro:wind_param
     namespace="${namespace}"
     link_name="${namespace}/base_link"
-    wind_pub_topic="wind"/> -->
+    wind_pub_topic="wind"/>
   <!-- Mount an Altimeter -->
-  <!-- <xacro:include filename="$(find fcu_sim_plugins)/xacro/altimeter.xacro"/>
+  <xacro:include filename="$(find fcu_sim_plugins)/xacro/altimeter.xacro"/>
   <xacro:Sonar_MB1030
     namespace="${namespace}"
     parent_link="${namespace}/base_link"
-    altimeter_topic="altimeter"/> -->
+    altimeter_topic="altimeter"/>
   <!-- Mount an RGBD Camera -->
   <xacro:include filename="$(find fcu_sim_plugins)/xacro/rgbd.xacro"/>
@@ -88,9 +78,9 @@
     parent_link="${namespace}/base_link"/>
   <!-- Laser Scanner -->
-  <!-- <xacro:include filename="$(find fcu_sim_plugins)/xacro/laser_scanner.xacro"/>
+  <xacro:include filename="$(find fcu_sim_plugins)/xacro/laser_scanner.xacro"/>
   <xacro:hokuyo_UTM-30LX
     namespace="${namespace}"
     parent_link="${namespace}/base_link"
-    visualize="false"/> -->
+    visualize="false"/>
     <!-- Collision Sensor -->
     <!-- TODO  http://gazebosim.org/tutorials?tut=contact_sensor-->

File: fcu_sim_plugins/xacro/ROSflight_SIL.xacro (robot description, xacro)
@@ -4,20 +4,20 @@
     <!-- Forces And Moments Plugin -->
     <xacro:macro
-      name="mikey_hil"
+      name="mikey_ROSflight_SIL"
       params="namespace parent_link">
-      <xacro:multirotor_hil_macro
+      <xacro:fcu_sim_ROSflight_sil_plugin
         namespace="${namespace}/hil"
         parent_link="${namespace}/base_link"
         wind_speed_topic="gazebo/wind_speed"
-        command_topic="servo_output_raw"
+        command_topic="extended_command"
         parent_frame_id="${parent_link}"
         mu="1"
         rotor_max_thrust="14.961"
-        rotor_F1="-0.00001"
-        rotor_F2="0.0452"
-        rotor_F3="-35.117"
-        rotor_T1="-0.00000002"
-        rotor_T2="0.00008"
-        rotor_T3="-0.0586"
+        rotor_F1="1.5e-5"
+        rotor_F2="-0.024451"
+        rotor_F3="9.00225"
+        rotor_T1="-2.22e-7"
+        rotor_T2="3.51e-4"
+        rotor_T3="-0.12531"
         rotor_tau_down="0.1644"
         rotor_tau_up="0.2164"
@@ -49,8 +49,8 @@
         <inertia ixx="0.00001" ixy="0.0" ixz="0.0" iyy="0.00001" iyz="0.0" izz="0.00001" />
         <origin xyz="0.0 0.0 0.0" rpy="0.0 0.0 0.0" />
-      </xacro:multirotor_hil_macro>
+      </xacro:fcu_sim_ROSflight_sil_plugin>
     </xacro:macro>
   <!-- Macro to add a generic multirotor forces and moments plugin. -->
-  <xacro:macro name="multirotor_hil_macro"
+  <xacro:macro name="fcu_sim_ROSflight_sil_plugin"
     params="
         namespace parent_link wind_speed_topic command_topic parent_frame_id
@@ -64,5 +64,5 @@
         *inertia *origin">
     <!-- link -->
-    <link name="${namespace}/multirotor_hil_link">
+    <link name="${namespace}/ROSflight_SIL_link">
       <inertial>
         <xacro:insert_block name="inertia" />
@@ -71,14 +71,14 @@
     </link>
     <!-- joint -->
-    <joint name="${namespace}/multirotor_hil_joint" type="revolute">
+    <joint name="${namespace}/aircraft_forces_and_moments_joint" type="revolute">
       <parent link="${parent_link}" />
       <xacro:insert_block name="origin" />
-      <child link="${namespace}/multirotor_hil_link" />
+      <child link="${namespace}/ROSflight_SIL_link" />
       <limit upper="0" lower="0" effort="0" velocity="0" />
     </joint>
     <!-- plugin -->
     <gazebo>
-      <plugin filename="libfcu_sim_naze_hil_multirotor_plugin.so" name="multirotor_hil">
-        <linkName>${namespace}/multirotor_hil_link</linkName>
+      <plugin filename="libfcu_sim_ROSflight_sil_plugin.so" name="multirotor_hil">
+        <linkName>${namespace}/ROSflight_SIL_link</linkName>
         <robotNamespace>${namespace}</robotNamespace>
         <windSpeedTopic>${wind_speed_topic}</windSpeedTopic>
