Commit message: fixed IMU so gravity is applied right direction

File: fcu_sim/urdf/shredder/shredder_base.xacro (robot description, xacro)
@@ -63,25 +63,25 @@
   <!--Enable Wind -->
   <xacro:include filename="$(find fcu_sim_plugins)/xacro/wind.xacro"/>
-  <xacro:wind_param
+  <!-- <xacro:wind_param
     namespace="${namespace}"
     link_name="${namespace}/base_link"
-    wind_pub_topic="wind"/>
+    wind_pub_topic="wind"/> -->
   <!-- Mount an Altimeter -->
   <xacro:include filename="$(find fcu_sim_plugins)/xacro/altimeter.xacro"/>
-  <xacro:Sonar_MB1030
+  <xacro:perfect_baro
     namespace="${namespace}"
     parent_link="${namespace}/base_link"
     altimeter_topic="altimeter"/>
   <!-- Mount an RGBD Camera -->
-  <xacro:include filename="$(find fcu_sim_plugins)/xacro/rgbd.xacro"/>
+  <!-- <xacro:include filename="$(find fcu_sim_plugins)/xacro/rgbd.xacro"/>
   <xacro:xtion
     namespace="${namespace}"
-    parent_link="${namespace}/base_link"/>
+    parent_link="${namespace}/base_link"/> -->
   <!-- Laser Scanner -->
-  <xacro:include filename="$(find fcu_sim_plugins)/xacro/velodyne.xacro"/>
+  <!-- <xacro:include filename="$(find fcu_sim_plugins)/xacro/velodyne.xacro"/>
   <xacro:velodyne_custom
     namespace="${namespace}"
     parent_link="${namespace}/base_link"
-    visualize="false"/>
+    visualize="false"/> -->
   <!-- GPS -->
   <xacro:include filename="$(find fcu_sim_plugins)/xacro/GPS.xacro"/>

File: fcu_sim_plugins/xacro/altimeter.xacro (robot description, xacro)
@@ -2,4 +2,25 @@
 <robot xmlns:xacro="http://ros.org/wiki/xacro">
   <xacro:property name="pi" value="3.14159265359" />
+  <!-- Perfect Barometer -->
+  <xacro:macro
+    name="perfect_baro"
+    params="namespace parent_link altimeter_topic">
+    <xacro:altimeter_plugin_macro
+      namespace="${namespace}"
+      altimeter_suffix="sonar"
+      parent_link="${parent_link}"
+      altimeter_topic="${altimeter_topic}"
+      mass_altimeter_sensor="0.0043"
+      altimeter_min_range="0.0"
+      altimeter_max_range="1000.0"
+      altimeter_error_stdev="0.0000000001"
+      altimeter_field_of_view="0.000001"
+      altimeter_publish_rate="20"
+      altimeter_noise_on="0"
+      publish_float="0" >
+      <inertia ixx="0.00001" ixy="0.0" ixz="0.0" iyy="0.00001" iyz="0.0" izz="0.00001" />
+      <origin xyz="0 0 0" rpy="0 0 0" />
+    </xacro:altimeter_plugin_macro>
+  </xacro:macro>
   <!-- Sonar  HC-SR04 -->
   <xacro:macro
@@ -65,4 +86,24 @@
     </xacro:altimeter_plugin_macro>
   </xacro:macro>
+  <xacro:macro
+    name="Sonar_MB1030"
+    params="namespace parent_link altimeter_topic">
+    <xacro:altimeter_plugin_macro
+      namespace="${namespace}"
+      altimeter_suffix=""
+      parent_link="${parent_link}"
+      altimeter_topic="${altimeter_topic}"
+      mass_altimeter_sensor="0.0043"
+      altimeter_min_range="0.381"
+      altimeter_max_range="6.45"
+      altimeter_error_stdev="0.10"
+      altimeter_field_of_view="1.107"
+      altimeter_publish_rate="20"
+      altimeter_noise_on="1"
+      publish_float="0" >
+      <inertia ixx="0.00001" ixy="0.0" ixz="0.0" iyy="0.00001" iyz="0.0" izz="0.00001" />
+      <origin xyz="0 0 0" rpy="0 0 0" />
+    </xacro:altimeter_plugin_macro>
+  </xacro:macro>
   <!-- Macro to add an altimeter. -->
   <xacro:macro name="altimeter_plugin_macro"

Commit message: tested and working magnetometer

File: fcu_sim/urdf/shredder/shredder_base.xacro (robot description, xacro)
@@ -74,4 +74,13 @@
     parent_link="${namespace}/base_link"
     altimeter_topic="altimeter"/>
+  <!-- Mount a Magnetometer -->
+  <!-- Default Inclination and Declination for Provo, UT -->
+  <xacro:include filename="$(find fcu_sim_plugins)/xacro/magnetometer.xacro"/>
+  <xacro:hmc5883l
+    namespace="${namespace}"
+    parent_link="${namespace}/base_link"
+    mag_topic="mag/data"
+    inclination="1.14316156541"
+    declination="0.198584539676"/>
   <!-- Mount an RGBD Camera -->
   <!-- <xacro:include filename="$(find fcu_sim_plugins)/xacro/rgbd.xacro"/>

File: fcu_sim_plugins/xacro/magnetometer.xacro (robot description, xacro)
@@ -1,9 +1,8 @@
 <?xml version="1.0"?>
 <robot xmlns:xacro="http://ros.org/wiki/xacro">
-  <xacro:property name="pi" value="3.14159265359" />
-  <!-- Perfect Barometer -->
+  <!-- HMC5883L (on Naze32 and PixHawk) -->
   <xacro:macro
     name="hmc5883l"
-    params="namespace parent_link mag_topic inclination declination"/>
+    params="namespace parent_link mag_topic inclination declination">
     <xacro:magnetometer_plugin_macro
       namespace="${namespace}"
@@ -11,4 +10,5 @@
       mag_topic="${mag_topic}"
       noise_sigma="0.02"
+      bias_sigma="0.02"
       pub_rate="160"
       declination="${declination}"
@@ -18,5 +18,5 @@
     </xacro:magnetometer_plugin_macro>
   </xacro:macro>
-    <!-- Macro to add an altimeter. -->
+    <!-- Macro to add a magnetometer. -->
   <xacro:macro name="magnetometer_plugin_macro"
     params="namespace
@@ -24,4 +24,5 @@
             mag_topic
             noise_sigma
+            bias_sigma
             pub_rate
             declination
@@ -29,5 +30,5 @@
             *inertia
             *origin">
-    <!-- altimeter link -->
+    <!-- mag link -->
     <link name="${namespace}/magnetometer_link">
       <inertial>
@@ -37,5 +38,5 @@
       </inertial>
     </link>
-    <!-- magnetometer joint -->
+    <!-- mag joint -->
     <joint name="${namespace}/magnetometer_joint" type="revolute">
       <xacro:insert_block name="origin" />
@@ -46,12 +47,12 @@
     <gazebo>
       <plugin filename="libfcu_sim_magnetometer_plugin.so" name="fcu_sim_magnetometer_plugin">
-      <namespace>${namespace}<namespace/>
-      <linkName>${linkName}<linkName/>
-      <mag_topic>${mag_topic}<mag_topic/>
-      <noise_sigma>${noise_sigma}<noise_sigma/>
-      <bias_sigma>${bias_sigma}<bias_sigma/>
-      <pub_rate>${pub_rate}<pub_rate/>
-      <declination>${declination}<declination/>
-      <inclination>${inclination}<inclination/>
+      <namespace>${namespace}</namespace>
+      <linkName>${namespace}/magnetometer_link</linkName>
+      <mag_topic>${mag_topic}</mag_topic>
+      <noise_sigma>${noise_sigma}</noise_sigma>
+      <bias_sigma>${bias_sigma}</bias_sigma>
+      <pub_rate>${pub_rate}</pub_rate>
+      <declination>${declination}</declination>
+      <inclination>${inclination}</inclination>
       </plugin>
     </gazebo>

Commit message: stopped using millenium falcon because it caused Gazebo 7 to crash

File: fcu_sim/urdf/shredder/shredder_base.xacro (robot description, xacro)
@@ -8,5 +8,5 @@
 <xacro:property name="namespace" value="shredder" />
 <xacro:property name="use_mesh_file" value="true" />
-<xacro:property name="mesh_file" value="package://fcu_sim/meshes/Millennium_Falcon.dae" />
+<xacro:property name="mesh_file" value="package://fcu_sim/meshes/firefly.dae" />
 <xacro:property name="mass" value="3.81" /> <!-- [kg] -->
 <xacro:property name="body_width" value="0.505" /> <!-- [m] -->
@@ -27,6 +27,6 @@
     <geometry>
       <xacro:if value="${use_mesh_file}">
-        <mesh filename="${mesh_file}" scale="0.001 0.001 0.001" />
-        <!-- <mesh filename="${mesh_file}" scale="1 1 1" /> -->
+        <!-- <mesh filename="${mesh_file}" scale="0.001 0.001 0.001" /> -->
+        <mesh filename="${mesh_file}" scale="1 1 1" />
       </xacro:if>
       <xacro:unless value="${use_mesh_file}">
@@ -47,5 +47,5 @@
   <!-- ************************* ROTOR DYNAMICS ********************** -->
   <!-- ROSflight_SIL -->
-  <xacro:include filename="$(find fcu_sim_plugins)/xacro/ROSflight_SIL.xacro"/>
+  <!-- <xacro:include filename="$(find fcu_sim_plugins)/xacro/ROSflight_SIL.xacro"/> -->
   <!-- <xacro:mikey_ROSflight_SIL namespace="${namespace}" parent_link="${namespace}/base_link"/> -->
   <!-- Simplified Dynamics -->
