Commit message: Fixed gimbal physics
Reduced the gimbal mass by two orders of magnitude. This appears to fix the issue in Gazebo that was causing the fixedwing to fly erratically when a gimbal was attached.

File: fcu_sim_plugins/xacro/gimbal.xacro (robot description, xacro)
@@ -16,5 +16,5 @@
       pose_topic="${pose_topic}"
       command_topic="${command_topic}"
-      mass="0.001"
+      mass="0.00001"
       x_rotation_range="1000000000"
       y_rotation_range="1000000000"
@@ -50,5 +50,5 @@
       <inertial>
         <inertia ixx="0.00001" ixy="0.0" ixz="0.0" iyy="0.00001" iyz="0.0" izz="0.00001" />
-        <mass value="0.0001" />
+        <mass value="${mass}" />
         <origin xyz="0 0 0" rpy = "0 0 0"/>
       </inertial>
@@ -65,5 +65,5 @@
       <inertial>
         <inertia ixx="0.00001" ixy="0.0" ixz="0.0" iyy="0.00001" iyz="0.0" izz="0.00001" />
-        <mass value="0.0001" />
+        <mass value="${mass}" />
         <origin xyz="0 0 0" rpy = "0 0 0"/>
       </inertial>
@@ -80,5 +80,5 @@
       <inertial>
         <inertia ixx="0.00001" ixy="0.0" ixz="0.0" iyy="0.00001" iyz="0.0" izz="0.00001" />
-        <mass value="0.0001" />
+        <mass value="${mass}" />
         <origin xyz="0 0 0" rpy = "0 0 0"/>
       </inertial>
