Commit message: some cleanup

File: fcu_sim_plugins/xacro/laser_scanner.xacro (robot description, xacro)
@@ -6,5 +6,6 @@
     params="namespace
             parent_link
-            visualize">
+            visualize
+            *origin">
     <xacro:laser_scanner
       namespace="${namespace}"
@@ -18,5 +19,5 @@
       max_angle="pi/2"
       update_rate="40">
-      <origin xyz="0.09525 0 -0.0127" rpy="0 0 0" />
+      <xacro:insert_block name="origin"/>
     </xacro:laser_scanner>
   </xacro:macro>
