Commit message: got rid of unecessary links in xacro files

File: fcu_sim_plugins/xacro/GPS.xacro (robot description, xacro)
@@ -32,24 +32,9 @@
       sample_time mass_gps_sensor
       *inertia *origin">
-    <!-- GPS link -->
-    <link name="${namespace}/GPS_link">
-      <inertial>
-        <xacro:insert_block name="inertia" />
-        <mass value="${mass_gps_sensor}" />
-        <origin xyz="0 0 0" rpy="0 0 0" />
-      </inertial>
-    </link>
-    <!-- GPS joint -->
-    <joint name="${namespace}/GPS_joint" type="revolute">
-      <xacro:insert_block name="origin" />
-      <parent link="${parent_link}" />
-      <child link="${namespace}/GPS_link" />
-      <limit upper="0" lower="0" effort="0" velocity="0" />
-    </joint>
     <!-- Load Plugin -->
     <gazebo>
       <plugin filename="libGPS_plugin.so" name="fcu_sim_GPS_plugin">
       <namespace>${namespace}</namespace>
-      <linkName>${namespace}/GPS_link</linkName>
+      <linkName>${parent_link}</linkName>
       <GPSTopic>${gps_topic}</GPSTopic>
       <north_stdev>${north_stdev}</north_stdev>

File: fcu_sim_plugins/xacro/ROSflight_SIL.xacro (robot description, xacro)
@@ -112,27 +112,15 @@
         ground_effect_a ground_effect_b ground_effect_c ground_effect_d ground_effect_e
         num_rotors rotor_max_thrust rotor_F1 rotor_F2 rotor_F3 rotor_T1 rotor_T2 rotor_T3
-        rotor_tau_down rotor_tau_up  rotor1_distance rotor1_angle rotor1_direction rotor2_distance rotor2_angle rotor2_direction rotor3_distance rotor3_angle rotor3_direction rotor4_distance rotor4_angle
+        rotor_tau_down rotor_tau_up  rotor1_distance rotor1_angle
+        rotor1_direction rotor2_distance rotor2_angle rotor2_direction
+        rotor3_distance rotor3_angle rotor3_direction rotor4_distance rotor4_angle
         rotor4_direction rotor5_distance rotor5_angle rotor5_direction rotor6_distance
         rotor6_angle rotor6_direction rotor7_distance rotor7_angle  rotor7_direction
         rotor8_distance rotor8_angle  rotor8_direction
         *inertia *origin">
-    <!-- link -->
-    <link name="${namespace}/ROSflight_SIL_link">
-      <inertial>
-        <xacro:insert_block name="inertia" />
-        <mass value="0.001"/>  <!-- [kg] -->
-      </inertial>
-    </link>
-    <!-- joint -->
-    <joint name="${namespace}/aircraft_forces_and_moments_joint" type="revolute">
-      <parent link="${parent_link}" />
-      <xacro:insert_block name="origin" />
-      <child link="${namespace}/ROSflight_SIL_link" />
-      <limit upper="0" lower="0" effort="0" velocity="0" />
-    </joint>
     <!-- plugin -->
     <gazebo>
       <plugin filename="libROSflight_sil_plugin.so" name="multirotor_hil">
-        <linkName>${namespace}/ROSflight_SIL_link</linkName>
+        <linkName>${parent_link}</linkName>
         <robotNamespace>${namespace}</robotNamespace>
         <windSpeedTopic>${wind_speed_topic}</windSpeedTopic>

File: fcu_sim_plugins/xacro/aircraft_truth.xacro (robot description, xacro)
@@ -1,5 +1,5 @@
 <?xml version="1.0"?>
 <robot xmlns:xacro="http://ros.org/wiki/xacro">
-  <!-- Configure GPS -->
+  <!-- Configure Aircraft Truth Macro -->
     <xacro:macro
       name="aircraft_truth"

File: fcu_sim_plugins/xacro/airspeed.xacro (robot description, xacro)
@@ -9,39 +9,18 @@
       parent_link="${parent_link}"
       airspeed_topic="${airspeed_topic}"
-      mass_airspeed_sensor="0.001"
       pressure_bias="00.0"
       pressure_noise_sigma="2.0"
       max_pressure="4000.0"
       air_density="1.225"
-      min_pressure="0.0">
-      <inertia ixx="0.00001" ixy="0.0" ixz="0.0" iyy="0.00001" iyz="0.0" izz="0.00001" />
-      <origin xyz="0 0 0" rpy="0 0 0" />
-    </xacro:airspeed_plugin_macro>
+      min_pressure="0.0"/>
   </xacro:macro>
     <!-- Macro to add an Airspeed. -->
   <xacro:macro name="airspeed_plugin_macro"
-    params="namespace parent_link airspeed_topic pressure_bias pressure_noise_sigma air_density
-      mass_airspeed_sensor max_pressure min_pressure
-      *inertia *origin">
-    <!-- Airspeed link -->
-    <link name="${namespace}/airspeed_link">
-      <inertial>
-        <xacro:insert_block name="inertia" />
-        <mass value="${mass_airspeed_sensor}" />
-        <origin xyz="0 0 0" rpy="0 0 0" />
-      </inertial>
-    </link>
-    <!-- Airspeed joint -->
-    <joint name="${namespace}/airspeed_joint" type="revolute">
-      <xacro:insert_block name="origin" />
-      <parent link="${parent_link}" />
-      <child link="${namespace}/airspeed_link" />
-      <limit upper="0" lower="0" effort="0" velocity="0" />
-    </joint>
+    params="namespace parent_link airspeed_topic pressure_bias pressure_noise_sigma air_density max_pressure min_pressure">
     <!-- Load Plugin -->
     <gazebo>
       <plugin filename="libairspeed_plugin.so" name="fcu_sim_airspeed_plugin">
         <namespace>${namespace}</namespace>
-        <linkName>${namespace}/airspeed_link</linkName>
+        <linkName>${parent_link}</linkName>
         <airspeedTopic>${airspeed_topic}</airspeedTopic>
         <pressureBias>${pressure_bias}</pressureBias> <!-- [Pascals] -->

File: fcu_sim_plugins/xacro/barometer.xacro (robot description, xacro)
@@ -30,23 +30,8 @@
     namespace parent_link baro_topic
     noise_stdev update_rate noise_on">
-    <!-- altimeter link -->
-    <link name="${namespace}/barometer_link">
-      <inertial>
-        <inertia ixx="0.00001" ixy="0.0" ixz="0.0" iyy="0.00001" iyz="0.0" izz="0.00001" />
-        <mass value="0.0001"/>
-        <origin xyz="0 0 0" rpy="0 0 0" />
-      </inertial>
-    </link>
-    <!-- altimeter joint -->
-    <joint name="${namespace}/barometer_joint" type="revolute">
-      <origin xyz="0 0 0" rpy="0 0 0" />
-      <parent link="${parent_link}" />
-      <child link="${namespace}/barometer_link" />
-      <limit upper="0" lower="0" effort="0" velocity="0" />
-    </joint>
     <gazebo>
       <plugin filename="libbarometer_plugin.so" name="${namespace}_barometer_plugin">
         <namespace>${namespace}</namespace>
-        <linkName>${namespace}/barometer_link</linkName>
+        <linkName>${parent_link}</linkName>
         <messageTopic>${baro_topic}</messageTopic>
         <noiseStdev>${noise_stdev}</noiseStdev>

File: fcu_sim_plugins/xacro/imu.xacro (robot description, xacro)
@@ -7,8 +7,6 @@
     <xacro:imu_plugin_macro
       namespace="${namespace}"
-      imu_suffix=""
       parent_link="${parent_link}"
       imu_topic="${imu_topic}"
-      mass_imu_sensor="0.0001"
       gyroscope_noise_density="0.0"
       gyroscopoe_random_walk="0.0"
@@ -20,6 +18,4 @@
       accelerometer_turn_on_bias_sigma="0.0"
       perfect_imu="true">
-      <inertia ixx="0.00001" ixy="0.0" ixz="0.0" iyy="0.00001" iyz="0.0" izz="0.00001" />
-      <origin xyz="0 0 0" rpy="0 0 0" />
     </xacro:imu_plugin_macro>
   </xacro:macro>
@@ -29,8 +25,6 @@
     <xacro:imu_plugin_macro
       namespace="${namespace}"
-      imu_suffix=""
       parent_link="${parent_link}"
       imu_topic="${imu_topic}"
-      mass_imu_sensor="0.015"
       gyroscope_noise_density="0.0003394"
       gyroscopoe_random_walk="0.000038785"
@@ -42,6 +36,4 @@
       accelerometer_turn_on_bias_sigma="0.1960"
       perfect_imu="false">
-      <inertia ixx="0.00001" ixy="0.0" ixz="0.0" iyy="0.00001" iyz="0.0" izz="0.00001" />
-      <origin xyz="0 0 0" rpy="0 0 0" />
     </xacro:imu_plugin_macro>
   </xacro:macro>
@@ -52,8 +44,6 @@
     <xacro:imu_plugin_macro
       namespace="${namespace}"
-      imu_suffix=""
       parent_link="${parent_link}"
       imu_topic="${imu_topic}"
-      mass_imu_sensor="0.015"
       gyroscope_noise_density="0.008726646"
       gyroscopoe_random_walk="0.000038785"
@@ -71,6 +61,6 @@
     <!-- Macro to add an IMU. -->
   <xacro:macro name="imu_plugin_macro"
-    params="namespace imu_suffix parent_link imu_topic
-      mass_imu_sensor gyroscope_noise_density gyroscopoe_random_walk
+    params="namespace parent_link imu_topic
+      gyroscope_noise_density gyroscopoe_random_walk
       gyroscope_bias_correlation_time gyroscope_turn_on_bias_sigma
       accelerometer_noise_density accelerometer_random_walk
@@ -78,25 +68,10 @@
       perfect_imu
       *inertia *origin">
-    <!-- IMU link -->
-    <link name="${namespace}/imu${imu_suffix}_link">
-      <inertial>
-        <xacro:insert_block name="inertia" />
-        <mass value="${mass_imu_sensor}" />
-        <origin xyz="0 0 0" rpy="0 0 0" />
-      </inertial>
-    </link>
-    <!-- IMU joint -->
-    <joint name="${namespace}/imu${imu_suffix}_joint" type="revolute">
-      <xacro:insert_block name="origin" />
-      <parent link="${parent_link}" />
-      <child link="${namespace}/imu${imu_suffix}_link" />
-      <limit upper="0" lower="0" effort="0" velocity="0" />
-    </joint>
     <gazebo>
-      <plugin filename="libimu_plugin.so" name="fcu_sim_imu${imu_suffix}_plugin">
+      <plugin filename="libimu_plugin.so" name="${namespace}_imu_plugin">
       <!-- A good description of the IMU parameters can be found in the kalibr documentation:
            https://github.com/ethz-asl/kalibr/wiki/IMU-Noise-Model-and-Intrinsics -->
         <robotNamespace>${namespace}</robotNamespace> <!-- (string, required): ros namespace in which the messages are published -->
-        <linkName>${namespace}/imu${imu_suffix}_link</linkName> <!-- (string, required): name of the body which holds the IMU sensor -->
+        <linkName>${parent_link}</linkName> <!-- (string, required): name of the body which holds the IMU sensor -->
         <imuTopic>${imu_topic}</imuTopic> <!-- (string): name of the sensor output topic and prefix of service names (defaults to imu) -->
         <gyroscopeNoiseDensity>${gyroscope_noise_density}</gyroscopeNoiseDensity> <!-- Gyroscope noise density (two-sided spectrum) [rad/s/sqrt(Hz)] -->

File: fcu_sim_plugins/xacro/magnetometer.xacro (robot description, xacro)
@@ -14,6 +14,4 @@
       declination="${declination}"
       inclination="${inclination}">
-      <inertia ixx="0.00001" ixy="0.0" ixz="0.0" iyy="0.00001" iyz="0.0" izz="0.00001" />
-      <origin xyz="0 0 0" rpy="0 0 0" />
     </xacro:magnetometer_plugin_macro>
   </xacro:macro>
@@ -30,23 +28,8 @@
             *inertia
             *origin">
-    <!-- mag link -->
-    <link name="${namespace}/magnetometer_link">
-      <inertial>
-        <xacro:insert_block name="inertia" />
-        <mass value="0.0001" />
-        <origin xyz="0 0 0" rpy="0 0 0" />
-      </inertial>
-    </link>
-    <!-- mag joint -->
-    <joint name="${namespace}/magnetometer_joint" type="revolute">
-      <xacro:insert_block name="origin" />
-      <parent link="${parent_link}" />
-      <child link="${namespace}/magnetometer_link" />
-      <limit upper="0" lower="0" effort="0" velocity="0" />
-    </joint>
     <gazebo>
       <plugin filename="magnetometer_plugin.so" name="fcu_sim_magnetometer_plugin">
       <namespace>${namespace}</namespace>
-      <linkName>${namespace}/magnetometer_link</linkName>
+      <linkName>${parent_link}</linkName>
       <mag_topic>${mag_topic}</mag_topic>
       <noise_sigma>${noise_sigma}</noise_sigma>

File: fcu_sim_plugins/xacro/multirotor_forces_and_moments.xacro (robot description, xacro)
@@ -36,8 +36,5 @@
         alt_P="16.0"
         alt_I="5.0"
-        alt_D="32.0">
-        <inertia ixx="0.00001" ixy="0.0" ixz="0.0" iyy="0.00001" iyz="0.0" izz="0.00001" />
-        <origin xyz="0.0 0.0 0.0" rpy="0.0 0.0 0.0" />
-      </xacro:multirotor_forces_and_moments_macro>
+        alt_D="32.0"/>
     </xacro:macro>
     <xacro:macro
@@ -75,8 +72,5 @@
         alt_P="16.0"
         alt_I="5.0"
-        alt_D="32.0">
-        <inertia ixx="0.00001" ixy="0.0" ixz="0.0" iyy="0.00001" iyz="0.0" izz="0.00001" />
-        <origin xyz="0.0 0.0 0.0" rpy="0.0 0.0 0.0" />
-      </xacro:multirotor_forces_and_moments_macro>
+        alt_D="32.0"/>
     </xacro:macro>
   <!-- Macro to add a generic multirotor forces and moments plugin. -->
@@ -86,23 +80,9 @@
         mu max_l max_m max_n max_F tau_up_l tau_up_m tau_up_n tau_up_F tau_down_l tau_down_m
         tau_down_n tau_down_F roll_P roll_I roll_D pitch_P pitch_I pitch_D yaw_P yaw_I yaw_D alt_P
-        alt_I alt_D *inertia *origin">
-    <!-- link -->
-    <link name="${namespace}/multirotor_forces_and_moments_link">
-      <inertial>
-        <xacro:insert_block name="inertia" />
-        <mass value="0.001"/>
-      </inertial>
-    </link>
-    <!-- joint -->
-    <joint name="${namespace}/multirotor_forces_and_moments_joint" type="revolute">
-      <parent link="${parent_link}" />
-      <xacro:insert_block name="origin" />
-      <child link="${namespace}/multirotor_forces_and_moments_link" />
-      <limit upper="0" lower="0" effort="0" velocity="0" />
-    </joint>
+        alt_I alt_D">
     <!-- plugin -->
     <gazebo>
       <plugin filename="libmultirotor_forces_and_moments_plugin.so" name="multirotor_forces_and_moments">
-        <linkName>${namespace}/multirotor_forces_and_moments_link</linkName>
+        <linkName>${parent_link}</linkName>
         <namespace>${namespace}</namespace>
         <windSpeedTopic>${wind_speed_topic}</windSpeedTopic>

File: fcu_sim_plugins/xacro/odometry_sensor.xacro (robot description, xacro)
@@ -7,5 +7,4 @@
       <xacro:odometry_plugin_macro
         namespace="${namespace}/ground_truth"
-        odometry_sensor_suffix=""
         parent_link="${namespace}/base_link"
         pose_topic="pose"
@@ -15,5 +14,4 @@
         odometry_topic="odometry"
         parent_frame_id="world"
-        mass_odometry_sensor="0.00001"
         measurement_divisor="1"
         measurement_delay="0"
@@ -29,37 +27,20 @@
         enable_odometry_map="false"
         odometry_map=""
-        image_scale="">
-        <inertia ixx="0.00001" ixy="0.0" ixz="0.0" iyy="0.00001" iyz="0.0" izz="0.00001" />
-        <origin xyz="0.0 0.0 0.0" rpy="0.0 0.0 0.0" />
-      </xacro:odometry_plugin_macro>
+        image_scale=""/>
     </xacro:macro>
   <!-- Macro to add a generic odometry sensor. -->
   <xacro:macro name="odometry_plugin_macro"
     params="
-      namespace odometry_sensor_suffix parent_link pose_topic pose_with_covariance_topic
+      namespace parent_link pose_topic pose_with_covariance_topic
       position_topic transform_topic odometry_topic parent_frame_id
-      mass_odometry_sensor measurement_divisor measurement_delay unknown_delay
+      measurement_divisor measurement_delay unknown_delay
       noise_normal_position noise_normal_quaternion noise_normal_linear_velocity
       noise_normal_angular_velocity noise_uniform_position
       noise_uniform_quaternion noise_uniform_linear_velocity
       noise_uniform_angular_velocity enable_odometry_map odometry_map
-      image_scale *inertia *origin">
-    <!-- odometry link -->
-    <link name="${namespace}/odometry_sensor${odometry_sensor_suffix}_link">
-      <inertial>
-        <xacro:insert_block name="inertia" />
-        <mass value="${mass_odometry_sensor}" />  <!-- [kg] -->
-      </inertial>
-    </link>
-    <!-- odometry joint -->
-    <joint name="${namespace}/odometry_sensor${odometry_sensor_suffix}_joint" type="revolute">
-      <parent link="${parent_link}" />
-      <xacro:insert_block name="origin" />
-      <child link="${namespace}/odometry_sensor${odometry_sensor_suffix}_link" />
-      <limit upper="0" lower="0" effort="0" velocity="0" />
-    </joint>
+      image_scale">
     <gazebo>
-      <plugin filename="libodometry_plugin.so" name="odometry_sensor${odometry_sensor_suffix}">
-        <linkName>${namespace}/odometry_sensor${odometry_sensor_suffix}_link</linkName>
+      <plugin filename="libodometry_plugin.so" name="${namespace}_odometry_sensor">
+        <linkName>${parent_link}</linkName>
         <robotNamespace>${namespace}</robotNamespace>
         <poseTopic>${pose_topic}</poseTopic>

Commit message: added perfect_GPS option

File: fcu_sim_plugins/xacro/GPS.xacro (robot description, xacro)
@@ -2,7 +2,7 @@
 <robot xmlns:xacro="http://ros.org/wiki/xacro">
   <!-- Configure GPS -->
-    <xacro:macro
-      name="GPS_BYU"
-      params="namespace parent_link GPS_topic update_rate">
+  <xacro:macro
+	name="GPS_BYU"
+	params="namespace parent_link GPS_topic update_rate">
     <xacro:gps_plugin_macro
       namespace="${namespace}"
@@ -16,4 +16,26 @@
       east_k_GPS="0.00091"
       alt_k_GPS="0.00091"
+      sample_time="${1.0/update_rate}"
+      initial_latitude="40.267320"
+      initial_longitude="-111.635629"
+      initial_altitude="1491.0">
+      <inertia ixx="0.00001" ixy="0.0" ixz="0.0" iyy="0.00001" iyz="0.0" izz="0.00001" />
+      <origin xyz="0 0 0" rpy="0 0 0" />
+    </xacro:gps_plugin_macro>
+  </xacro:macro>
+  <xacro:macro
+	name="perfect_GPS"
+	params="namespace parent_link GPS_topic update_rate">
+    <xacro:gps_plugin_macro
+      namespace="${namespace}"
+      parent_link="${parent_link}"
+      gps_topic="${GPS_topic}"
+      mass_gps_sensor="0.001"
+      north_stdev="0.0"
+      east_stdev="0.0"
+      alt_stdev="0.0"
+      north_k_GPS="0.0"
+      east_k_GPS="0.0"
+      alt_k_GPS="0.0"
       sample_time="${1.0/update_rate}"
       initial_latitude="40.267320"

Commit message: added macro for Venus GPS, current values are not correct

File: fcu_sim_plugins/xacro/GPS.xacro (robot description, xacro)
@@ -24,4 +24,28 @@
     </xacro:gps_plugin_macro>
   </xacro:macro>
+  <!-- this GPS sensor needs correct values -->
+  <xacro:macro
+	name="Venus_GPS"
+	params="namespace parent_link GPS_topic update_rate">
+    <xacro:gps_plugin_macro
+      namespace="${namespace}"
+      parent_link="${parent_link}"
+      gps_topic="${GPS_topic}"
+      mass_gps_sensor="0.001"
+      north_stdev="0.021"
+      east_stdev="0.021"
+      alt_stdev="0.041"
+      north_k_GPS="0.00091"
+      east_k_GPS="0.00091"
+      alt_k_GPS="0.00091"
+      sample_time="${1.0/update_rate}"
+      initial_latitude="40.267320"
+      initial_longitude="-111.635629"
+      initial_altitude="1491.0">
+      <inertia ixx="0.00001" ixy="0.0" ixz="0.0" iyy="0.00001" iyz="0.0" izz="0.00001" />
+      <origin xyz="0 0 0" rpy="0 0 0" />
+    </xacro:gps_plugin_macro>
+  </xacro:macro>
+  <!-- GPS without noise -->
   <xacro:macro
 	name="perfect_GPS"
