Commit message: fixed imu and magnetometer xacros

File: fcu_sim_plugins/xacro/imu.xacro (robot description, xacro)
@@ -18,4 +18,6 @@
       accelerometer_turn_on_bias_sigma="0.0"
       perfect_imu="true">
+      <inertia ixx="0.00001" ixy="0.0" ixz="0.0" iyy="0.00001" iyz="0.0" izz="0.00001" />
+      <origin xyz="0 0 0" rpy="0 0 0" />
     </xacro:imu_plugin_macro>
   </xacro:macro>
@@ -36,4 +38,6 @@
       accelerometer_turn_on_bias_sigma="0.1960"
       perfect_imu="false">
+      <inertia ixx="0.00001" ixy="0.0" ixz="0.0" iyy="0.00001" iyz="0.0" izz="0.00001" />
+      <origin xyz="0 0 0" rpy="0 0 0" />
     </xacro:imu_plugin_macro>
   </xacro:macro>

File: fcu_sim_plugins/xacro/magnetometer.xacro (robot description, xacro)
@@ -14,4 +14,6 @@
       declination="${declination}"
       inclination="${inclination}">
+      <inertia ixx="0.00001" ixy="0.0" ixz="0.0" iyy="0.00001" iyz="0.0" izz="0.00001" />
+      <origin xyz="0 0 0" rpy="0 0 0" />
     </xacro:magnetometer_plugin_macro>
   </xacro:macro>
@@ -29,5 +31,5 @@
             *origin">
     <gazebo>
-      <plugin filename="magnetometer_plugin.so" name="fcu_sim_magnetometer_plugin">
+      <plugin filename="libmagnetometer_plugin.so" name="fcu_sim_magnetometer_plugin">
       <namespace>${namespace}</namespace>
       <linkName>${parent_link}</linkName>

Commit message: fixed imu plugin

File: fcu_sim_plugins/xacro/imu.xacro (robot description, xacro)
@@ -33,4 +33,19 @@
       acc_bias_walk_stdev="0.00001" />
   </xacro:macro>
+  <xacro:macro
+    name="IMU_MPU6050_multirotor_calibrated"
+    params="namespace parent_link imu_topic update_rate">
+  <xacro:imu_plugin_macro
+    namespace="${namespace}"
+    parent_link="${parent_link}"
+    update_rate="${update_rate}"
+    imu_topic="${imu_topic}"
+    gyro_stdev="0.13"
+    gyro_bias_range="0.00"
+    gyro_bias_walk_stdev="0.0001"
+    acc_stdev="1.15"
+    acc_bias_range="0.00"
+    acc_bias_walk_stdev="0.0001" />
+</xacro:macro>
     <!-- Macro to add an IMU. -->
   <xacro:macro name="imu_plugin_macro"
