Commit message: fixed a couple off bugs in forces and moments plugin

File: fcu_sim/urdf/junker/junker_base.xacro (robot description, xacro)
@@ -125,5 +125,5 @@
     <xacro:caster
       radius="0.05">
-      <origin xyz="-${body_length*0.5} 0 -${body_height*0.5}"/>
+      <origin xyz="-${body_length*0.5} 0 -${body_height*0.4}"/>
     </xacro:caster>
   </link>
@@ -133,5 +133,5 @@
     namespace="${namespace}"
     frame_rate="30"
-    rgb_range=""
+    rgb_range="1000"
     parent_link="${namespace}/base_link"
     image_topic="chase/rgb"
@@ -224,9 +224,16 @@
     </plugin>
   </gazebo>
-  <!-- Odometry Sensor -->
+  <gazebo>
+    <plugin filename="libfcu_sim_aircraft_truth_plugin.so" name="aircraft_truth_plugin">
+      <namespace>${namespace}</namespace>
+      <linkName>${namespace}/base_link</linkName>
+      <windSpeedTopic>${wind_speed_topic}</windSpeedTopic>
+    </plugin>
+  </gazebo>
+  <!-- Odometry Sensor
   <xacro:include filename="$(find fcu_sim_plugins)/xacro/odometry_sensor.xacro"/>
   <xacro:ground_truth
     namespace="${namespace}"
     parent_link="${namespace}/base_link">
-  </xacro:ground_truth>
+  </xacro:ground_truth> -->
 </robot>

Commit message: controller launch files, everything is setup for the controller, it just isn't tunned very good

File: fcu_sim/urdf/junker/junker_base.xacro (robot description, xacro)
@@ -10,21 +10,21 @@
   <xacro:property name="body_height" value="1.0" />
   <xacro:property name="body_length" value="1.6"/>
-  <xacro:property name="mass" value="13.5"/>
-  <xacro:property name="Jx" value="0.8244"/>
-  <xacro:property name="Jy" value="1.135"/>
-  <xacro:property name="Jz" value="1.759"/>
-  <xacro:property name="Jxz" value=".1204"/>
+  <xacro:property name="mass" value="1.5"/>
+  <xacro:property name="Jx" value="0.1147"/>
+  <xacro:property name="Jy" value="0.0576"/>
+  <xacro:property name="Jz" value="0.1712"/>
+  <xacro:property name="Jxz" value="0.0015"/>
   <xacro:property name="rho" value="1.2682"/>
-  <xacro:property name="wing_s" value="0.55"/>
-  <xacro:property name="wing_b" value="2.8956"/>
-  <xacro:property name="wing_c" value="0.18994"/>
+  <xacro:property name="wing_s" value="0.2589"/>
+  <xacro:property name="wing_b" value="1.4224"/>
+  <xacro:property name="wing_c" value="0.3302"/>
   <xacro:property name="wing_M" value="0.55"/>
   <xacro:property name="wing_epsilon" value="2.8956"/>
   <xacro:property name="wing_alpha0" value="0.18994"/>
-  <xacro:property name="k_motor" value="80.0"/>
+  <xacro:property name="k_motor" value="40.0"/>
   <xacro:property name="k_T_P" value="0.0"/>
   <xacro:property name="k_Omega" value="0.0"/>
   <xacro:property name="prop_e" value="0.9"/>
-  <xacro:property name="prop_S" value="0.202"/>
+  <xacro:property name="prop_S" value="0.0314"/>
   <xacro:property name="prop_C" value="1.0"/>
   <xacro:property name="C_L_O" value="0.28"/>
@@ -38,5 +38,5 @@
   <xacro:property name="C_L_delta_r" value="0.0"/>
   <xacro:property name="C_D_O" value="0.03"/>
-  <xacro:property name="C_D_alpha" value="0.30"/>
+  <xacro:property name="C_D_alpha" value="0.2108"/>
   <xacro:property name="C_D_beta" value="0.0"/>
   <xacro:property name="C_D_p" value="0.0437"/>
@@ -55,5 +55,5 @@
   <xacro:property name="C_ell_delta_e" value="0.0"/>
   <xacro:property name="C_ell_delta_r" value="0.105"/>
-  <xacro:property name="C_m_O" value="-0.02338"/>
+  <xacro:property name="C_m_O" value="0.0"/>
   <xacro:property name="C_m_alpha" value="-0.38"/>
   <xacro:property name="C_m_beta" value="0.0"/>
@@ -81,5 +81,5 @@
   <xacro:property name="C_Y_delta_a" value="0.0"/>
   <xacro:property name="C_Y_delta_e" value="0.0"/>
-  <xacro:property name="C_Y_delta_r" value="-0.017"/>
+  <xacro:property name="C_Y_delta_r" value="-0.17"/>
   <!-- Property Blocks -->
   <xacro:property name="inertia">

Commit message: added airspeed, barometer, MPU6050 and GPS plugins

File: fcu_sim/urdf/junker/junker_base.xacro (robot description, xacro)
@@ -224,4 +224,5 @@
     </plugin>
   </gazebo>
+  <!-- Sensors -->
   <gazebo>
     <plugin filename="libfcu_sim_aircraft_truth_plugin.so" name="aircraft_truth_plugin">
@@ -231,9 +232,36 @@
     </plugin>
   </gazebo>
-  <!-- Odometry Sensor
-  <xacro:include filename="$(find fcu_sim_plugins)/xacro/odometry_sensor.xacro"/>
-  <xacro:ground_truth
-    namespace="${namespace}"
-    parent_link="${namespace}/base_link">
-  </xacro:ground_truth> -->
+  <!-- Airspeed -->
+  <xacro:include filename="$(find fcu_sim_plugins)/xacro/airspeed.xacro"/>
+  <xacro:airspeed_MPXV5004G
+    namespace="${namespace}"
+    parent_link="${namespace}/base_link"
+    airspeed_topic="airspeed/data">
+  </xacro:airspeed_MPXV5004G>
+  <!-- GPS -->
+  <xacro:include filename="$(find fcu_sim_plugins)/xacro/GPS.xacro"/>
+  <xacro:GPS_BYU
+    namespace="${namespace}"
+    parent_link="${namespace}/base_link"
+    GPS_topic="gps/data">
+  </xacro:GPS_BYU>
+  <!-- Sonar and Barometer -->
+  <xacro:include filename="$(find fcu_sim_plugins)/xacro/altimeter.xacro"/>
+  <xacro:Sonar_HC-SR04
+    namespace="${namespace}"
+    parent_link="${namespace}/base_link"
+    altimeter_topic="sonar/data">
+  </xacro:Sonar_HC-SR04>
+  <xacro:Barometer_MS5611
+    namespace="${namespace}"
+    parent_link="${namespace}/base_link"
+    altimeter_topic="baro/data">
+  </xacro:Barometer_MS5611>
+  <!-- IMU -->
+  <xacro:include filename="$(find fcu_sim_plugins)/xacro/imu.xacro"/>
+  <xacro:IMU_MPU6050
+    namespace="${namespace}"
+    parent_link="${namespace}/base_link"
+    imu_topic="imu/data">
+  </xacro:IMU_MPU6050>
 </robot>

File: fcu_sim_plugins/xacro/altimeter.xacro (robot description, xacro)
@@ -2,4 +2,44 @@
 <robot xmlns:xacro="http://ros.org/wiki/xacro">
   <xacro:property name="pi" value="3.14159265359" />
+  <!-- Sonar  HC-SR04 -->
+  <xacro:macro
+    name="Sonar_HC-SR04"
+    params="namespace parent_link altimeter_topic">
+    <xacro:altimeter_plugin_macro
+      namespace="${namespace}"
+      altimeter_suffix="sonar"
+      parent_link="${parent_link}"
+      altimeter_topic="${altimeter_topic}"
+      mass_altimeter_sensor="0.0043"
+      altimeter_min_range="0.2"
+      altimeter_max_range="4.0"
+      altimeter_error_stdev="0.2"
+      altimeter_field_of_view="0.2618"
+      altimeter_publish_rate="20"
+      altimeter_noise_on="true" >
+      <inertia ixx="0.00001" ixy="0.0" ixz="0.0" iyy="0.00001" iyz="0.0" izz="0.00001" />
+      <origin xyz="0 0 0" rpy="0 0 0" />
+    </xacro:altimeter_plugin_macro>
+  </xacro:macro>
+  <!-- Barometer  MS5611-->
+  <xacro:macro
+    name="Barometer_MS5611"
+    params="namespace parent_link altimeter_topic">
+    <xacro:altimeter_plugin_macro
+      namespace="${namespace}"
+      altimeter_suffix="baro"
+      parent_link="${parent_link}"
+      altimeter_topic="${altimeter_topic}"
+      mass_altimeter_sensor="0.0043"
+      altimeter_min_range="-10000.0"
+      altimeter_max_range="10000.0"
+      altimeter_error_stdev="8.0"
+      altimeter_field_of_view="0.0"
+      altimeter_publish_rate="20"
+      altimeter_noise_on="true" >
+      <inertia ixx="0.00001" ixy="0.0" ixz="0.0" iyy="0.00001" iyz="0.0" izz="0.00001" />
+      <origin xyz="0 0 0" rpy="0 0 0" />
+    </xacro:altimeter_plugin_macro>
+  </xacro:macro>
   <!-- LV-MaxSonar-EZ3 MB1030 -->
   <xacro:macro

File: fcu_sim_plugins/xacro/imu.xacro (robot description, xacro)
@@ -6,5 +6,4 @@
       name="IMU_ADIS16448"
       params="namespace parent_link imu_topic">
-    <!-- ADIS16448 IMU. -->
     <xacro:imu_plugin_macro
       namespace="${namespace}"
@@ -18,4 +17,26 @@
       gyroscope_turn_on_bias_sigma="0.0087"
       accelerometer_noise_density="0.004"
+      accelerometer_random_walk="0.006"
+      accelerometer_bias_correlation_time="300.0"
+      accelerometer_turn_on_bias_sigma="0.1960">
+      <inertia ixx="0.00001" ixy="0.0" ixz="0.0" iyy="0.00001" iyz="0.0" izz="0.00001" />
+      <origin xyz="0 0 0" rpy="0 0 0" />
+    </xacro:imu_plugin_macro>
+  </xacro:macro>
+  <!-- Configure IMU -->
+    <xacro:macro
+      name="IMU_MPU6050"
+      params="namespace parent_link imu_topic">
+    <xacro:imu_plugin_macro
+      namespace="${namespace}"
+      imu_suffix=""
+      parent_link="${parent_link}"
+      imu_topic="${imu_topic}"
+      mass_imu_sensor="0.015"
+      gyroscope_noise_density="0.0008726646"
+      gyroscopoe_random_walk="0.000038785"
+      gyroscope_bias_correlation_time="1000.0"
+      gyroscope_turn_on_bias_sigma="0.0087"
+      accelerometer_noise_density="0.008"
       accelerometer_random_walk="0.006"
       accelerometer_bias_correlation_time="300.0"

Commit message: fcu changes

File: fcu_sim/urdf/junker/junker_base.xacro (robot description, xacro)
@@ -6,5 +6,5 @@
   <xacro:property name="command_topic" value="/command"/>
   <xacro:property name="use_mesh_file" value="true" />
-  <xacro:property name="mesh_file" value="package://fcu_sim/meshes/ju-87.dae"/>
+  <xacro:property name="mesh_file" value="package://fcu_sim/meshes/c130.dae"/>
   <xacro:property name="body_width" value="1.4"/>
   <xacro:property name="body_height" value="1.0" />
@@ -98,8 +98,8 @@
     </inertial>
     <visual name="plane_visual">
-      <origin xyz="0 0 0" rpy="1.570796 0 1.570796" />
+      <origin xyz="0 0 -1" rpy="0 0 1.570796" />
       <geometry>
         <xacro:if value="${use_mesh_file}">
-          <mesh filename="${mesh_file}" scale="0.002 0.002 0.002" />
+          <mesh filename="${mesh_file}" scale="0.1 0.1 0.1" />
         </xacro:if>
         <xacro:unless value="${use_mesh_file}">
@@ -141,5 +141,5 @@
   <!-- Color -->
   <gazebo reference="${namespace}/base_link">
-    <material>Gazebo/Red</material>
+    <material>Gazebo/Blue</material>
   </gazebo>
   <!-- Add Aerodynamics -->

File: fcu_sim_plugins/xacro/rgbd.xacro (robot description, xacro)
@@ -14,9 +14,9 @@
       depth_range="6.5"
       rgb_range=""
-      image_topic="/camera/rgb/image_raw"
-      depth_topic="/camera/depth/image_raw"
-      image_camera_info_topic="/camera/rgb/camera_info"
-      depth_camera_info_topic="/camera/depth/camera_info"
-      pointcloud_topic="/camera/pointcloud">
+      image_topic="${namespace}/camera/rgb/image_raw"
+      depth_topic="${namespace}/camera/depth/image_raw"
+      image_camera_info_topic="${namespace}/camera/rgb/camera_info"
+      depth_camera_info_topic="${namespace}/camera/depth/camera_info"
+      pointcloud_topic="${namespace}/camera/pointcloud">
       <origin xyz="0.127 0 -0.0889" rpy="0 0 0" /> <!-- for shredder -->
     </xacro:depth_camera>
@@ -38,14 +38,14 @@
             *origin">
     <link name="${namespace}/camera_link">
-      <collision>
+      <!-- <collision>
         <xacro:insert_block name="origin" />
         <geometry>
           <cylinder length="0.01" radius="0.007" />
         </geometry>
-      </collision>
+      </collision> -->
       <inertial>
-        <mass value="1e-4" />
+        <mass value="1e-3" />
         <origin xyz="0 0 0" rpy="0 0 0" />
-        <inertia ixx="1e-4" ixy="0" ixz="0" iyy="1e-4" iyz="0" izz="1e-4" />
+        <inertia ixx="1e-3" ixy="0" ixz="0" iyy="1e-3" iyz="0" izz="1e-3" />
       </inertial>
     </link>

File: fcu_sim_plugins/xacro/rotor.xacro (robot description, xacro)
@@ -76,5 +76,5 @@
         <motorConstant>${motor_constant}</motorConstant>
         <momentConstant>${moment_constant}</momentConstant>
-        <commandSubTopic>gazebo/command/motor_speed</commandSubTopic>
+        <commandSubTopic>command/motor_speed</commandSubTopic>
         <motorNumber>${motor_number}</motorNumber>
         <rotorDragCoefficient>${rotor_drag_coefficient}</rotorDragCoefficient>
