Commit message: gimbal working

File: fcu_sim/urdf/junker/junker_base.xacro (robot description, xacro)
@@ -98,8 +98,8 @@
     </inertial>
     <visual name="plane_visual">
-      <origin xyz="0 0 -1" rpy="0 0 1.570796" />
+      <origin xyz=".5 0 -.5" rpy="0 0 -1.570796" />
       <geometry>
         <xacro:if value="${use_mesh_file}">
-          <mesh filename="${mesh_file}" scale="0.1 0.1 0.1" />
+          <mesh filename="${mesh_file}" scale="0.01 0.01 0.01" />
         </xacro:if>
         <xacro:unless value="${use_mesh_file}">
@@ -131,10 +131,10 @@
   <xacro:include filename="$(find fcu_sim_plugins)/xacro/camera.xacro"/>
   <xacro:simple_camera
-    namespace="${namespace}"
+    namespace="${namespace}/chase"
     frame_rate="30"
     rgb_range="1000"
     parent_link="${namespace}/base_link"
-    image_topic="chase/rgb"
-    image_camera_info_topic="chase/camera_info">
+    image_topic="rgb"
+    image_camera_info_topic="camera_info">
     <origin xyz="-${1.1*body_length} 0 ${0.8*body_height}"/>
   </xacro:simple_camera>
@@ -232,4 +232,14 @@
     </plugin>
   </gazebo>
+  <!-- Gimbal -->
+  <xacro:include filename="$(find fcu_sim_plugins)/xacro/gimbal.xacro"/>
+  <xacro:gimbal_ZENMUSE
+    namespace="${namespace}"
+    parent_link="${namespace}/base_link"
+    camera_topic="rgb"
+    pose_topic="${namespace}/gimbal/pose"
+    command_topic="${namespace}/gimbal/control">
+    <origin xyz="0 0 1" ryp="0 0 0"/>
+  </xacro:gimbal_ZENMUSE>
   <!-- Airspeed -->
   <xacro:include filename="$(find fcu_sim_plugins)/xacro/airspeed.xacro"/>

File: fcu_sim_plugins/xacro/camera.xacro (robot description, xacro)
@@ -14,5 +14,5 @@
             parent_link
             *origin">
-    <link name="${namespace}/chase_camera_base_link">
+    <link name="${namespace}/camera_base_link">
       <inertial>
         <mass value="0.001"/>
@@ -20,5 +20,5 @@
         <xacro:insert_block name="empty_inertia"/>
       </inertial>
-      <visual name="chase_camera_visual">
+      <visual name="${namespace}/camera_visual">
         <xacro:insert_block name="origin"/>
         <geometry>
@@ -27,11 +27,11 @@
       </visual>
     </link>
-    <joint name="${namespace}/chase_camera_joint" type="fixed">
+    <joint name="${namespace}/camera_joint" type="fixed">
       <xacro:insert_block name="origin"/>
       <parent link="${parent_link}"/>
-      <child link="${namespace}/chase_camera_base_link"/>
+      <child link="${namespace}/camera_base_link"/>
       <limit upper="0" lower="0" effort="0" velocity="0"/>
     </joint>
-    <gazebo reference="${namespace}/chase_camera_base_link">
+    <gazebo reference="${namespace}/camera_base_link">
       <sensor type="camera" name="${namespace}/camera">
         <always_on>true</always_on>

File: fcu_sim_plugins/xacro/gimbal.xacro (robot description, xacro)
@@ -1,19 +1,18 @@
 <?xml version="1.0"?>
 <robot xmlns:xacro="http://ros.org/wiki/xacro">
-  <xacro:property name="pi" value="3.14159265359" />
-    <!-- Configure Airspeed -->
+    <!-- Configure ZENMUSE Gimbal -->
     <xacro:macro
       name="gimbal_ZENMUSE"
-      params="namespace parent_link camera_topic pose_topic control_topic *origin">
+      params="namespace parent_link camera_topic pose_topic command_topic *origin">
     <xacro:gimbal_plugin_macro
       namespace="${namespace}"
       parent_link="${parent_link}"
       camera_topic="${camera_topic}"
-      pose_topic="${camera_topic}"
-      control_topic="${camera_topic}"
+      pose_topic="${pose_topic}"
+      command_topic="${command_topic}"
       mass="0.001"
-      x_rotation_range="4"
-      y_rotation_range="4"
-      z_rotation_range="100000000000000"
+      x_rotation_range="1000000000"
+      y_rotation_range="0000000000"
+      z_rotation_range="1000000000"
       time_constant="0.25">
       <inertia ixx="0.00001" ixy="0.0" ixz="0.0" iyy="0.00001" iyz="0.0" izz="0.00001" />
@@ -22,8 +21,34 @@
   </xacro:macro>
     <!-- Macro to add a Gimbal -->
-  <xacro:macro name="gimbal_plugin_macro"
-    params="namespace parent_link camera_topic pose_topic control_topic
+  <xacro:macro
+    name="gimbal_plugin_macro"
+    params="namespace parent_link camera_topic pose_topic command_topic
       mass x_rotation_range y_rotation_range z_rotation_range time_constant
       *inertia *origin">
+    <!-- Base Link  -->
+    <link name="${namespace}/gimbal/base_link">
+      <inertial>
+        <inertia ixx="0.00001" ixy="0.0" ixz="0.0" iyy="0.00001" iyz="0.0" izz="0.00001" />
+        <mass value="${mass}" />
+        <xacro:insert_block name="origin" />
+      </inertial>
+      <visual name="${namespace}/gimbal_base_visual">
+        <!-- <xacro:insert_block name="origin"/> -->
+        <origin xyz="0 0 0" rpy = "0 0 0"/>
+        <geometry>
+          <box size="0.1 0.1 0.1"/>
+        </geometry>
+      </visual>
+    </link>
+    <gazebo reference="${namespace}/gimbal/base_link">
+      <material>Gazebo/Blue</material>
+    </gazebo>
+    <!-- Base Joint -->
+    <joint name="${namespace}/gimbal_base_joint" type="revolute">
+      <xacro:insert_block name="origin" />
+      <parent link="${parent_link}" />
+      <child link="${namespace}/gimbal/base_link" />
+      <limit upper="0" lower="0" effort="0" velocity="0"/>
+    </joint>
     <!-- Yaw Link -->
     <link name="${namespace}/gimbal/yaw_link">
@@ -31,16 +56,22 @@
         <inertia ixx="0.00001" ixy="0.0" ixz="0.0" iyy="0.00001" iyz="0.0" izz="0.00001" />
         <mass value="0.0001" />
-        <xacro:insert_block name="origin" />
+        <origin xyz="0 0 0" rpy = "0 0 0"/>
       </inertial>
+      <visual name="${namespace}/gimbal_yaw_visual">
+        <origin xyz="0 0 0" rpy = "0 0 0"/>
+        <geometry>
+          <box size="0.1 0.1 0.1"/>
+        </geometry>
+      </visual>
     </link>
+    <gazebo reference="${namespace}/gimbal/yaw_link">
+      <material>Gazebo/Red</material>
+    </gazebo>
     <!-- Yaw joint -->
     <joint name="${namespace}/gimbal_yaw_joint" type="revolute">
-      <xacro:insert_block name="origin" />
-      <parent link="${parent_link}" />
+      <pose xyz="0 0 0" rpy = "0 0 0"/>
+      <parent link="${namespace}/gimbal/base_link" />
       <child link="${namespace}/gimbal/yaw_link" />
-      <axis>
-        <xyz> 0 0 1</xyz>
-      </axis>
-      <limit upper="${z_rotation_range}" lower="-${z_rotation_range}" effort="1000" velocity="5000"/>
+      <limit upper="${z_rotation_range}" lower="${-1.0*z_rotation_range}" effort="1000" velocity="5000"/>
     </joint>
     <!-- Roll Link -->
@@ -49,46 +80,80 @@
         <inertia ixx="0.00001" ixy="0.0" ixz="0.0" iyy="0.00001" iyz="0.0" izz="0.00001" />
         <mass value="0.0001" />
-        <xacro:insert_block name="origin" />
+        <origin xyz="0 0 0" rpy = "0 0 0"/>
       </inertial>
+      <visual name="${namespace}/gimbal_roll_visual">
+        <origin xyz="0 0 0" rpy = "0 0 0"/>
+        <geometry>
+          <box size="0.1 0.1 0.1"/>
+        </geometry>
+      </visual>
     </link>
+    <gazebo reference="${namespace}/gimbal/roll_link">
+      <material>Gazebo/Green</material>
+    </gazebo>
     <!-- Roll joint -->
     <joint name="${namespace}/gimbal_roll_joint" type="revolute">
-      <xacro:insert_block name="origin" />
+      <origin xyz="0 0 0" rpy = "0 0 0"/>
       <parent link="${namespace}/gimbal/yaw_link" />
       <child link="${namespace}/gimbal/roll_link" />
-      <axis>
-        <xyz> 1 0 0</xyz>
-      </axis>
-      <limit upper="${x_rotation_range}" lower="-${x_rotation_range}" effort="1000" velocity="5000"/>
+      <limit upper="${x_rotation_range}" lower="${-1.0*x_rotation_range}" effort="1000" velocity="5000"/>
     </joint>
     <!-- Pitch Link -->
     <link name="${namespace}/gimbal/pitch_link">
       <inertial>
-        <xacro:insert_block name="inertia" />
-        <mass value="${mass}" />
-        <xacro:insert_block name="origin" />
+        <inertia ixx="0.00001" ixy="0.0" ixz="0.0" iyy="0.00001" iyz="0.0" izz="0.00001" />
+        <mass value="0.0001" />
+        <origin xyz="0 0 0" rpy = "0 0 0"/>
       </inertial>
+      <visual name="${namespace}/gimbal_pitch_visual">
+        <origin xyz="0 0 0" rpy = "0 0 0"/>
+        <geometry>
+          <box size="0.1 0.1 0.1"/>
+        </geometry>
+      </visual>
     </link>
+    <gazebo reference="${namespace}/gimbal/pitch_link">
+      <material>Gazebo/Yellow</material>
+    </gazebo>
     <!-- Pitch joint -->
     <joint name="${namespace}/gimbal_pitch_joint" type="revolute">
-      <xacro:insert_block name="origin" />
-      <parent link="${namespace}/gimbal/yaw_link" />
+      <origin xyz="0 0 0" rpy = "0 0 0"/>
+      <parent link="${namespace}/gimbal/roll_link" />
       <child link="${namespace}/gimbal/pitch_link" />
-      <axis>
-        <xyz> 0 1 0</xyz>
-      </axis>
-      <limit upper="${y_rotation_range}" lower="-${y_rotation_range}" effort="1000" velocity="5000"/>
+      <limit upper="${x_rotation_range}" lower="${-1.0*x_rotation_range}" effort="1000" velocity="5000"/>
     </joint>
     <!-- Attach a Camera -->
-    <xacro:include filename="$(find fcu_sim_plugins)/xacro/camera.xacro"/>
-    <xacro:simple_camera
-      namespace="${namespace}"
-      frame_rate="30"
-      rgb_range="10000"
-      image_topic="${camera_topic}"
-      image_camera_info_topic="${camera_topic}/camera_info"
-      parent_link="${namespace}/gimbal/pitch_link">
-      <xacro:insert_block name="origin"/>
-    </xacro>
+    <gazebo reference="${namespace}/gimbal/pitch_link">
+      <sensor type="camera" name="gimbal/camera">
+        <always_on>true</always_on>
+        <update_rate>30</update_rate>
+        <camera>
+          <horizontal_fov>2</horizontal_fov>
+          <image>
+            <format>R8G8B8</format>
+            <width>640</width>
+            <height>480</height>
+          </image>
+          <clip>
+            <near>0.01</near>
+            <far>1000</far>
+          </clip>
+        </camera>
+        <plugin name="${namespace}/gimbal_camera" filename="libgazebo_ros_camera.so">
+          <robotNamespace>${namespace}</robotNamespace>
+          <alwaysOn>true</alwaysOn>
+          <updateRate>30</updateRate>
+          <cameraName>gimbal/camera</cameraName>
+          <imageTopicName>${camera_topic}</imageTopicName>
+          <cameraInfoTopicName>${camera_topic}/camera_info</cameraInfoTopicName>
+          <frameName>gimbal_camera</frameName>
+          <distortionK1>0.0</distortionK1>
+          <distortionK2>0.0</distortionK2>
+          <distortionK3>0.0</distortionK3>
+          <distortionT1>0.0</distortionT1>
+          <distortionT2>0.0</distortionT2>
+        </plugin>
+      </sensor>
+    </gazebo>
     <!-- Load Gimbal Controller Plugin -->
     <gazebo>
@@ -96,11 +161,9 @@
         <namespace>${namespace}</namespace>
         <yawJoint>${namespace}/gimbal_yaw_joint</yawJoint>
-        <pitchJoint>${namespace}/gimbal_roll_joint</pitchJoint>
-        <rollJoint>${namespace}/gimbal_pitch_joint</rollJoint>
+        <pitchJoint>${namespace}/gimbal_pitch_joint</pitchJoint>
+        <rollJoint>${namespace}/gimbal_roll_joint</rollJoint>
         <timeConstant>${time_constant}</timeConstant>
-        <pressureNoiseSigma>${pressure_noise_sigma}</pressureNoiseSigma> <!-- [Pascals] -->
-        <airDensity>${air_density}</airDensity> <!-- [kg/m^3] -->
-        <maxPressure>${max_pressure}</maxPressure> <!-- [Pascals] -->
-        <minPressure>${min_pressure}</minPressure> <!-- [Pascals] -->
+        <commandTopic>${command_topic}</commandTopic>
+        <poseTopic>${pose_topic}</poseTopic>
       </plugin>
     </gazebo>

Commit message: cleaned up gimbal files, tested and working in sim

File: fcu_sim/urdf/junker/junker_base.xacro (robot description, xacro)
@@ -101,5 +101,5 @@
       <geometry>
         <xacro:if value="${use_mesh_file}">
-          <mesh filename="${mesh_file}" scale="0.01 0.01 0.01" />
+          <mesh filename="${mesh_file}" scale="0.25 0.25 0.25" />
         </xacro:if>
         <xacro:unless value="${use_mesh_file}">
@@ -240,5 +240,5 @@
     pose_topic="${namespace}/gimbal/pose"
     command_topic="${namespace}/gimbal/control">
-    <origin xyz="0 0 1" ryp="0 0 0"/>
+    <origin xyz="2 0 0" ryp="0 0 0"/>
   </xacro:gimbal_ZENMUSE>
   <!-- Airspeed -->

File: fcu_sim_plugins/xacro/gimbal.xacro (robot description, xacro)
@@ -33,15 +33,5 @@
         <xacro:insert_block name="origin" />
       </inertial>
-      <visual name="${namespace}/gimbal_base_visual">
-        <!-- <xacro:insert_block name="origin"/> -->
-        <origin xyz="0 0 0" rpy = "0 0 0"/>
-        <geometry>
-          <box size="0.1 0.1 0.1"/>
-        </geometry>
-      </visual>
     </link>
-    <gazebo reference="${namespace}/gimbal/base_link">
-      <material>Gazebo/Blue</material>
-    </gazebo>
     <!-- Base Joint -->
     <joint name="${namespace}/gimbal_base_joint" type="revolute">
@@ -58,14 +48,5 @@
         <origin xyz="0 0 0" rpy = "0 0 0"/>
       </inertial>
-      <visual name="${namespace}/gimbal_yaw_visual">
-        <origin xyz="0 0 0" rpy = "0 0 0"/>
-        <geometry>
-          <box size="0.1 0.1 0.1"/>
-        </geometry>
-      </visual>
     </link>
-    <gazebo reference="${namespace}/gimbal/yaw_link">
-      <material>Gazebo/Red</material>
-    </gazebo>
     <!-- Yaw joint -->
     <joint name="${namespace}/gimbal_yaw_joint" type="revolute">
@@ -82,14 +63,5 @@
         <origin xyz="0 0 0" rpy = "0 0 0"/>
       </inertial>
-      <visual name="${namespace}/gimbal_roll_visual">
-        <origin xyz="0 0 0" rpy = "0 0 0"/>
-        <geometry>
-          <box size="0.1 0.1 0.1"/>
-        </geometry>
-      </visual>
     </link>
-    <gazebo reference="${namespace}/gimbal/roll_link">
-      <material>Gazebo/Green</material>
-    </gazebo>
     <!-- Roll joint -->
     <joint name="${namespace}/gimbal_roll_joint" type="revolute">
@@ -106,14 +78,5 @@
         <origin xyz="0 0 0" rpy = "0 0 0"/>
       </inertial>
-      <visual name="${namespace}/gimbal_pitch_visual">
-        <origin xyz="0 0 0" rpy = "0 0 0"/>
-        <geometry>
-          <box size="0.1 0.1 0.1"/>
-        </geometry>
-      </visual>
     </link>
-    <gazebo reference="${namespace}/gimbal/pitch_link">
-      <material>Gazebo/Yellow</material>
-    </gazebo>
     <!-- Pitch joint -->
     <joint name="${namespace}/gimbal_pitch_joint" type="revolute">

Commit message: fixed the fixedwing launch file and xacro so they are working

File: fcu_sim/urdf/junker/junker_base.xacro (robot description, xacro)
@@ -6,5 +6,5 @@
   <xacro:property name="command_topic" value="/command"/>
   <xacro:property name="use_mesh_file" value="true" />
-  <xacro:property name="mesh_file" value="package://fcu_sim/meshes/c130.dae"/>
+  <xacro:property name="mesh_file" value="package://fcu_sim/meshes/ju-87.dae"/>
   <xacro:property name="body_width" value="1.4"/>
   <xacro:property name="body_height" value="1.0" />
@@ -98,8 +98,8 @@
     </inertial>
     <visual name="plane_visual">
-      <origin xyz=".5 0 -.5" rpy="0 0 -1.570796" />
+      <origin xyz="0 0 0" rpy="1.570796 0 1.570796" />
       <geometry>
         <xacro:if value="${use_mesh_file}">
-          <mesh filename="${mesh_file}" scale="0.25 0.25 0.25" />
+          <mesh filename="${mesh_file}" scale="0.002 0.002 0.002" />
         </xacro:if>
         <xacro:unless value="${use_mesh_file}">

Commit message: added velodyne and world for reactive planner testing

File: fcu_sim/urdf/junker/junker_base.xacro (robot description, xacro)
@@ -240,5 +240,5 @@
     pose_topic="${namespace}/gimbal/pose"
     command_topic="${namespace}/gimbal/control">
-    <origin xyz="2 0 0" ryp="0 0 0"/>
+    <origin xyz="2 0 0" rpy="0 0 0"/>
   </xacro:gimbal_ZENMUSE>
   <!-- Airspeed -->

File: fcu_sim/urdf/shredder/shredder_base.xacro (robot description, xacro)
@@ -8,5 +8,5 @@
 <xacro:property name="namespace" value="shredder" />
 <xacro:property name="use_mesh_file" value="true" />
-<xacro:property name="mesh_file" value="package://fcu_sim/meshes/firefly.dae" />
+<xacro:property name="mesh_file" value="package://fcu_sim/meshes/Millennium_Falcon.dae" />
 <xacro:property name="mass" value="3.81" /> <!-- [kg] -->
 <xacro:property name="body_width" value="0.505" /> <!-- [m] -->
@@ -24,8 +24,9 @@
   </inertial>
   <visual>
-    <origin xyz="0 0 0" rpy="0 0 0" />
+    <origin xyz="0 0 0" rpy="0 0 1.571" />
     <geometry>
       <xacro:if value="${use_mesh_file}">
-        <mesh filename="${mesh_file}" scale="1 1 1" />
+        <mesh filename="${mesh_file}" scale="0.001 0.001 0.001" />
+        <!-- <mesh filename="${mesh_file}" scale="1 1 1" /> -->
       </xacro:if>
       <xacro:unless value="${use_mesh_file}">
@@ -77,11 +78,13 @@
   <xacro:xtion
     namespace="${namespace}"
-    parent_link="${namespace}/base_link"/> -->
+    parent_link="${namespace}/bavese_link"/> -->
   <!-- Laser Scanner -->
-  <!-- <xacro:include filename="$(find fcu_sim_plugins)/xacro/velodyne.xacro"/>
+  <xacro:include filename="$(find fcu_sim_plugins)/xacro/velodyne.xacro"/>
   <xacro:velodyne_custom
     namespace="${namespace}"
     parent_link="${namespace}/base_link"
-    visualize="false"/> -->
+    visualize="false">
+    <origin xyz="${body_width+0.1} 0 0" rpy="0 0 0"/>
+  </xacro:velodyne_custom>
   <!-- GPS -->
   <xacro:include filename="$(find fcu_sim_plugins)/xacro/GPS.xacro"/>
@@ -90,3 +93,14 @@
     parent_link="${namespace}/base_link"
     GPS_topic="gps"/>
+  <!-- Camera -->
+  <xacro:include filename="$(find fcu_sim_plugins)/xacro/camera.xacro"/>
+  <xacro:simple_camera
+    namespace="${namespace}"
+    frame_rate="30"
+    rgb_range="1000"
+    parent_link="${namespace}/base_link"
+    image_topic="rgb"
+    image_camera_info_topic="camera_info">
+    <origin xyz="${body_width+0.1} 0 0" rpy="0 0 0"/>
+  </xacro:simple_camera>
 </robot>

File: fcu_sim_plugins/xacro/gimbal.xacro (robot description, xacro)
@@ -4,5 +4,10 @@
     <xacro:macro
       name="gimbal_ZENMUSE"
-      params="namespace parent_link camera_topic pose_topic command_topic *origin">
+      params="namespace
+              parent_link
+              camera_topic
+              pose_topic
+              command_topic
+              *origin">
     <xacro:gimbal_plugin_macro
       namespace="${namespace}"
@@ -13,5 +18,5 @@
       mass="0.001"
       x_rotation_range="1000000000"
-      y_rotation_range="0000000000"
+      y_rotation_range="1000000000"
       z_rotation_range="1000000000"
       time_constant="0.25">

File: fcu_sim_plugins/xacro/multirotor_forces_and_moments.xacro (robot description, xacro)
@@ -13,5 +13,5 @@
         parent_frame_id="${parent_link}"
         mass="3.81"
-        mu="1"
+        mu="0.01"
         max_l="12.542"
         max_m="12.542"

File: fcu_sim_plugins/xacro/velodyne.xacro (robot description, xacro)
@@ -2,37 +2,39 @@
 <robot xmlns:xacro="http://ros.org/wiki/xacro">
   <xacro:property name="pi" value="3.14159265359" />
-  <!-- Hokuyo UTM-30LX-->
   <xacro:macro
     name="velodyne_custom"
     params="namespace
             parent_link
-            visualize">
+            visualize
+            *origin">
     <xacro:laser_scanner
       namespace="${namespace}"
       parent_link="${parent_link}"
-      num_samples="720"
       visualize="${visualize}"
       min_range="0.1"
-      max_range="10"
-      res_range="0.03"
-      min_angle="-pi/2"
-      max_angle="pi/2"
-      update_rate="40">
-      <origin xyz="0.09525 0 -0.0127" rpy="0 0 0" />
+      max_range="40"
+      resolution="0.03"
+      update_rate="40"
+      horizontal_range="2.0944"
+      vertical_range="0.1"
+      num_horizontal_points="40"
+      num_vertical_points="2">
+      <xacro:insert_block name="origin"/>
     </xacro:laser_scanner>
   </xacro:macro>
-  <!-- Macro to add a laser scanner. -->
+  <!-- Macro to add a velodyne laser scanner. -->
   <xacro:macro
     name="laser_scanner"
     params="namespace
             parent_link
-            num_samples
             visualize
             min_range
             max_range
-            res_range
-            min_angle
-            max_angle
+            resolution
             update_rate
+            horizontal_range
+            vertical_range
+            num_horizontal_points
+            num_vertical_points
             *origin">
     <link name="${namespace}/laser_link">
@@ -63,20 +65,18 @@
         <scan>
           <horizontal>
-            <samples>60</samples>
-            <resolution>3</resolution>
-            <min_angle>-1.570796</min_angle>
-            <max_angle>1.570796</max_angle>
+            <samples>${num_horizontal_points}</samples>
+            <min_angle>${-horizontal_range/2.0}</min_angle>
+            <max_angle>${horizontal_range/2.0}</max_angle>
           </horizontal>
           <vertical>
-              <samples>60</samples>
-              <resolution>3</resolution>
-              <min_angle>-1.570796</min_angle>
-              <max_angle>1.570796</max_angle>
+            <samples>${num_vertical_points}</samples>
+            <min_angle>${-vertical_range/2.0}</min_angle>
+            <max_angle>${vertical_range/2.0}</max_angle>
           </vertical>
         </scan>
         <range>
-          <min>0.10</min>
-          <max>30.0</max>
-          <resolution>0.01</resolution>
+          <min>${min_range}</min>
+          <max>${max_range}</max>
+          <resolution>${resolution}</resolution>
         </range>
         <noise>
