Commit message: got started on cleanup

File: fcu_sim/urdf/junker/junker_base.xacro (robot description, xacro)
@@ -145,5 +145,5 @@
   <!-- Add Aerodynamics -->
   <gazebo>
-    <plugin filename="libfcu_sim_aircraft_forces_and_moments_plugin.so" name="aircraft_forces_and_moments_plugin">
+    <plugin filename="aircraft_forces_and_moments_plugin.so" name="aircraft_forces_and_moments_plugin">
       <namespace>${namespace}</namespace>
       <linkName>${namespace}/base_link</linkName>
@@ -226,5 +226,5 @@
   <!-- Sensors -->
   <gazebo>
-    <plugin filename="libfcu_sim_aircraft_truth_plugin.so" name="aircraft_truth_plugin">
+    <plugin filename="aircraft_truth_plugin.so" name="aircraft_truth_plugin">
       <namespace>${namespace}</namespace>
       <linkName>${namespace}/base_link</linkName>

File: fcu_sim/urdf/shredder/shredder_base.xacro (robot description, xacro)
@@ -47,9 +47,9 @@
   <!-- ************************* ROTOR DYNAMICS ********************** -->
   <!-- ROSflight_SIL -->
-  <!-- <xacro:include filename="$(find fcu_sim_plugins)/xacro/ROSflight_SIL.xacro"/> -->
-  <!-- <xacro:mikey_ROSflight_SIL namespace="${namespace}" parent_link="${namespace}/base_link"/> -->
+  <xacro:include filename="$(find fcu_sim_plugins)/xacro/ROSflight_SIL.xacro"/>
+  <xacro:mikey_ROSflight_SIL namespace="${namespace}" parent_link="${namespace}/base_link"/>
   <!-- Simplified Dynamics -->
-  <xacro:include filename="$(find fcu_sim_plugins)/xacro/multirotor_forces_and_moments.xacro"/>
-  <xacro:shredder_forces_and_moments namespace="${namespace}" parent_link="${namespace}/base_link"/>
+  <!-- <xacro:include filename="$(find fcu_sim_plugins)/xacro/multirotor_forces_and_moments.xacro"/> -->
+  <!-- <xacro:shredder_forces_and_moments namespace="${namespace}" parent_link="${namespace}/base_link"/> -->
   <!-- ***************** SENSORS ******************* -->
   <!-- Ground Truth -->
@@ -69,12 +69,12 @@
     wind_pub_topic="wind"/> -->
   <!-- Mount an Altimeter -->
-  <xacro:include filename="$(find fcu_sim_plugins)/xacro/altimeter.xacro"/>
+  <!-- <xacro:include filename="$(find fcu_sim_plugins)/xacro/altimeter.xacro"/>
   <xacro:perfect_baro
     namespace="${namespace}"
     parent_link="${namespace}/base_link"
-    altimeter_topic="altimeter"/>
+    altimeter_topic="altimeter"/> -->
   <!-- Mount a Magnetometer -->
   <!-- Default Inclination and Declination for Provo, UT -->
-  <xacro:include filename="$(find fcu_sim_plugins)/xacro/magnetometer.xacro"/>
+  <!-- <xacro:include filename="$(find fcu_sim_plugins)/xacro/magnetometer.xacro"/>
   <xacro:hmc5883l
     namespace="${namespace}"
@@ -82,5 +82,5 @@
     mag_topic="mag/data"
     inclination="1.14316156541"
-    declination="0.198584539676"/>
+    declination="0.198584539676"/> -->
   <!-- Mount an RGBD Camera -->
   <!-- <xacro:include filename="$(find fcu_sim_plugins)/xacro/rgbd.xacro"/>
@@ -88,5 +88,5 @@
     namespace="${namespace}"
     parent_link="${namespace}/bavese_link"/> -->
-  <!-- Laser Scanner -->
+  <!-- Block Laser Scanner -->
   <!-- <xacro:include filename="$(find fcu_sim_plugins)/xacro/velodyne.xacro"/>
   <xacro:velodyne_custom
@@ -103,9 +103,9 @@
     visualize="false"/> -->
   <!-- GPS -->
-  <xacro:include filename="$(find fcu_sim_plugins)/xacro/GPS.xacro"/>
+  <!-- <xacro:include filename="$(find fcu_sim_plugins)/xacro/GPS.xacro"/>
   <xacro:GPS_BYU
     namespace="${namespace}"
     parent_link="${namespace}/base_link"
-    GPS_topic="gps"/>
+    GPS_topic="gps"/> -->
   <!-- Camera -->
   <xacro:include filename="$(find fcu_sim_plugins)/xacro/camera.xacro"/>

File: fcu_sim_plugins/xacro/GPS.xacro (robot description, xacro)
@@ -50,5 +50,5 @@
     <!-- Load Plugin -->
     <gazebo>
-      <plugin filename="libfcu_sim_GPS_plugin.so" name="fcu_sim_GPS_plugin">
+      <plugin filename="libGPS_plugin.so" name="fcu_sim_GPS_plugin">
       <namespace>${namespace}</namespace>
       <linkName>${namespace}/GPS_link</linkName>

File: fcu_sim_plugins/xacro/ROSflight_SIL.xacro (robot description, xacro)
@@ -4,7 +4,7 @@
     <!-- Forces And Moments Plugin -->
     <xacro:macro
-      name="square_quad"
+      name="square_quad_SIL"
       params="namespace parent_link">
-      <xacro:fcu_sim_ROSflight_sil_plugin
+      <xacro:ROSflight_sil_plugin
         namespace="${namespace}/hil"
         parent_link="${namespace}/base_link"
@@ -12,5 +12,6 @@
         command_topic="extended_command"
         parent_frame_id="${parent_link}"
-        mu="1"
+        linear_mu="1"
+        angular_mu="0.3"
         rotor_max_thrust="14.961"
         rotor_F1="1.5e-5"
@@ -49,10 +50,10 @@
         <inertia ixx="0.00001" ixy="0.0" ixz="0.0" iyy="0.00001" iyz="0.0" izz="0.00001" />
         <origin xyz="0.0 0.0 0.0" rpy="0.0 0.0 0.0" />
-      </xacro:fcu_sim_ROSflight_sil_plugin>
+      </xacro:ROSflight_sil_plugin>
     </xacro:macro>
     <xacro:macro
       name="mikey_ROSflight_SIL"
       params="namespace parent_link">
-      <xacro:fcu_sim_ROSflight_sil_plugin
+      <xacro:ROSflight_sil_plugin
         namespace="${namespace}/hil"
         parent_link="${namespace}/base_link"
@@ -103,8 +104,8 @@
         <inertia ixx="0.00001" ixy="0.0" ixz="0.0" iyy="0.00001" iyz="0.0" izz="0.00001" />
         <origin xyz="0.0 0.0 0.0" rpy="0.0 0.0 0.0" />
-      </xacro:fcu_sim_ROSflight_sil_plugin>
+      </xacro:ROSflight_sil_plugin>
     </xacro:macro>
   <!-- Macro to add a generic multirotor forces and moments plugin. -->
-  <xacro:macro name="fcu_sim_ROSflight_sil_plugin"
+  <xacro:macro name="ROSflight_sil_plugin"
     params="
         namespace parent_link wind_speed_topic command_topic parent_frame_id
@@ -133,5 +134,5 @@
     <!-- plugin -->
     <gazebo>
-      <plugin filename="libfcu_sim_ROSflight_sil_plugin.so" name="multirotor_hil">
+      <plugin filename="libROSflight_sil_plugin.so" name="multirotor_hil">
         <linkName>${namespace}/ROSflight_SIL_link</linkName>
         <robotNamespace>${namespace}</robotNamespace>

File: fcu_sim_plugins/xacro/aircraft_forces_and_moments.xacro (robot description, xacro)
@@ -107,5 +107,5 @@
     </joint>
     <gazebo>
-      <plugin filename="libfcu_sim_aircraft_and_moments_plugin.so" name="aircraft_forces_and_moments">
+      <plugin filename="libaircraft_and_moments_plugin.so" name="aircraft_forces_and_moments">
         <linkName>${namespace}/aircraft_forces_and_moments_link</linkName>
         <robotNamespace>${namespace}</robotNamespace>

File: fcu_sim_plugins/xacro/airspeed.xacro (robot description, xacro)
@@ -42,5 +42,5 @@
     <!-- Load Plugin -->
     <gazebo>
-      <plugin filename="libfcu_sim_airspeed_plugin.so" name="fcu_sim_airspeed_plugin">
+      <plugin filename="libairspeed_plugin.so" name="fcu_sim_airspeed_plugin">
         <namespace>${namespace}</namespace>
         <linkName>${namespace}/airspeed_link</linkName>

File: fcu_sim_plugins/xacro/altimeter.xacro (robot description, xacro)
@@ -129,5 +129,5 @@
     </joint>
     <gazebo>
-      <plugin filename="libfcu_sim_altimeter_plugin.so" name="fcu_sim_altimeter${altimeter_suffix}_plugin">
+      <plugin filename="libaltimeter_plugin.so" name="fcu_sim_altimeter${altimeter_suffix}_plugin">
       <!-- A good description of the altimeter parameters can be found in the kalibr documentation:
            https://github.com/ethz-asl/kalibr/wiki/altimeter-Noise-Model-and-Intrinsics -->

File: fcu_sim_plugins/xacro/gimbal.xacro (robot description, xacro)
@@ -126,5 +126,5 @@
     <!-- Load Gimbal Controller Plugin -->
     <gazebo>
-      <plugin filename="libfcu_sim_gimbal_plugin.so" name="fcu_sim_gimbal_plugin">
+      <plugin filename="libgimbal_plugin.so" name="fcu_sim_gimbal_plugin">
         <namespace>${namespace}</namespace>
         <yawJoint>${namespace}/gimbal_yaw_joint</yawJoint>

File: fcu_sim_plugins/xacro/imu.xacro (robot description, xacro)
@@ -95,5 +95,5 @@
     </joint>
     <gazebo>
-      <plugin filename="libfcu_sim_imu_plugin.so" name="fcu_sim_imu${imu_suffix}_plugin">
+      <plugin filename="libimu_plugin.so" name="fcu_sim_imu${imu_suffix}_plugin">
       <!-- A good description of the IMU parameters can be found in the kalibr documentation:
            https://github.com/ethz-asl/kalibr/wiki/IMU-Noise-Model-and-Intrinsics -->

File: fcu_sim_plugins/xacro/magnetometer.xacro (robot description, xacro)
@@ -46,5 +46,5 @@
     </joint>
     <gazebo>
-      <plugin filename="libfcu_sim_magnetometer_plugin.so" name="fcu_sim_magnetometer_plugin">
+      <plugin filename="magnetometer_plugin.so" name="fcu_sim_magnetometer_plugin">
       <namespace>${namespace}</namespace>
       <linkName>${namespace}/magnetometer_link</linkName>

File: fcu_sim_plugins/xacro/multirotor_forces_and_moments.xacro (robot description, xacro)
@@ -92,5 +92,5 @@
       <inertial>
         <xacro:insert_block name="inertia" />
-        <mass value="0.001"/>  <!-- [kg] -->
+        <mass value="0.001"/>
       </inertial>
     </link>
@@ -104,5 +104,5 @@
     <!-- plugin -->
     <gazebo>
-      <plugin filename="libfcu_sim_multirotor_forces_and_moments_plugin.so" name="multirotor_forces_and_moments">
+      <plugin filename="libmultirotor_forces_and_moments_plugin.so" name="multirotor_forces_and_moments">
         <linkName>${namespace}/multirotor_forces_and_moments_link</linkName>
         <robotNamespace>${namespace}</robotNamespace>

File: fcu_sim_plugins/xacro/odometry_sensor.xacro (robot description, xacro)
@@ -61,5 +61,5 @@
     </joint>
     <gazebo>
-      <plugin filename="libfcu_sim_odometry_plugin.so" name="odometry_sensor${odometry_sensor_suffix}">
+      <plugin filename="libodometry_plugin.so" name="odometry_sensor${odometry_sensor_suffix}">
         <linkName>${namespace}/odometry_sensor${odometry_sensor_suffix}_link</linkName>
         <robotNamespace>${namespace}</robotNamespace>

File: fcu_sim_plugins/xacro/wind.xacro (robot description, xacro)
@@ -27,5 +27,5 @@
           wind_gust_force_variance wind_gust_direction">
     <gazebo>
-      <plugin filename="libfcu_sim_wind_plugin.so" name="gazebo_wind_plugin">
+      <plugin filename="libwind_plugin.so" name="gazebo_wind_plugin">
         <robotNamespace>${namespace}</robotNamespace> <!-- (string, required): ros namespace in which the messages are published -->
         <xyzOffset>${xyz_offset}</xyzOffset> <!-- (Vector3, required): -->
