Commit message: a lot of cleanup.  Split barometer and sonar into different plugins, changed output of barometer to fcu_common/Barometer message.  Removed all redefinitions of pi.  Moved aircraft_forces_and_moments into it's own plugin.  Now outputting fcu_common/Airspeed instead of FluidPressure

File: fcu_sim/urdf/junker/junker_base.xacro (robot description, xacro)
@@ -15,85 +15,14 @@
   <xacro:property name="Jz" value="0.1712"/>
   <xacro:property name="Jxz" value="0.0015"/>
-  <xacro:property name="rho" value="1.2682"/>
-  <xacro:property name="wing_s" value="0.2589"/>
-  <xacro:property name="wing_b" value="1.4224"/>
-  <xacro:property name="wing_c" value="0.3302"/>
-  <xacro:property name="wing_M" value="0.55"/>
-  <xacro:property name="wing_epsilon" value="2.8956"/>
-  <xacro:property name="wing_alpha0" value="0.18994"/>
-  <xacro:property name="k_motor" value="40.0"/>
-  <xacro:property name="k_T_P" value="0.0"/>
-  <xacro:property name="k_Omega" value="0.0"/>
-  <xacro:property name="prop_e" value="0.9"/>
-  <xacro:property name="prop_S" value="0.0314"/>
-  <xacro:property name="prop_C" value="1.0"/>
-  <xacro:property name="C_L_O" value="0.28"/>
-  <xacro:property name="C_L_alpha" value="3.45"/>
-  <xacro:property name="C_L_beta" value="0.0"/>
-  <xacro:property name="C_L_p" value="0.0"/>
-  <xacro:property name="C_L_q" value="0.0"/>
-  <xacro:property name="C_L_r" value="0.0"/>
-  <xacro:property name="C_L_delta_a" value="0.0"/>
-  <xacro:property name="C_L_delta_e" value="-0.36"/>
-  <xacro:property name="C_L_delta_r" value="0.0"/>
-  <xacro:property name="C_D_O" value="0.03"/>
-  <xacro:property name="C_D_alpha" value="0.2108"/>
-  <xacro:property name="C_D_beta" value="0.0"/>
-  <xacro:property name="C_D_p" value="0.0437"/>
-  <xacro:property name="C_D_q" value="0.0"/>
-  <xacro:property name="C_D_r" value="0.0"/>
-  <xacro:property name="C_D_delta_a" value="0.0"/>
-  <xacro:property name="C_D_delta_e" value="0.0"/>
-  <xacro:property name="C_D_delta_r" value="0.0"/>
-  <xacro:property name="C_ell_O" value="0.0"/>
-  <xacro:property name="C_ell_alpha" value="0.00"/>
-  <xacro:property name="C_ell_beta" value="-0.12"/>
-  <xacro:property name="C_ell_p" value="-0.26"/>
-  <xacro:property name="C_ell_q" value="0.0"/>
-  <xacro:property name="C_ell_r" value="0.14"/>
-  <xacro:property name="C_ell_delta_a" value="0.08"/>
-  <xacro:property name="C_ell_delta_e" value="0.0"/>
-  <xacro:property name="C_ell_delta_r" value="0.105"/>
-  <xacro:property name="C_m_O" value="0.0"/>
-  <xacro:property name="C_m_alpha" value="-0.38"/>
-  <xacro:property name="C_m_beta" value="0.0"/>
-  <xacro:property name="C_m_p" value="0.0"/>
-  <xacro:property name="C_m_q" value="-3.6"/>
-  <xacro:property name="C_m_r" value="0.0"/>
-  <xacro:property name="C_m_delta_a" value="0.0"/>
-  <xacro:property name="C_m_delta_e" value="-0.5"/>
-  <xacro:property name="C_m_delta_r" value="0.0"/>
-  <xacro:property name="C_n_O" value="0.0"/>
-  <xacro:property name="C_n_alpha" value="0.0"/>
-  <xacro:property name="C_n_beta" value="0.25"/>
-  <xacro:property name="C_n_p" value="0.022"/>
-  <xacro:property name="C_n_q" value="0.0"/>
-  <xacro:property name="C_n_r" value="-0.35"/>
-  <xacro:property name="C_n_delta_a" value="0.06"/>
-  <xacro:property name="C_n_delta_e" value="0.0"/>
-  <xacro:property name="C_n_delta_r" value="-0.032"/>
-  <xacro:property name="C_Y_O" value="0.0"/>
-  <xacro:property name="C_Y_alpha" value="0.00"/>
-  <xacro:property name="C_Y_beta" value="-0.98"/>
-  <xacro:property name="C_Y_p" value="0.0"/>
-  <xacro:property name="C_Y_q" value="0.0"/>
-  <xacro:property name="C_Y_r" value="0.0"/>
-  <xacro:property name="C_Y_delta_a" value="0.0"/>
-  <xacro:property name="C_Y_delta_e" value="0.0"/>
-  <xacro:property name="C_Y_delta_r" value="-0.17"/>
   <!-- Property Blocks -->
-  <xacro:property name="inertia">
-    <inertia ixx="0.8244" ixy="0.0" ixz=".1204" iyy="1.135" iyz="0.0" izz="1.759" />
-  </xacro:property>
     <xacro:property name="empty_inertia">
     <inertia ixx="0.0001" ixy="0.0" ixz="0.0" iyy="0.0001" iyz="0.0" izz="0.001" />
   </xacro:property>
   <!-- Instantiate Link and Visual -->
-  <xacro:include filename="$(find fcu_sim_plugins)/xacro/wheel.xacro"/>
   <link name="${namespace}/base_link">
     <inertial>
-      <mass value="${mass}" />
+      <mass value="0.00001" />
       <origin xyz="0 0 0" />
-      <xacro:insert_block name="inertia" />
+      <xacro:insert_block name="empty_inertia" />
     </inertial>
     <visual name="plane_visual">
@@ -115,4 +44,5 @@
     </collision>
     <!-- Wheels -->
+    <xacro:include filename="$(find fcu_sim_plugins)/xacro/wheel.xacro"/>
     <xacro:caster
       radius="0.05">
@@ -143,85 +73,10 @@
     <material>Gazebo/Blue</material>
   </gazebo>
-  <!-- Add Aerodynamics -->
-  <gazebo>
-    <plugin filename="aircraft_forces_and_moments_plugin.so" name="aircraft_forces_and_moments_plugin">
-      <namespace>${namespace}</namespace>
-      <linkName>${namespace}/base_link</linkName>
-      <windSpeedTopic>${wind_speed_topic}</windSpeedTopic>
-      <commandTopic>${command_topic}</commandTopic>
-      <mass>${mass}</mass>
-      <Jx>${Jx}</Jx>
-      <Jy>${Jy}</Jy>
-      <Jz>${Jz}</Jz>
-      <Jxz>${Jxz}</Jxz>
-      <rho>${rho}</rho>
-      <wing_s>${wing_s}</wing_s>
-      <wing_b>${wing_b}</wing_b>
-      <wing_c>${wing_c}</wing_c>
-      <wing_M>${wing_M}</wing_M>
-      <wing_epsilon>${wing_epsilon}</wing_epsilon>
-      <wing_alpha0>${wing_alpha0}</wing_alpha0>
-      <k_motor>${k_motor}</k_motor>
-      <k_T_P>${k_T_P}</k_T_P>
-      <k_Omega>${k_Omega}</k_Omega>
-      <prop_e>${prop_e}</prop_e>
-      <prop_S>${prop_S}</prop_S>
-      <prop_C>${prop_C}</prop_C>
-      <C_L_O>${C_L_O}</C_L_O>
-      <C_L_alpha>${C_L_alpha}</C_L_alpha>
-      <C_L_beta>${C_L_beta}</C_L_beta>
-      <C_L_p>${C_L_p}</C_L_p>
-      <C_L_q>${C_L_q}</C_L_q>
-      <C_L_r>${C_L_r}</C_L_r>
-      <C_L_delta_a>${C_L_delta_a}</C_L_delta_a>
-      <C_L_delta_e>${C_L_delta_e}</C_L_delta_e>
-      <C_L_delta_r>${C_L_delta_r}</C_L_delta_r>
-      <C_D_O>${C_D_O}</C_D_O>
-      <C_D_alpha>${C_D_alpha}</C_D_alpha>
-      <C_D_beta>${C_D_beta}</C_D_beta>
-      <C_D_p>${C_D_p}</C_D_p>
-      <C_D_q>${C_D_q}</C_D_q>
-      <C_D_r>${C_D_r}</C_D_r>
-      <C_D_delta_a>${C_D_delta_a}</C_D_delta_a>
-      <C_D_delta_e>${C_D_delta_e}</C_D_delta_e>
-      <C_D_delta_r>${C_D_delta_r}</C_D_delta_r>
-      <C_ell_O>${C_ell_O}</C_ell_O>
-      <C_ell_alpha>${C_ell_alpha}</C_ell_alpha>
-      <C_ell_beta>${C_ell_beta}</C_ell_beta>
-      <C_ell_p>${C_ell_p}</C_ell_p>
-      <C_ell_q>${C_ell_q}</C_ell_q>
-      <C_ell_r>${C_ell_r}</C_ell_r>
-      <C_ell_delta_a>${C_ell_delta_a}</C_ell_delta_a>
-      <C_ell_delta_e>${C_ell_delta_e}</C_ell_delta_e>
-      <C_ell_delta_r>${C_ell_delta_r}</C_ell_delta_r>
-      <C_m_O>${C_m_O}</C_m_O>
-      <C_m_alpha>${C_m_alpha}</C_m_alpha>
-      <C_m_beta>${C_m_beta}</C_m_beta>
-      <C_m_p>${C_m_p}</C_m_p>
-      <C_m_q>${C_m_q}</C_m_q>
-      <C_m_r>${C_m_r}</C_m_r>
-      <C_m_delta_a>${C_m_delta_a}</C_m_delta_a>
-      <C_m_delta_e>${C_m_delta_e}</C_m_delta_e>
-      <C_m_delta_r>${C_m_delta_r}</C_m_delta_r>
-      <C_n_O>${C_n_O}</C_n_O>
-      <C_n_alpha>${C_n_alpha}</C_n_alpha>
-      <C_n_beta>${C_n_beta}</C_n_beta>
-      <C_n_p>${C_n_p}</C_n_p>
-      <C_n_q>${C_n_q}</C_n_q>
-      <C_n_r>${C_n_r}</C_n_r>
-      <C_n_delta_a>${C_n_delta_a}</C_n_delta_a>
-      <C_n_delta_e>${C_n_delta_e}</C_n_delta_e>
-      <C_n_delta_r>${C_n_delta_r}</C_n_delta_r>
-      <C_Y_O>${C_Y_O}</C_Y_O>
-      <C_Y_alpha>${C_Y_alpha}</C_Y_alpha>
-      <C_Y_beta>${C_Y_beta}</C_Y_beta>
-      <C_Y_p>${C_Y_p}</C_Y_p>
-      <C_Y_q>${C_Y_q}</C_Y_q>
-      <C_Y_r>${C_Y_r}</C_Y_r>
-      <C_Y_delta_a>${C_Y_delta_a}</C_Y_delta_a>
-      <C_Y_delta_e>${C_Y_delta_e}</C_Y_delta_e>
-      <C_Y_delta_r>${C_Y_delta_r}</C_Y_delta_r>
-    </plugin>
-  </gazebo>
+  <!-- Aerodynamics -->
+  <xacro:include filename="$(find fcu_sim_plugins)/xacro/aircraft_forces_and_moments.xacro"/>
+  <xacro:aerosonde
+    namespace="${namespace}"
+    parent_link="${namespace}/base_link"
+    command_topic="comamand"/>
   <!-- Sensors -->
   <gazebo>
@@ -238,4 +93,5 @@
     parent_link="${namespace}/base_link"
     camera_topic="rgb"
+    frame_rate="30"
     pose_topic="${namespace}/gimbal/pose"
     command_topic="${namespace}/gimbal/control"
@@ -257,16 +113,19 @@
     GPS_topic="gps/data">
   </xacro:GPS_BYU>
-  <!-- Sonar and Barometer -->
-  <xacro:include filename="$(find fcu_sim_plugins)/xacro/altimeter.xacro"/>
-  <xacro:Sonar_HC-SR04
-    namespace="${namespace}"
-    parent_link="${namespace}/base_link"
-    altimeter_topic="sonar/data">
-  </xacro:Sonar_HC-SR04>
+  <!-- Barometer -->
+  <xacro:include filename="$(find fcu_sim_plugins)/xacro/barometer.xacro"/>
   <xacro:Barometer_MS5611
     namespace="${namespace}"
     parent_link="${namespace}/base_link"
-    altimeter_topic="baro/data">
+    baro_topic="baro/data">
   </xacro:Barometer_MS5611>
+  <!-- Sonar -->
+  <xacro:include filename="$(find fcu_sim_plugins)/xacro/sonar.xacro"/>
+  <xacro:Sonar_MB1030
+    namespace="${namespace}"
+    parent_link="${namespace}/base_link"
+    sonar_topic="sonar/data">
+    <origin xyz="0 0 0" rpy="0 0 0"/>
+  </xacro:Sonar_MB1030>
   <!-- IMU -->
   <xacro:include filename="$(find fcu_sim_plugins)/xacro/imu.xacro"/>

File: fcu_sim/urdf/mikey/mikey_base.xacro (robot description, xacro)
@@ -4,5 +4,5 @@
 Author: James Jackson
 -->
-<robot name="shredder" xmlns:xacro="http://ros.org/wiki/xacro">
+<robot name="mikey" xmlns:xacro="http://ros.org/wiki/xacro">
   <!-- Properties -->
   <xacro:property name="namespace" value="mikey" />
@@ -49,5 +49,5 @@
   <!-- Simplified Dynamics -->
   <xacro:include filename="$(find fcu_sim_plugins)/xacro/multirotor_forces_and_moments.xacro"/>
-  <xacro:mikey_forces_and_moments namespace="${namespace}" parent_link="${namespace}/base_link"/>
+  <xacro:mikey_forces_and_moments namespace="${namespace}" parent_link="${namespace}/base_link" command_topic="command"/>
   <!-- ***************** SENSORS ******************* -->
   <!-- Ground Truth -->

File: fcu_sim_plugins/xacro/GPS.xacro (robot description, xacro)
@@ -1,5 +1,4 @@
 <?xml version="1.0"?>
 <robot xmlns:xacro="http://ros.org/wiki/xacro">
-  <xacro:property name="pi" value="3.14159265359" />
   <!-- Configure GPS -->
     <xacro:macro

File: fcu_sim_plugins/xacro/ROSflight_SIL.xacro (robot description, xacro)
@@ -1,5 +1,4 @@
 <?xml version="1.0"?>
 <robot xmlns:xacro="http://ros.org/wiki/xacro">
-  <xacro:property name="pi" value="3.14159265359" />
     <!-- Forces And Moments Plugin -->
     <xacro:macro

File: fcu_sim_plugins/xacro/aircraft_forces_and_moments.xacro (robot description, xacro)
@@ -1,15 +1,14 @@
 <?xml version="1.0"?>
 <robot xmlns:xacro="http://ros.org/wiki/xacro">
-  <xacro:property name="pi" value="3.14159265359" />
     <!-- Forces And Moments Plugin -->
     <xacro:macro
-      name="aircraft_forces_and_moments"
-      params="namespace parent_link">
+      name="aerosonde"
+      params="namespace parent_link command_topic">
       <xacro:aircraft_forces_and_moments_macro
         namespace="${namespace}/aircraft_forces_and_moments"
         parent_link="${namespace}/base_link"
         wind_speed_topic="gazebo/wind_speed"
-        command_topic="control_surface_deflection"
-        parent_frame_id="airplane"
+        command_topic="command_topic"
+        parent_frame_id="${namespace}/base_link"
         mass="13.5"
         Jx="0.8244"
@@ -83,7 +82,5 @@
         C_Y_delta_a="0.0"
         C_Y_delta_e="0.0"
-        C_Y_delta_r="-0.017"
-        <inertia ixx="0.00001" ixy="0.0" ixz="0.0" iyy="0.00001" iyz="0.0" izz="0.00001" />
-        <origin xyz="0.0 0.0 0.0" rpy="0.0 0.0 0.0" />
+        C_Y_delta_r="-0.017">
       </xacro:aircraft_forces_and_moments_macro>
     </xacro:macro>
@@ -91,9 +88,18 @@
   <xacro:macro name="aircraft_forces_and_moments_macro"
     params="
-        namespace  parent_link wind_speed_topic command_topic parent_frame_id mass Jx Jy Jz Jxz rho wing_s wing_b wing_c wing_M wing_epsilon wing_alpha0 k_motor k_T_P k_Omega prop_e prop_S prop_C C_L_O C_L_alpha C_L_beta C_L_p C_L_q C_L_r C_L_delta_a C_L_delta_e C_L_delta_r C_D_O C_D_alpha C_D_beta C_D_p C_D_q C_D_r C_D_delta_a C_D_delta_e C_D_delta_r C_ell_O C_ell_alpha C_ell_beta C_ell_p C_ell_q C_ell_r C_ell_delta_a C_ell_delta_e C_ell_delta_r C_m_O C_m_alpha C_m_beta C_m_p C_m_q C_m_r C_m_delta_a C_m_delta_e C_m_delta_r C_n_O C_n_alpha C_n_beta C_n_p C_n_q C_n_r C_n_delta_a C_n_delta_e C_n_delta_r C_Y_O C_Y_alpha C_Y_beta C_Y_p C_Y_q C_Y_r C_Y_delta_a C_Y_delta_e C_Y_delta_r *inertia">
+        namespace  parent_link wind_speed_topic command_topic parent_frame_id
+        mass Jx Jy Jz Jxz rho wing_s wing_b wing_c wing_M wing_epsilon
+        wing_alpha0 k_motor k_T_P k_Omega prop_e prop_S prop_C C_L_O C_L_alpha
+        C_L_beta C_L_p C_L_q C_L_r C_L_delta_a C_L_delta_e C_L_delta_r C_D_O
+        C_D_alpha C_D_beta C_D_p C_D_q C_D_r C_D_delta_a C_D_delta_e C_D_delta_r
+        C_ell_O C_ell_alpha C_ell_beta C_ell_p C_ell_q C_ell_r C_ell_delta_a
+        C_ell_delta_e C_ell_delta_r C_m_O C_m_alpha C_m_beta C_m_p C_m_q C_m_r
+        C_m_delta_a C_m_delta_e C_m_delta_r C_n_O C_n_alpha C_n_beta C_n_p C_n_q
+        C_n_r C_n_delta_a C_n_delta_e C_n_delta_r C_Y_O C_Y_alpha C_Y_beta C_Y_p
+        C_Y_q C_Y_r C_Y_delta_a C_Y_delta_e C_Y_delta_r">
     <!-- link -->
     <link name="${namespace}/aircraft_forces_and_moments_link">
       <inertial>
-        <xacro:insert_block name="inertia" />
+        <inertia ixx="${Jx}" ixy="0.00" ixz="${Jxz}" iyy="${Jy}" iyz="0.0" izz="${Jz}" />
         <mass value="${mass}" />  <!-- [kg] -->
       </inertial>
@@ -102,5 +108,5 @@
     <joint name="${namespace}/aircraft_forces_and_moments_joint" type="revolute">
       <parent link="${parent_link}" />
-      <xacro:insert_block name="origin" />
+      <origin xyz="0 0 0" rpy="0 0 0"/>
       <child link="${namespace}/aircraft_forces_and_moments_link" />
       <limit upper="0" lower="0" effort="0" velocity="0" />

File: fcu_sim_plugins/xacro/airspeed.xacro (robot description, xacro)
@@ -1,5 +1,4 @@
 <?xml version="1.0"?>
 <robot xmlns:xacro="http://ros.org/wiki/xacro">
-  <xacro:property name="pi" value="3.14159265359" />
     <!-- Configure Airspeed -->
     <xacro:macro

File: fcu_sim_plugins/xacro/camera.xacro (robot description, xacro)
@@ -1,5 +1,4 @@
 <?xml version="1.0"?>
 <robot xmlns:xacro="http://ros.org/wiki/xacro">
-  <xacro:property name="pi" value="3.14159265359" />
   <xacro:property name="empty_inertia">
     <inertia ixx="0.0001" ixy="0.0" ixz="0.0" iyy="0.0001" iyz="0.0" izz="0.001" />
@@ -20,10 +19,4 @@
         <xacro:insert_block name="empty_inertia"/>
       </inertial>
-      <!-- <visual name="${namespace}/camera_visual">
-        <xacro:insert_block name="origin"/>
-        <geometry>
-          <sphere radius="0.05"/>
-        </geometry>
-      </visual> -->
     </link>
     <joint name="${namespace}/camera_joint" type="fixed">

File: fcu_sim_plugins/xacro/gimbal.xacro (robot description, xacro)
@@ -7,5 +7,5 @@
               parent_link
               camera_topic
-	      frame_rate
+	            frame_rate
               pose_topic
               command_topic

File: fcu_sim_plugins/xacro/imu.xacro (robot description, xacro)
@@ -1,5 +1,4 @@
 <?xml version="1.0"?>
 <robot xmlns:xacro="http://ros.org/wiki/xacro">
-  <xacro:property name="pi" value="3.14159265359" />
     <!-- Configure IMU -->
     <xacro:macro

File: fcu_sim_plugins/xacro/laser_scanner.xacro (robot description, xacro)
@@ -1,5 +1,4 @@
 <?xml version="1.0"?>
 <robot xmlns:xacro="http://ros.org/wiki/xacro">
-  <xacro:property name="pi" value="3.14159265359" />
   <!-- Hokuyo UTM-30LX-->
   <xacro:macro

File: fcu_sim_plugins/xacro/multirotor_forces_and_moments.xacro (robot description, xacro)
@@ -1,5 +1,4 @@
 <?xml version="1.0"?>
 <robot xmlns:xacro="http://ros.org/wiki/xacro">
-  <xacro:property name="pi" value="3.14159265359" />
     <!-- Forces And Moments Plugin -->
     <xacro:macro

File: fcu_sim_plugins/xacro/odometry_sensor.xacro (robot description, xacro)
@@ -1,5 +1,4 @@
 <?xml version="1.0"?>
 <robot xmlns:xacro="http://ros.org/wiki/xacro">
-  <xacro:property name="pi" value="3.14159265359" />
     <!-- Odometry Sensor -->
     <xacro:macro

File: fcu_sim_plugins/xacro/rgbd.xacro (robot description, xacro)
@@ -1,5 +1,4 @@
 <?xml version="1.0"?>
 <robot xmlns:xacro="http://ros.org/wiki/xacro">
-  <xacro:property name="pi" value="3.14159265359" />
   <!-- XTION -->
   <xacro:macro

File: fcu_sim_plugins/xacro/velodyne.xacro (robot description, xacro)
@@ -1,5 +1,4 @@
 <?xml version="1.0"?>
 <robot xmlns:xacro="http://ros.org/wiki/xacro">
-  <xacro:property name="pi" value="3.14159265359" />
   <xacro:macro
     name="velodyne_custom"

File: fcu_sim_plugins/xacro/wind.xacro (robot description, xacro)
@@ -1,5 +1,4 @@
 <?xml version="1.0"?>
 <robot xmlns:xacro="http://ros.org/wiki/xacro">
-  <xacro:property name="pi" value="3.14159265359" />
   <!-- Wind Parameters -->
   <xacro:macro

Commit message: got ros_plane topics all hooked up

File: fcu_sim/urdf/junker/junker_base.xacro (robot description, xacro)
@@ -16,5 +16,5 @@
   <xacro:property name="Jxz" value="0.0015"/>
   <!-- Property Blocks -->
-    <xacro:property name="empty_inertia">
+  <xacro:property name="empty_inertia">
     <inertia ixx="0.0001" ixy="0.0" ixz="0.0" iyy="0.0001" iyz="0.0" izz="0.001" />
   </xacro:property>
@@ -22,7 +22,7 @@
   <link name="${namespace}/base_link">
     <inertial>
-      <mass value="0.00001" />
+      <mass value="0.001" />
       <origin xyz="0 0 0" />
-      <xacro:insert_block name="empty_inertia" />
+      <inertia ixx="0.001" ixy="0.00" ixz="0.00" iyy="0.001" iyz="0.00" izz="0.001" />
     </inertial>
     <visual name="plane_visual">
@@ -78,13 +78,11 @@
     namespace="${namespace}"
     parent_link="${namespace}/base_link"
-    command_topic="comamand"/>
+    command_topic="command"/>
   <!-- Sensors -->
-  <gazebo>
-    <plugin filename="aircraft_truth_plugin.so" name="aircraft_truth_plugin">
-      <namespace>${namespace}</namespace>
-      <linkName>${namespace}/base_link</linkName>
-      <windSpeedTopic>${wind_speed_topic}</windSpeedTopic>
-    </plugin>
-  </gazebo>
+  <xacro:include filename="$(find fcu_sim_plugins)/xacro/aircraft_truth.xacro"/>
+  <xacro:aircraft_truth
+    namespace="${namespace}"
+    parent_link="${namespace}/base_link"
+    wind_speed_topic="gazebo/wind_speed"/>
   <!-- Gimbal -->
   <xacro:include filename="$(find fcu_sim_plugins)/xacro/gimbal.xacro"/>

File: fcu_sim_plugins/xacro/GPS.xacro (robot description, xacro)
@@ -6,5 +6,5 @@
       params="namespace parent_link GPS_topic">
     <xacro:gps_plugin_macro
-      namespace=""
+      namespace="${namespace}"
       parent_link="${parent_link}"
       gps_topic="${GPS_topic}"

File: fcu_sim_plugins/xacro/aircraft_forces_and_moments.xacro (robot description, xacro)
@@ -6,10 +6,10 @@
       params="namespace parent_link command_topic">
       <xacro:aircraft_forces_and_moments_macro
-        namespace="${namespace}/aircraft_forces_and_moments"
+        namespace="${namespace}"
         parent_link="${namespace}/base_link"
         wind_speed_topic="gazebo/wind_speed"
-        command_topic="command_topic"
+        command_topic="${command_topic}"
         parent_frame_id="${namespace}/base_link"
-        mass="13.5"
+        mass="1.5"
         Jx="0.8244"
         Jy="1.135"
@@ -102,5 +102,5 @@
       <inertial>
         <inertia ixx="${Jx}" ixy="0.00" ixz="${Jxz}" iyy="${Jy}" iyz="0.0" izz="${Jz}" />
-        <mass value="${mass}" />  <!-- [kg] -->
+        <mass value="${mass}" />
       </inertial>
     </link>
@@ -113,7 +113,7 @@
     </joint>
     <gazebo>
-      <plugin filename="libaircraft_and_moments_plugin.so" name="aircraft_forces_and_moments">
+      <plugin filename="libaircraft_forces_and_moments_plugin.so" name="${namespace}_aircraft_forces_and_moments">
         <linkName>${namespace}/aircraft_forces_and_moments_link</linkName>
-        <robotNamespace>${namespace}</robotNamespace>
+        <namespace>${namespace}</namespace>
         <windSpeedTopic>${wind_speed_topic}</windSpeedTopic>
         <commandTopic>${command_topic}</commandTopic>

Commit message: fixedwind and multirotor example working perfectly

File: fcu_sim/urdf/junker/junker_base.xacro (robot description, xacro)
@@ -22,7 +22,7 @@
   <link name="${namespace}/base_link">
     <inertial>
-      <mass value="0.001" />
+      <mass value="${mass}" />
       <origin xyz="0 0 0" />
-      <inertia ixx="0.001" ixy="0.00" ixz="0.00" iyy="0.001" iyz="0.00" izz="0.001" />
+      <inertia ixx="${Jx}" ixy="0.00" ixz="${Jxz}" iyy="${Jy}" iyz="0.00" izz="${Jz}" />
     </inertial>
     <visual name="plane_visual">
@@ -58,4 +58,10 @@
     </xacro:caster>
   </link>
+  <!-- Aerodynamics -->
+  <xacro:include filename="$(find fcu_sim_plugins)/xacro/aircraft_forces_and_moments.xacro"/>
+  <xacro:aerosonde
+    namespace="${namespace}"
+    parent_link="${namespace}/base_link"
+    command_topic="command"/>
   <!-- Chase Camera -->
   <xacro:include filename="$(find fcu_sim_plugins)/xacro/camera.xacro"/>
@@ -73,10 +79,4 @@
     <material>Gazebo/Blue</material>
   </gazebo>
-  <!-- Aerodynamics -->
-  <xacro:include filename="$(find fcu_sim_plugins)/xacro/aircraft_forces_and_moments.xacro"/>
-  <xacro:aerosonde
-    namespace="${namespace}"
-    parent_link="${namespace}/base_link"
-    command_topic="command"/>
   <!-- Sensors -->
   <xacro:include filename="$(find fcu_sim_plugins)/xacro/aircraft_truth.xacro"/>

File: fcu_sim_plugins/xacro/aircraft_forces_and_moments.xacro (robot description, xacro)
@@ -98,21 +98,9 @@
         C_n_r C_n_delta_a C_n_delta_e C_n_delta_r C_Y_O C_Y_alpha C_Y_beta C_Y_p
         C_Y_q C_Y_r C_Y_delta_a C_Y_delta_e C_Y_delta_r">
-    <!-- link -->
-    <link name="${namespace}/aircraft_forces_and_moments_link">
-      <inertial>
-        <inertia ixx="${Jx}" ixy="0.00" ixz="${Jxz}" iyy="${Jy}" iyz="0.0" izz="${Jz}" />
-        <mass value="${mass}" />
-      </inertial>
-    </link>
-    <!-- odometry joint -->
-    <joint name="${namespace}/aircraft_forces_and_moments_joint" type="revolute">
-      <parent link="${parent_link}" />
-      <origin xyz="0 0 0" rpy="0 0 0"/>
-      <child link="${namespace}/aircraft_forces_and_moments_link" />
-      <limit upper="0" lower="0" effort="0" velocity="0" />
-    </joint>
     <gazebo>
-      <plugin filename="libaircraft_forces_and_moments_plugin.so" name="${namespace}_aircraft_forces_and_moments">
-        <linkName>${namespace}/aircraft_forces_and_moments_link</linkName>
+      <plugin
+        filename="libaircraft_forces_and_moments_plugin.so"
+        name="${namespace}_aircraft_forces_and_moments">
+        <linkName>${parent_link}</linkName>
         <namespace>${namespace}</namespace>
         <windSpeedTopic>${wind_speed_topic}</windSpeedTopic>
