Commit message: added color arg to single launch files

File: fcu_sim/urdf/mikey/mikey_base.xacro (robot description, xacro)
@@ -57,4 +57,7 @@
     </collision>
   </link>
+  <gazebo reference="${namespace}/base_link">
+    <material>Gazebo/$(arg color)</material>
+  </gazebo>
   <!-- ************************* ROTOR DYNAMICS ********************** -->
 <!--   <gazebo>
@@ -66,5 +69,5 @@
   </gazebo> -->
   <!-- **************** ROTORS ***************** -->
-  <xacro:include filename="$(find fcu_sim_plugins)/xacro/rotor.xacro" />
+  <xacro:include filename="$(find fcu_sim_plugins)/xacro/rotor.xacro" />${namespace}/base_link
   <xacro:vertical_rotor
     robot_namespace="${namespace}"
@@ -195,8 +198,6 @@
   <!-- ***************** SENSORS ******************* -->
   <!-- Ground Truth -->
-  <xacro:if value="$(arg enable_ground_truth)">
-    <xacro:include filename="$(find fcu_sim_plugins)/xacro/odometry_sensor.xacro"/>
-    <xacro:ground_truth namespace="${namespace}" parent_link="${namespace}/base_link" />
-  </xacro:if>
+  <xacro:include filename="$(find fcu_sim_plugins)/xacro/odometry_sensor.xacro"/>
+  <xacro:ground_truth namespace="${namespace}" parent_link="${namespace}/base_link" />
   <!-- Mount an IMU -->
   <xacro:include filename="$(find fcu_sim_plugins)/xacro/imu.xacro"/>

File: fcu_sim/urdf/shredder/shredder_base.xacro (robot description, xacro)
@@ -57,4 +57,7 @@
     </collision>
   </link>
+  <gazebo reference="${namespace}/base_link">
+    <material>Gazebo/$(arg color)</material>
+  </gazebo>
   <!-- ************************* ROTOR DYNAMICS ********************** -->
 <!--   <gazebo>
@@ -193,8 +196,6 @@
   <!-- ***************** SENSORS ******************* -->
   <!-- Ground Truth -->
-  <xacro:if value="$(arg enable_ground_truth)">
-    <xacro:include filename="$(find fcu_sim_plugins)/xacro/odometry_sensor.xacro"/>
-    <xacro:ground_truth namespace="${namespace}" parent_link="${namespace}/base_link" />
-  </xacro:if>
+  <xacro:include filename="$(find fcu_sim_plugins)/xacro/odometry_sensor.xacro"/>
+  <xacro:ground_truth namespace="${namespace}" parent_link="${namespace}/base_link" />
   <!-- Mount an IMU -->
   <xacro:include filename="$(find fcu_sim_plugins)/xacro/imu.xacro"/>

Commit message: got ready for contact sensor

File: fcu_sim/urdf/mikey/mikey_base.xacro (robot description, xacro)
@@ -11,6 +11,6 @@
   <xacro:property name="mesh_file" value="package://fcu_sim/meshes/firefly.dae" />
   <xacro:property name="mass" value="3.81" /> <!-- [kg] -->
-  <xacro:property name="body_width" value="0.1" /> <!-- [m] -->
-  <xacro:property name="body_height" value="0.16" /> <!-- [m] -->
+  <xacro:property name="body_width" value="0.505" /> <!-- [m] -->
+  <xacro:property name="body_height" value="0.1" /> <!-- [m] -->
   <xacro:property name="mass_rotor" value="0.005" /> <!-- [kg] -->
   <xacro:property name="arm_length" value="0.3429" /> <!-- [m] -->
@@ -46,5 +46,5 @@
         </xacro:if>
         <xacro:unless value="${use_mesh_file}">
-          <box size="${body_width} ${body_width} ${body_height}"/> <!-- [m] [m] [m] -->
+          <cylinder length="${body_height}" radius="${body_width}"/>
         </xacro:unless>
       </geometry>
@@ -53,5 +53,5 @@
       <origin xyz="0 0 0" rpy="0 0 0" />
       <geometry>
-        <box size="${body_width} ${body_width} ${body_height}" /> <!-- [m] [m] [m] -->
+        <cylinder length="${body_height}" radius="${body_width}"/>
       </geometry>
     </collision>
@@ -206,9 +206,9 @@
     imu_topic="imu"/>
   <!--Enable Wind -->
-  <xacro:include filename="$(find fcu_sim_plugins)/xacro/wind.xacro"/>
+  <!-- <xacro:include filename="$(find fcu_sim_plugins)/xacro/wind.xacro"/>
   <xacro:wind_param
     namespace="${namespace}"
     link_name="${namespace}/base_link"
-    wind_pub_topic="wind"/>
+    wind_pub_topic="wind"/> -->
   <!-- Mount an Altimeter -->
   <xacro:include filename="$(find fcu_sim_plugins)/xacro/altimeter.xacro"/>
@@ -228,3 +228,5 @@
     parent_link="${namespace}/base_link"
     visualize="false"/>
+    <!-- Collision Sensor -->
+    <!-- TODO  http://gazebosim.org/tutorials?tut=contact_sensor-->
 </robot>

File: fcu_sim/urdf/shredder/shredder_base.xacro (robot description, xacro)
@@ -5,56 +5,56 @@
 -->
 <robot name="shredder" xmlns:xacro="http://ros.org/wiki/xacro">
-  <!-- Properties -->
-  <xacro:property name="namespace" value="$(arg mav_name)" />
-  <xacro:property name="rotor_velocity_slowdown_sim" value="10" />
-  <xacro:property name="use_mesh_file" value="true" />
-  <xacro:property name="mesh_file" value="package://fcu_sim/meshes/firefly.dae" />
-  <xacro:property name="mass" value="3.81" /> <!-- [kg] -->
-  <xacro:property name="body_width" value="0.1" /> <!-- [m] -->
-  <xacro:property name="body_height" value="0.16" /> <!-- [m] -->
-  <xacro:property name="mass_rotor" value="0.005" /> <!-- [kg] -->
-  <xacro:property name="arm_length" value="0.3429" /> <!-- [m] -->
-  <xacro:property name="rotor_offset_top" value="0.06985" /> <!-- [m] -->
-  <xacro:property name="radius_rotor" value="0.1524" /> <!-- [m] -->
-  <xacro:property name="motor_constant" value="1.426e-5" /> <!-- [N-s/rad] -->
-  <xacro:property name="moment_constant" value="0.055" /> <!-- [m] -->
-  <xacro:property name="time_constant_up" value="0.0215" /> <!-- [s] -->
-  <xacro:property name="time_constant_down" value="0.0375" /> <!-- [s] -->
-  <xacro:property name="max_rot_velocity" value="1177.89" /> <!-- [rad/s] -->
-  <xacro:property name="sin30" value="0.5" />
-  <xacro:property name="cos30" value="0.866025403784" />
-  <xacro:property name="rotor_drag_coefficient" value="8.06428e-05" />
-  <xacro:property name="rolling_moment_coefficient" value="0.000001" />
-  <xacro:property name="body_inertia">
-    <inertia ixx="0.0347563" ixy="0.0" ixz="0.0" iyy="0.0458929" iyz="0.0" izz="0.0977" />
-  </xacro:property>
-  <xacro:property name="rotor_inertia">
-    <xacro:box_inertia x="${radius_rotor}" y="0.015" z="0.003" mass="${mass_rotor*rotor_velocity_slowdown_sim}" />
-  </xacro:property>
-  <!-- *********************** GAZEBO ROBOT DEFINITION ******************* -->
-  <link name="${namespace}/base_link">
-    <inertial>
-      <mass value="${mass}" />  <!-- [kg] -->
-      <origin xyz="0 0 0" />
-      <xacro:insert_block name="body_inertia" />
-    </inertial>
-    <visual>
-      <origin xyz="0 0 0" rpy="0 0 0" />
-      <geometry>
-        <xacro:if value="${use_mesh_file}">
-          <mesh filename="${mesh_file}" scale="1 1 1" />
-        </xacro:if>
-        <xacro:unless value="${use_mesh_file}">
-          <box size="${body_width} ${body_width} ${body_height}"/> <!-- [m] [m] [m] -->
-        </xacro:unless>
-      </geometry>
-    </visual>
-    <collision>
-      <origin xyz="0 0 0" rpy="0 0 0" />
-      <geometry>
-        <box size="${body_width} ${body_width} ${body_height}" /> <!-- [m] [m] [m] -->
-      </geometry>
-    </collision>
-  </link>
+<!-- Properties -->
+<xacro:property name="namespace" value="mikey" />
+<xacro:property name="rotor_velocity_slowdown_sim" value="10" />
+<xacro:property name="use_mesh_file" value="true" />
+<xacro:property name="mesh_file" value="package://fcu_sim/meshes/firefly.dae" />
+<xacro:property name="mass" value="3.81" /> <!-- [kg] -->
+<xacro:property name="body_width" value="0.505" /> <!-- [m] -->
+<xacro:property name="body_height" value="0.1" /> <!-- [m] -->
+<xacro:property name="mass_rotor" value="0.005" /> <!-- [kg] -->
+<xacro:property name="arm_length" value="0.3429" /> <!-- [m] -->
+<xacro:property name="rotor_offset_top" value="0.06985" /> <!-- [m] -->
+<xacro:property name="radius_rotor" value="0.1524" /> <!-- [m] -->
+<xacro:property name="motor_constant" value="1.426e-5" /> <!-- [N-s/rad] -->
+<xacro:property name="moment_constant" value="0.055" /> <!-- [m] -->
+<xacro:property name="time_constant_up" value="0.0215" /> <!-- [s] -->
+<xacro:property name="time_constant_down" value="0.0375" /> <!-- [s] -->
+<xacro:property name="max_rot_velocity" value="1177.89" /> <!-- [rad/s] -->
+<xacro:property name="sin30" value="0.5" />
+<xacro:property name="cos30" value="0.866025403784" />
+<xacro:property name="rotor_drag_coefficient" value="8.06428e-05" />
+<xacro:property name="rolling_moment_coefficient" value="0.000001" />
+<xacro:property name="body_inertia">
+  <inertia ixx="0.0347563" ixy="0.0" ixz="0.0" iyy="0.0458929" iyz="0.0" izz="0.0977" />
+</xacro:property>
+<xacro:property name="rotor_inertia">
+  <xacro:box_inertia x="${radius_rotor}" y="0.015" z="0.003" mass="${mass_rotor*rotor_velocity_slowdown_sim}" />
+</xacro:property>
+<!-- *********************** GAZEBO ROBOT DEFINITION ******************* -->
+<link name="${namespace}/base_link">
+  <inertial>
+    <mass value="${mass}" />  <!-- [kg] -->
+    <origin xyz="0 0 0" />
+    <xacro:insert_block name="body_inertia" />
+  </inertial>
+  <visual>
+    <origin xyz="0 0 0" rpy="0 0 0" />
+    <geometry>
+      <xacro:if value="${use_mesh_file}">
+        <mesh filename="${mesh_file}" scale="1 1 1" />
+      </xacro:if>
+      <xacro:unless value="${use_mesh_file}">
+        <cylinder length="${body_height}" radius="${body_width}"/>
+      </xacro:unless>
+    </geometry>
+  </visual>
+  <collision>
+    <origin xyz="0 0 0" rpy="0 0 0" />
+    <geometry>
+      <cylinder length="${body_height}" radius="${body_width}"/>
+    </geometry>
+  </collision>
+</link>
   <!-- ************************* ROTOR DYNAMICS ********************** -->
 <!--   <gazebo>

Commit message: fixed rgbd camera xacro, added a yaw arg to launch file

File: fcu_sim/urdf/mikey/mikey_base.xacro (robot description, xacro)
@@ -51,7 +51,7 @@
     </visual>
     <collision>
-      <origin xyz="0 0 0" rpy="0 0 0" />
+      <origin xyz="0 0 ${body_height/2.0}" rpy="0 0 0" />
       <geometry>
-        <cylinder length="${body_height}" radius="${body_width}"/>
+        <cylinder length="${0.1}" radius="${body_width}"/>
       </geometry>
     </collision>
@@ -207,9 +207,9 @@
     imu_topic="imu"/>
   <!--Enable Wind -->
-  <!-- <xacro:include filename="$(find fcu_sim_plugins)/xacro/wind.xacro"/>
+  <xacro:include filename="$(find fcu_sim_plugins)/xacro/wind.xacro"/>
   <xacro:wind_param
     namespace="${namespace}"
     link_name="${namespace}/base_link"
-    wind_pub_topic="wind"/> -->
+    wind_pub_topic="wind"/>
   <!-- Mount an Altimeter -->
   <xacro:include filename="$(find fcu_sim_plugins)/xacro/altimeter.xacro"/>

File: fcu_sim/urdf/shredder/shredder_base.xacro (robot description, xacro)
@@ -6,5 +6,5 @@
 <robot name="shredder" xmlns:xacro="http://ros.org/wiki/xacro">
 <!-- Properties -->
-<xacro:property name="namespace" value="mikey" />
+<xacro:property name="namespace" value="shredder" />
 <xacro:property name="rotor_velocity_slowdown_sim" value="10" />
 <xacro:property name="use_mesh_file" value="true" />
@@ -51,7 +51,7 @@
   </visual>
   <collision>
-    <origin xyz="0 0 0" rpy="0 0 0" />
+    <origin xyz="0 0 ${body_height/2.0}" rpy="0 0 0" />
     <geometry>
-      <cylinder length="${body_height}" radius="${body_width}"/>
+      <cylinder length="${0.1}" radius="${body_width}"/>
     </geometry>
   </collision>
@@ -201,5 +201,5 @@
   <xacro:include filename="$(find fcu_sim_plugins)/xacro/imu.xacro"/>
   <xacro:IMU_ADIS16448
-    namespace=""
+    namespace="${namespace}"
     parent_link="${namespace}/base_link"
     imu_topic="imu"/>
@@ -207,5 +207,5 @@
   <xacro:include filename="$(find fcu_sim_plugins)/xacro/wind.xacro"/>
   <xacro:wind_param
-    namespace=""
+    namespace="${namespace}"
     link_name="${namespace}/base_link"
     wind_pub_topic="wind"/>
@@ -213,5 +213,5 @@
   <xacro:include filename="$(find fcu_sim_plugins)/xacro/altimeter.xacro"/>
   <xacro:Sonar_MB1030
-    namespace=""
+    namespace="${namespace}"
     parent_link="${namespace}/base_link"
     altimeter_topic="altimeter"/>
@@ -219,10 +219,10 @@
   <xacro:include filename="$(find fcu_sim_plugins)/xacro/rgbd.xacro"/>
   <xacro:xtion
-    namespace=""
+    namespace="${namespace}"
     parent_link="${namespace}/base_link"/>
   <!-- Laser Scanner -->
   <xacro:include filename="$(find fcu_sim_plugins)/xacro/laser_scanner.xacro"/>
   <xacro:hokuyo_UTM-30LX
-    namespace=""
+    namespace="${namespace}"
     parent_link="${namespace}/base_link"
     visualize="false"/>

File: fcu_sim_plugins/xacro/rgbd.xacro (robot description, xacro)
@@ -14,9 +14,9 @@
       depth_range="6.5"
       rgb_range=""
-      image_topic="${namespace}/camera/rgb/image_raw"
-      depth_topic="${namespace}/camera/depth/image_raw"
-      image_camera_info_topic="${namespace}/camera/rgb/camera_info"
-      depth_camera_info_topic="${namespace}/camera/depth/camera_info"
-      pointcloud_topic="${namespace}/camera/pointcloud">
+      image_topic="rgb/image_raw"
+      depth_topic="depth/image_raw"
+      image_camera_info_topic="rgb/camera_info"
+      depth_camera_info_topic="depth/camera_info"
+      pointcloud_topic="camera/pointcloud">
       <origin xyz="0.127 0 -0.0889" rpy="0 0 0" /> <!-- for shredder -->
     </xacro:depth_camera>
@@ -71,5 +71,5 @@
           <horizontal_fov>2</horizontal_fov>
           <image>
-            <format>L8</format>
+            <format>R8G8B8</format>
             <width>640</width>
             <height>480</height>

Commit message: HIL may be working

File: fcu_sim/urdf/mikey/mikey_base.xacro (robot description, xacro)
@@ -61,139 +61,6 @@
   </gazebo>
   <!-- ************************* ROTOR DYNAMICS ********************** -->
-<!--   <gazebo>
-    <plugin filename="libfcu_sim_multirotor_base_plugin.so" name="multirotor_base_plugin">
-      <robotNamespace>${namespace}</robotNamespace>
-      <linkName>${namespace}/base_link</linkName>
-      <rotorVelocitySlowdownSim>${rotor_velocity_slowdown_sim}</rotorVelocitySlowdownSim>
-    </plugin>
-  </gazebo> -->
-  <!-- **************** ROTORS ***************** -->
-  <xacro:include filename="$(find fcu_sim_plugins)/xacro/rotor.xacro" />${namespace}/base_link
-  <xacro:vertical_rotor
-    robot_namespace="${namespace}"
-    suffix="front"
-    direction="cw"
-    motor_constant="${motor_constant}"
-    moment_constant="${moment_constant}"
-    parent="${namespace}/base_link"
-    mass_rotor="${mass_rotor}"
-    radius_rotor="${radius_rotor}"
-    time_constant_up="${time_constant_up}"
-    time_constant_down="${time_constant_down}"
-    max_rot_velocity="${max_rot_velocity}"
-    motor_number="0"
-    rotor_drag_coefficient="${rotor_drag_coefficient}"
-    rolling_moment_coefficient="${rolling_moment_coefficient}"
-    color="Red"
-    use_own_mesh="false"
-    mesh="">
-    <origin xyz="${arm_length} 0 ${rotor_offset_top}" rpy="0 0 0" />
-    <xacro:insert_block name="rotor_inertia" />
-  </xacro:vertical_rotor>
-  <xacro:vertical_rotor
-    robot_namespace="${namespace}"
-    suffix="front_left"
-    direction="ccw"
-    motor_constant="${motor_constant}"
-    moment_constant="${moment_constant}"
-    parent="${namespace}/base_link"
-    mass_rotor="${mass_rotor}"
-    radius_rotor="${radius_rotor}"
-    time_constant_up="${time_constant_up}"
-    time_constant_down="${time_constant_down}"
-    max_rot_velocity="${max_rot_velocity}"
-    motor_number="1"
-    rotor_drag_coefficient="${rotor_drag_coefficient}"
-    rolling_moment_coefficient="${rolling_moment_coefficient}"
-    color="Black"
-    use_own_mesh="false"
-    mesh="">
-    <origin xyz="${sin30*arm_length} ${cos30*arm_length} ${rotor_offset_top}" rpy="0 0 0" />
-    <xacro:insert_block name="rotor_inertia" />
-  </xacro:vertical_rotor>
-  <xacro:vertical_rotor
-    robot_namespace="${namespace}"
-    suffix="back_left"
-    direction="cw"
-    motor_constant="${motor_constant}"
-    moment_constant="${moment_constant}"
-    parent="${namespace}/base_link"
-    mass_rotor="${mass_rotor}"
-    radius_rotor="${radius_rotor}"
-    time_constant_up="${time_constant_up}"
-    time_constant_down="${time_constant_down}"
-    max_rot_velocity="${max_rot_velocity}"
-    motor_number="2"
-    rotor_drag_coefficient="${rotor_drag_coefficient}"
-    rolling_moment_coefficient="${rolling_moment_coefficient}"
-    color="Black"
-    use_own_mesh="false"
-    mesh="">
-    <origin xyz="-${sin30*arm_length} ${cos30*arm_length} ${rotor_offset_top}" rpy="0 0 0" />
-    <xacro:insert_block name="rotor_inertia" />
-  </xacro:vertical_rotor>
-  <xacro:vertical_rotor
-    robot_namespace="${namespace}"
-    suffix="back"
-    direction="ccw"
-    motor_constant="${motor_constant}"
-    moment_constant="${moment_constant}"
-    parent="${namespace}/base_link"
-    mass_rotor="${mass_rotor}"
-    radius_rotor="${radius_rotor}"
-    time_constant_up="${time_constant_up}"
-    time_constant_down="${time_constant_down}"
-    max_rot_velocity="${max_rot_velocity}"
-    motor_number="3"
-    rotor_drag_coefficient="${rotor_drag_coefficient}"
-    rolling_moment_coefficient="${rolling_moment_coefficient}"
-    color="Black"
-    use_own_mesh="false"
-    mesh="">
-    <origin xyz="-${arm_length} 0 ${rotor_offset_top}" rpy="0 0 0" />
-    <xacro:insert_block name="rotor_inertia" />
-  </xacro:vertical_rotor>
-  <xacro:vertical_rotor
-    robot_namespace="${namespace}"
-    suffix="right"
-    direction="cw"
-    motor_constant="${motor_constant}"
-    moment_constant="${moment_constant}"
-    parent="${namespace}/base_link"
-    mass_rotor="${mass_rotor}"
-    radius_rotor="${radius_rotor}"
-    time_constant_up="${time_constant_up}"
-    time_constant_down="${time_constant_down}"
-    max_rot_velocity="${max_rot_velocity}"
-    motor_number="4"
-    rotor_drag_coefficient="${rotor_drag_coefficient}"
-    rolling_moment_coefficient="${rolling_moment_coefficient}"
-    color="Black"
-    use_own_mesh="false"
-    mesh="">
-    <origin xyz="-${sin30*arm_length} -${cos30*arm_length} ${rotor_offset_top}" rpy="0 0 0" />
-    <xacro:insert_block name="rotor_inertia" />
-  </xacro:vertical_rotor>
-  <xacro:vertical_rotor
-    robot_namespace="${namespace}"
-    suffix="front_right"
-    direction="ccw"
-    motor_constant="${motor_constant}"
-    moment_constant="${moment_constant}"
-    parent="${namespace}/base_link"
-    mass_rotor="${mass_rotor}"
-    radius_rotor="${radius_rotor}"
-    time_constant_up="${time_constant_up}"
-    time_constant_down="${time_constant_down}"
-    max_rot_velocity="${max_rot_velocity}"
-    motor_number="5"
-    rotor_drag_coefficient="${rotor_drag_coefficient}"
-    rolling_moment_coefficient="${rolling_moment_coefficient}"
-    color="Black"
-    use_own_mesh="false"
-    mesh="">
-    <origin xyz="${sin30*arm_length} -${cos30*arm_length} ${rotor_offset_top}" rpy="0 0 0" />
-    <xacro:insert_block name="rotor_inertia" />
-  </xacro:vertical_rotor>
+  <xacro:include filename="$(find fcu_sim_plugins)/xacro/multirotor_hil.xacro"/>
+  <xacro:mikey_hil namespace="${namespace}" parent_link="${namespace}/base_link"/>
   <!-- ***************** SENSORS ******************* -->
   <!-- Ground Truth -->
@@ -205,5 +72,5 @@
     namespace="${namespace}"
     parent_link="${namespace}/base_link"
-    imu_topic="imu"/>
+    imu_topic="imu/data"/>
   <!--Enable Wind -->
   <xacro:include filename="$(find fcu_sim_plugins)/xacro/wind.xacro"/>

Commit message: got HIL working with naze

File: fcu_sim/urdf/mikey/mikey_base.xacro (robot description, xacro)
@@ -8,7 +8,7 @@
   <xacro:property name="namespace" value="mikey" />
   <xacro:property name="rotor_velocity_slowdown_sim" value="10" />
-  <xacro:property name="use_mesh_file" value="true" />
+  <xacro:property name="use_mesh_file" value="false" />
   <xacro:property name="mesh_file" value="package://fcu_sim/meshes/firefly.dae" />
-  <xacro:property name="mass" value="3.81" /> <!-- [kg] -->
+  <xacro:property name="mass" value="3.562" /> <!-- [kg] -->
   <xacro:property name="body_width" value="0.505" /> <!-- [m] -->
   <xacro:property name="body_height" value="0.1" /> <!-- [m] -->
@@ -29,7 +29,4 @@
     <inertia ixx="0.0347563" ixy="0.0" ixz="0.0" iyy="0.0458929" iyz="0.0" izz="0.0977" />
   </xacro:property>
-  <xacro:property name="rotor_inertia">
-    <xacro:box_inertia x="${radius_rotor}" y="0.015" z="0.003" mass="${mass_rotor*rotor_velocity_slowdown_sim}" />
-  </xacro:property>
   <!-- *********************** GAZEBO ROBOT DEFINITION ******************* -->
   <link name="${namespace}/base_link">
@@ -42,16 +39,16 @@
       <origin xyz="0 0 0" rpy="0 0 0" />
       <geometry>
-        <xacro:if value="${use_mesh_file}">
+        <!-- <xacro:if value="${use_mesh_file}">
           <mesh filename="${mesh_file}" scale="1 1 1" />
         </xacro:if>
-        <xacro:unless value="${use_mesh_file}">
+        <xacro:unless value="${use_mesh_file}"> -->
           <cylinder length="${body_height}" radius="${body_width}"/>
-        </xacro:unless>
+        <!-- </xacro:unless> -->
       </geometry>
     </visual>
     <collision>
-      <origin xyz="0 0 ${body_height/2.0}" rpy="0 0 0" />
+      <origin xyz="0 0 0" rpy="0 0 0" />
       <geometry>
-        <cylinder length="${0.1}" radius="${body_width}"/>
+        <cylinder length="${body_height}" radius="${body_width}"/>
       </geometry>
     </collision>
@@ -74,26 +71,26 @@
     imu_topic="imu/data"/>
   <!--Enable Wind -->
-  <xacro:include filename="$(find fcu_sim_plugins)/xacro/wind.xacro"/>
+  <!-- <xacro:include filename="$(find fcu_sim_plugins)/xacro/wind.xacro"/>
   <xacro:wind_param
     namespace="${namespace}"
     link_name="${namespace}/base_link"
-    wind_pub_topic="wind"/>
+    wind_pub_topic="wind"/> -->
   <!-- Mount an Altimeter -->
-  <xacro:include filename="$(find fcu_sim_plugins)/xacro/altimeter.xacro"/>
+  <!-- <xacro:include filename="$(find fcu_sim_plugins)/xacro/altimeter.xacro"/>
   <xacro:Sonar_MB1030
     namespace="${namespace}"
     parent_link="${namespace}/base_link"
-    altimeter_topic="altimeter"/>
+    altimeter_topic="altimeter"/> -->
   <!-- Mount an RGBD Camera -->
-  <xacro:include filename="$(find fcu_sim_plugins)/xacro/rgbd.xacro"/>
+  <!-- <xacro:include filename="$(find fcu_sim_plugins)/xacro/rgbd.xacro"/>
   <xacro:xtion
     namespace="${namespace}"
-    parent_link="${namespace}/base_link"/>
+    parent_link="${namespace}/base_link"/> -->
   <!-- Laser Scanner -->
-  <xacro:include filename="$(find fcu_sim_plugins)/xacro/laser_scanner.xacro"/>
+  <!-- <xacro:include filename="$(find fcu_sim_plugins)/xacro/laser_scanner.xacro"/>
   <xacro:hokuyo_UTM-30LX
     namespace="${namespace}"
     parent_link="${namespace}/base_link"
-    visualize="false"/>
+    visualize="false"/> -->
     <!-- Collision Sensor -->
     <!-- TODO  http://gazebosim.org/tutorials?tut=contact_sensor-->
