Commit message: fixed some issues with the estimator - gyro scales, stick arming, attitude control channel and MPU6050 Interrupt happening in HIL

File: fcu_sim/urdf/mikey/mikey_base.xacro (robot description, xacro)
@@ -8,5 +8,5 @@
   <xacro:property name="namespace" value="mikey" />
   <xacro:property name="rotor_velocity_slowdown_sim" value="10" />
-  <xacro:property name="use_mesh_file" value="false" />
+  <xacro:property name="use_mesh_file" value="true" />
   <xacro:property name="mesh_file" value="package://fcu_sim/meshes/firefly.dae" />
   <xacro:property name="mass" value="3.562" /> <!-- [kg] -->
@@ -39,10 +39,10 @@
       <origin xyz="0 0 0" rpy="0 0 0" />
       <geometry>
-        <!-- <xacro:if value="${use_mesh_file}">
+        <xacro:if value="${use_mesh_file}">
           <mesh filename="${mesh_file}" scale="1 1 1" />
         </xacro:if>
-        <xacro:unless value="${use_mesh_file}"> -->
+        <xacro:unless value="${use_mesh_file}">
           <cylinder length="${body_height}" radius="${body_width}"/>
-        <!-- </xacro:unless> -->
+        </xacro:unless>
       </geometry>
     </visual>

Commit message: removed stupid old plugins and files

File: fcu_sim/urdf/mikey/mikey_base.xacro (robot description, xacro)
@@ -10,20 +10,7 @@
   <xacro:property name="use_mesh_file" value="true" />
   <xacro:property name="mesh_file" value="package://fcu_sim/meshes/firefly.dae" />
-  <xacro:property name="mass" value="3.562" /> <!-- [kg] -->
-  <xacro:property name="body_width" value="0.505" /> <!-- [m] -->
-  <xacro:property name="body_height" value="0.1" /> <!-- [m] -->
-  <xacro:property name="mass_rotor" value="0.005" /> <!-- [kg] -->
-  <xacro:property name="arm_length" value="0.3429" /> <!-- [m] -->
-  <xacro:property name="rotor_offset_top" value="0.06985" /> <!-- [m] -->
-  <xacro:property name="radius_rotor" value="0.1524" /> <!-- [m] -->
-  <xacro:property name="motor_constant" value="1.426e-5" /> <!-- [N-s/rad] -->
-  <xacro:property name="moment_constant" value="0.055" /> <!-- [m] -->
-  <xacro:property name="time_constant_up" value="0.0215" /> <!-- [s] -->
-  <xacro:property name="time_constant_down" value="0.0375" /> <!-- [s] -->
-  <xacro:property name="max_rot_velocity" value="1177.89" /> <!-- [rad/s] -->
-  <xacro:property name="sin30" value="0.5" />
-  <xacro:property name="cos30" value="0.866025403784" />
-  <xacro:property name="rotor_drag_coefficient" value="8.06428e-05" />
-  <xacro:property name="rolling_moment_coefficient" value="0.000001" />
+  <xacro:property name="mass" value="3.562" />
+  <xacro:property name="body_width" value="0.505" />
+  <xacro:property name="body_height" value="0.1" />
   <xacro:property name="body_inertia">
     <inertia ixx="0.0347563" ixy="0.0" ixz="0.0" iyy="0.0458929" iyz="0.0" izz="0.0977" />
@@ -60,8 +47,8 @@
   <!-- ROSflight_SIL -->
   <xacro:include filename="$(find fcu_sim_plugins)/xacro/ROSflight_SIL.xacro"/>
-  <!-- <xacro:mikey_ROSflight_SIL namespace="${namespace}" parent_link="${namespace}/base_link"/> -->
+  <xacro:mikey_ROSflight_SIL namespace="${namespace}" parent_link="${namespace}/base_link"/>
   <!-- Simplified Dynamics -->
   <xacro:include filename="$(find fcu_sim_plugins)/xacro/multirotor_forces_and_moments.xacro"/>
-  <xacro:mikey_forces_and_moments namespace="${namespace}" parent_link="${namespace}/base_link"/>
+  <!-- <xacro:mikey_forces_and_moments namespace="${namespace}" parent_link="${namespace}/base_link"/> -->
   <!-- ***************** SENSORS ******************* -->
   <!-- Ground Truth -->

File: fcu_sim_plugins/xacro/multirotor_forces_and_moments.xacro (robot description, xacro)
@@ -7,5 +7,5 @@
       params="namespace parent_link">
       <xacro:multirotor_forces_and_moments_macro
-        namespace="${namespace}/aircraft_forces_and_moments"
+        namespace="${namespace}/multirotor_forces_and_moments"
         parent_link="${namespace}/base_link"
         wind_speed_topic="gazebo/wind_speed"
@@ -50,5 +50,5 @@
         alt_I alt_D *inertia *origin">
     <!-- link -->
-    <link name="${namespace}/aircraft_forces_and_moments_link">
+    <link name="${namespace}/multirotor_forces_and_moments_link">
       <inertial>
         <xacro:insert_block name="inertia" />
@@ -57,8 +57,8 @@
     </link>
     <!-- joint -->
-    <joint name="${namespace}/aircraft_forces_and_moments_joint" type="revolute">
+    <joint name="${namespace}/multirotor_forces_and_moments_joint" type="revolute">
       <parent link="${parent_link}" />
       <xacro:insert_block name="origin" />
-      <child link="${namespace}/aircraft_forces_and_moments_link" />
+      <child link="${namespace}/multirotor_forces_and_moments_link" />
       <limit upper="0" lower="0" effort="0" velocity="0" />
     </joint>
@@ -66,5 +66,5 @@
     <gazebo>
       <plugin filename="libfcu_sim_multirotor_forces_and_moments_plugin.so" name="multirotor_forces_and_moments">
-        <linkName>${namespace}/aircraft_forces_and_moments_link</linkName>
+        <linkName>${namespace}/multirotor_forces_and_moments_link</linkName>
         <robotNamespace>${namespace}</robotNamespace>
         <windSpeedTopic>${wind_speed_topic}</windSpeedTopic>

Commit message: controller is working, needs tuning

File: fcu_sim/urdf/mikey/mikey_base.xacro (robot description, xacro)
@@ -57,5 +57,5 @@
   <!-- Mount an IMU -->
   <xacro:include filename="$(find fcu_sim_plugins)/xacro/imu.xacro"/>
-  <xacro:IMU_ADIS16448
+  <xacro:IMU_MPU6050
     namespace="${namespace}"
     parent_link="${namespace}/base_link"

File: fcu_sim_plugins/xacro/ROSflight_SIL.xacro (robot description, xacro)
@@ -3,4 +3,52 @@
   <xacro:property name="pi" value="3.14159265359" />
     <!-- Forces And Moments Plugin -->
+    <xacro:macro
+      name="square_quad"
+      params="namespace parent_link">
+      <xacro:fcu_sim_ROSflight_sil_plugin
+        namespace="${namespace}/hil"
+        parent_link="${namespace}/base_link"
+        wind_speed_topic="gazebo/wind_speed"
+        command_topic="extended_command"
+        parent_frame_id="${parent_link}"
+        mu="1"
+        rotor_max_thrust="14.961"
+        rotor_F1="1.5e-5"
+        rotor_F2="-0.024451"
+        rotor_F3="9.00225"
+        rotor_T1="-2.22e-7"
+        rotor_T2="3.51e-4"
+        rotor_T3="-0.12531"
+        rotor_tau_down="0.1644"
+        rotor_tau_up="0.2164"
+        num_rotors="4"
+        rotor1_distance="0.30"
+        rotor1_angle="2.35619449019"
+        rotor1_direction="1"
+        rotor2_distance="0.30"
+        rotor2_angle="0.78539816339"
+        rotor2_direction="-1"
+        rotor3_distance="0.30"
+        rotor3_angle="-2.35619449019"
+        rotor3_direction="-1"
+        rotor4_distance="0.30"
+        rotor4_angle="-0.78539816339"
+        rotor4_direction="1"
+        rotor5_distance="0"
+        rotor5_angle="0"
+        rotor5_direction="1"
+        rotor6_distance="0"
+        rotor6_angle="0"
+        rotor6_direction="1"
+        rotor7_distance="0"
+        rotor7_angle="0"
+        rotor7_direction="1"
+        rotor8_distance="0"
+        rotor8_angle="0"
+        rotor8_direction="1">
+        <inertia ixx="0.00001" ixy="0.0" ixz="0.0" iyy="0.00001" iyz="0.0" izz="0.00001" />
+        <origin xyz="0.0 0.0 0.0" rpy="0.0 0.0 0.0" />
+      </xacro:fcu_sim_ROSflight_sil_plugin>
+    </xacro:macro>
     <xacro:macro
       name="mikey_ROSflight_SIL"

File: fcu_sim_plugins/xacro/imu.xacro (robot description, xacro)
@@ -3,4 +3,25 @@
   <xacro:property name="pi" value="3.14159265359" />
     <!-- Configure IMU -->
+    <xacro:macro
+      name="perfect_IMU"
+      params="namespace parent_link imu_topic">
+    <xacro:imu_plugin_macro
+      namespace="${namespace}"
+      imu_suffix=""
+      parent_link="${parent_link}"
+      imu_topic="${imu_topic}"
+      mass_imu_sensor="0.0001"
+      gyroscope_noise_density="0.0"
+      gyroscopoe_random_walk="0.0"
+      gyroscope_bias_correlation_time="1000.0"
+      gyroscope_turn_on_bias_sigma="0.000"
+      accelerometer_noise_density="0.000"
+      accelerometer_random_walk="0.000"
+      accelerometer_bias_correlation_time="300.0"
+      accelerometer_turn_on_bias_sigma="0.0">
+      <inertia ixx="0.00001" ixy="0.0" ixz="0.0" iyy="0.00001" iyz="0.0" izz="0.00001" />
+      <origin xyz="0 0 0" rpy="0 0 0" />
+    </xacro:imu_plugin_macro>
+  </xacro:macro>
     <xacro:macro
       name="IMU_ADIS16448"
@@ -15,5 +36,5 @@
       gyroscopoe_random_walk="0.000038785"
       gyroscope_bias_correlation_time="1000.0"
-      gyroscope_turn_on_bias_sigma="0.000"
+      gyroscope_turn_on_bias_sigma="0.0.008"
       accelerometer_noise_density="0.004"
       accelerometer_random_walk="0.006"
@@ -34,5 +55,5 @@
       imu_topic="${imu_topic}"
       mass_imu_sensor="0.015"
-      gyroscope_noise_density="0.0008726646"
+      gyroscope_noise_density="0.008726646"
       gyroscopoe_random_walk="0.000038785"
       gyroscope_bias_correlation_time="1000.0"

File: fcu_sim_plugins/xacro/rgbd.xacro (robot description, xacro)
@@ -13,5 +13,5 @@
       frame_rate="30"
       depth_range="6.5"
-      rgb_range=""
+      rgb_range="100000"
       image_topic="rgb/image_raw"
       depth_topic="depth/image_raw"

Commit message: moved shredder model to new forces_and_moments plugin

File: fcu_sim/urdf/mikey/mikey_base.xacro (robot description, xacro)
@@ -7,5 +7,4 @@
   <!-- Properties -->
   <xacro:property name="namespace" value="mikey" />
-  <xacro:property name="rotor_velocity_slowdown_sim" value="10" />
   <xacro:property name="use_mesh_file" value="true" />
   <xacro:property name="mesh_file" value="package://fcu_sim/meshes/firefly.dae" />

File: fcu_sim/urdf/shredder/shredder_base.xacro (robot description, xacro)
@@ -7,5 +7,4 @@
 <!-- Properties -->
 <xacro:property name="namespace" value="shredder" />
-<xacro:property name="rotor_velocity_slowdown_sim" value="10" />
 <xacro:property name="use_mesh_file" value="true" />
 <xacro:property name="mesh_file" value="package://fcu_sim/meshes/firefly.dae" />
@@ -13,22 +12,7 @@
 <xacro:property name="body_width" value="0.505" /> <!-- [m] -->
 <xacro:property name="body_height" value="0.1" /> <!-- [m] -->
-<xacro:property name="mass_rotor" value="0.005" /> <!-- [kg] -->
-<xacro:property name="arm_length" value="0.3429" /> <!-- [m] -->
-<xacro:property name="rotor_offset_top" value="0.06985" /> <!-- [m] -->
-<xacro:property name="radius_rotor" value="0.1524" /> <!-- [m] -->
-<xacro:property name="motor_constant" value="1.426e-5" /> <!-- [N-s/rad] -->
-<xacro:property name="moment_constant" value="0.055" /> <!-- [m] -->
-<xacro:property name="time_constant_up" value="0.0215" /> <!-- [s] -->
-<xacro:property name="time_constant_down" value="0.0375" /> <!-- [s] -->
-<xacro:property name="max_rot_velocity" value="1177.89" /> <!-- [rad/s] -->
-<xacro:property name="sin30" value="0.5" />
-<xacro:property name="cos30" value="0.866025403784" />
-<xacro:property name="rotor_drag_coefficient" value="8.06428e-05" />
 <xacro:property name="rolling_moment_coefficient" value="0.000001" />
 <xacro:property name="body_inertia">
   <inertia ixx="0.0347563" ixy="0.0" ixz="0.0" iyy="0.0458929" iyz="0.0" izz="0.0977" />
-</xacro:property>
-<xacro:property name="rotor_inertia">
-  <xacro:box_inertia x="${radius_rotor}" y="0.015" z="0.003" mass="${mass_rotor*rotor_velocity_slowdown_sim}" />
 </xacro:property>
 <!-- *********************** GAZEBO ROBOT DEFINITION ******************* -->
@@ -61,137 +45,7 @@
   </gazebo>
   <!-- ************************* ROTOR DYNAMICS ********************** -->
-<!--   <gazebo>
-    <plugin filename="libfcu_sim_multirotor_base_plugin.so" name="multirotor_base_plugin">
-      <robotNamespace>${namespace}</robotNamespace>
-      <linkName>${namespace}/base_link</linkName>
-      <rotorVelocitySlowdownSim>${rotor_velocity_slowdown_sim}</rotorVelocitySlowdownSim>
-    </plugin>
-  </gazebo> -->
-  <!-- **************** ROTORS ***************** -->
-  <xacro:include filename="$(find fcu_sim_plugins)/xacro/rotor.xacro" />
-  <xacro:vertical_rotor
-    robot_namespace="${namespace}"
-    suffix="front"
-    direction="cw"
-    motor_constant="${motor_constant}"
-    moment_constant="${moment_constant}"
-    parent="${namespace}/base_link"
-    mass_rotor="${mass_rotor}"
-    radius_rotor="${radius_rotor}"
-    time_constant_up="${time_constant_up}"
-    time_constant_down="${time_constant_down}"
-    max_rot_velocity="${max_rot_velocity}"
-    motor_number="0"
-    rotor_drag_coefficient="${rotor_drag_coefficient}"
-    rolling_moment_coefficient="${rolling_moment_coefficient}"
-    color="Red"
-    use_own_mesh="false"
-    mesh="">
-    <origin xyz="${arm_length} 0 ${rotor_offset_top}" rpy="0 0 0" />
-    <xacro:insert_block name="rotor_inertia" />
-  </xacro:vertical_rotor>
-  <xacro:vertical_rotor
-    robot_namespace="${namespace}"
-    suffix="front_left"
-    direction="ccw"
-    motor_constant="${motor_constant}"
-    moment_constant="${moment_constant}"
-    parent="${namespace}/base_link"
-    mass_rotor="${mass_rotor}"
-    radius_rotor="${radius_rotor}"
-    time_constant_up="${time_constant_up}"
-    time_constant_down="${time_constant_down}"
-    max_rot_velocity="${max_rot_velocity}"
-    motor_number="1"
-    rotor_drag_coefficient="${rotor_drag_coefficient}"
-    rolling_moment_coefficient="${rolling_moment_coefficient}"
-    color="Black"
-    use_own_mesh="false"
-    mesh="">
-    <origin xyz="${sin30*arm_length} ${cos30*arm_length} ${rotor_offset_top}" rpy="0 0 0" />
-    <xacro:insert_block name="rotor_inertia" />
-  </xacro:vertical_rotor>
-  <xacro:vertical_rotor robot_namespace="${namespace}"
-    suffix="back_left"
-    direction="cw"
-    motor_constant="${motor_constant}"
-    moment_constant="${moment_constant}"
-    parent="${namespace}/base_link"
-    mass_rotor="${mass_rotor}"
-    radius_rotor="${radius_rotor}"
-    time_constant_up="${time_constant_up}"
-    time_constant_down="${time_constant_down}"
-    max_rot_velocity="${max_rot_velocity}"
-    motor_number="2"
-    rotor_drag_coefficient="${rotor_drag_coefficient}"
-    rolling_moment_coefficient="${rolling_moment_coefficient}"
-    color="Black"
-    use_own_mesh="false"
-    mesh="">
-    <origin xyz="-${sin30*arm_length} ${cos30*arm_length} ${rotor_offset_top}" rpy="0 0 0" />
-    <xacro:insert_block name="rotor_inertia" />
-  </xacro:vertical_rotor>
-  <xacro:vertical_rotor robot_namespace="${namespace}"
-    suffix="back"
-    direction="ccw"
-    motor_constant="${motor_constant}"
-    moment_constant="${moment_constant}"
-    parent="${namespace}/base_link"
-    mass_rotor="${mass_rotor}"
-    radius_rotor="${radius_rotor}"
-    time_constant_up="${time_constant_up}"
-    time_constant_down="${time_constant_down}"
-    max_rot_velocity="${max_rot_velocity}"
-    motor_number="3"
-    rotor_drag_coefficient="${rotor_drag_coefficient}"
-    rolling_moment_coefficient="${rolling_moment_coefficient}"
-    color="Black"
-    use_own_mesh="false"
-    mesh="">
-    <origin xyz="-${arm_length} 0 ${rotor_offset_top}" rpy="0 0 0" />
-    <xacro:insert_block name="rotor_inertia" />
-  </xacro:vertical_rotor>
-  <xacro:vertical_rotor
-    robot_namespace="${namespace}"
-    suffix="right"
-    direction="cw"
-    motor_constant="${motor_constant}"
-    moment_constant="${moment_constant}"
-    parent="${namespace}/base_link"
-    mass_rotor="${mass_rotor}"
-    radius_rotor="${radius_rotor}"
-    time_constant_up="${time_constant_up}"
-    time_constant_down="${time_constant_down}"
-    max_rot_velocity="${max_rot_velocity}"
-    motor_number="4"
-    rotor_drag_coefficient="${rotor_drag_coefficient}"
-    rolling_moment_coefficient="${rolling_moment_coefficient}"
-    color="Black"
-    use_own_mesh="false"
-    mesh="">
-    <origin xyz="-${sin30*arm_length} -${cos30*arm_length} ${rotor_offset_top}" rpy="0 0 0" />
-    <xacro:insert_block name="rotor_inertia" />
-  </xacro:vertical_rotor>
-  <xacro:vertical_rotor
-    robot_namespace="${namespace}"
-    suffix="front_right"
-    direction="ccw"
-    motor_constant="${motor_constant}"
-    moment_constant="${moment_constant}"
-    parent="${namespace}/base_link"
-    mass_rotor="${mass_rotor}"
-    radius_rotor="${radius_rotor}"
-    time_constant_up="${time_constant_up}"
-    time_constant_down="${time_constant_down}"
-    max_rot_velocity="${max_rot_velocity}"
-    motor_number="5"
-    rotor_drag_coefficient="${rotor_drag_coefficient}"
-    rolling_moment_coefficient="${rolling_moment_coefficient}"
-    color="Black"
-    use_own_mesh="false"
-    mesh="">
-    <origin xyz="${sin30*arm_length} -${cos30*arm_length} ${rotor_offset_top}" rpy="0 0 0" />
-    <xacro:insert_block name="rotor_inertia" />
-  </xacro:vertical_rotor>
+  <!-- Simplified Dynamics -->
+  <xacro:include filename="$(find fcu_sim_plugins)/xacro/multirotor_forces_and_moments.xacro"/>
+  <xacro:shredder_forces_and_moments namespace="${namespace}" parent_link="${namespace}/base_link"/>
   <!-- ***************** SENSORS ******************* -->
   <!-- Ground Truth -->

File: fcu_sim_plugins/xacro/multirotor_forces_and_moments.xacro (robot description, xacro)
@@ -3,4 +3,43 @@
   <xacro:property name="pi" value="3.14159265359" />
     <!-- Forces And Moments Plugin -->
+    <xacro:macro
+      name="shredder_forces_and_moments"
+      params="namespace parent_link">
+      <xacro:multirotor_forces_and_moments_macro
+        namespace="${namespace}/multirotor_forces_and_moments"
+        parent_link="${namespace}/base_link"
+        wind_speed_topic="gazebo/wind_speed"
+        command_topic="extended_command"
+        parent_frame_id="${parent_link}"
+        mass="3.81"
+        mu="1"
+        max_l="12.542"
+        max_m="12.542"
+        max_n="0.164505"
+        max_F="109.86"
+        tau_up_l="0.1972"
+        tau_up_m="0.1972"
+        tau_up_n="0.1766"
+        tau_up_F="0.1766"
+        tau_down_l="0.1972"
+        tau_down_m="0.1972"
+        tau_down_n="0.2179"
+        tau_down_F="0.2179"
+        roll_P="25.0"
+        roll_I="0.0"
+        roll_D="8.0"
+        pitch_P="25.0"
+        pitch_I="0.0"
+        pitch_D="8.0"
+        yaw_P="10"
+        yaw_I="0.0"
+        yaw_D="0.0"
+        alt_P="16.0"
+        alt_I="5.0"
+        alt_D="32.0">
+        <inertia ixx="0.00001" ixy="0.0" ixz="0.0" iyy="0.00001" iyz="0.0" izz="0.00001" />
+        <origin xyz="0.0 0.0 0.0" rpy="0.0 0.0 0.0" />
+      </xacro:multirotor_forces_and_moments_macro>
+    </xacro:macro>
     <xacro:macro
       name="mikey_forces_and_moments"
@@ -11,5 +50,5 @@
         wind_speed_topic="gazebo/wind_speed"
         command_topic="extended_command"
-        parent_frame_id="airplane"
+        parent_frame_id="${parent_link}"
         mass="3.856"
         mu="1"

Commit message: ROSflight_SIL is now flying wh00t!

File: fcu_sim/urdf/mikey/mikey_base.xacro (robot description, xacro)
@@ -46,8 +46,8 @@
   <!-- ROSflight_SIL -->
   <xacro:include filename="$(find fcu_sim_plugins)/xacro/ROSflight_SIL.xacro"/>
-  <!-- <xacro:mikey_ROSflight_SIL namespace="${namespace}" parent_link="${namespace}/base_link"/> -->
+  <xacro:mikey_ROSflight_SIL namespace="${namespace}" parent_link="${namespace}/base_link" command_topic="command"/>
   <!-- Simplified Dynamics -->
   <xacro:include filename="$(find fcu_sim_plugins)/xacro/multirotor_forces_and_moments.xacro"/>
-  <xacro:mikey_forces_and_moments namespace="${namespace}" parent_link="${namespace}/base_link" command_topic="command"/>
+  <!-- <xacro:mikey_forces_and_moments namespace="${namespace}" parent_link="${namespace}/base_link" command_topic="command"/> -->
   <!-- ***************** SENSORS ******************* -->
   <!-- Ground Truth -->

File: fcu_sim_plugins/xacro/ROSflight_SIL.xacro (robot description, xacro)
@@ -4,10 +4,10 @@
     <xacro:macro
       name="square_quad_SIL"
-      params="namespace parent_link">
+      params="namespace parent_link command_topic">
       <xacro:ROSflight_sil_plugin
-        namespace="${namespace}/hil"
+        namespace="${namespace}"
         parent_link="${namespace}/base_link"
         wind_speed_topic="gazebo/wind_speed"
-        command_topic="extended_command"
+        command_topic="${command_topic}"
         parent_frame_id="${parent_link}"
         linear_mu="1"
@@ -25,14 +25,14 @@
         rotor1_distance="0.30"
         rotor1_angle="2.35619449019"
-        rotor1_direction="1"
+        rotor1_direction="-1"
         rotor2_distance="0.30"
         rotor2_angle="0.78539816339"
-        rotor2_direction="-1"
+        rotor2_direction="1"
         rotor3_distance="0.30"
         rotor3_angle="-2.35619449019"
-        rotor3_direction="-1"
+        rotor3_direction="1"
         rotor4_distance="0.30"
         rotor4_angle="-0.78539816339"
-        rotor4_direction="1"
+        rotor4_direction="-1"
         rotor5_distance="0"
         rotor5_angle="0"
@@ -46,17 +46,14 @@
         rotor8_distance="0"
         rotor8_angle="0"
-        rotor8_direction="1">
-        <inertia ixx="0.00001" ixy="0.0" ixz="0.0" iyy="0.00001" iyz="0.0" izz="0.00001" />
-        <origin xyz="0.0 0.0 0.0" rpy="0.0 0.0 0.0" />
-      </xacro:ROSflight_sil_plugin>
+        rotor8_direction="1"/>
     </xacro:macro>
     <xacro:macro
       name="mikey_ROSflight_SIL"
-      params="namespace parent_link">
+      params="namespace parent_link command_topic">
       <xacro:ROSflight_sil_plugin
-        namespace="${namespace}/hil"
+        namespace="${namespace}"
         parent_link="${namespace}/base_link"
         wind_speed_topic="gazebo/wind_speed"
-        command_topic="extended_command"
+        command_topic="${command_topic}"
         parent_frame_id="${parent_link}"
         linear_mu="1"
@@ -100,8 +97,5 @@
         rotor8_distance="0"
         rotor8_angle="0"
-        rotor8_direction="1">
-        <inertia ixx="0.00001" ixy="0.0" ixz="0.0" iyy="0.00001" iyz="0.0" izz="0.00001" />
-        <origin xyz="0.0 0.0 0.0" rpy="0.0 0.0 0.0" />
-      </xacro:ROSflight_sil_plugin>
+        rotor8_direction="1"/>
     </xacro:macro>
   <!-- Macro to add a generic multirotor forces and moments plugin. -->
@@ -117,16 +111,14 @@
         rotor4_direction rotor5_distance rotor5_angle rotor5_direction rotor6_distance
         rotor6_angle rotor6_direction rotor7_distance rotor7_angle  rotor7_direction
-        rotor8_distance rotor8_angle  rotor8_direction
-        *inertia *origin">
+        rotor8_distance rotor8_angle  rotor8_direction">
     <!-- plugin -->
     <gazebo>
       <plugin filename="libROSflight_sil_plugin.so" name="multirotor_hil">
         <linkName>${parent_link}</linkName>
-        <robotNamespace>${namespace}</robotNamespace>
+        <namespace>${namespace}</namespace>
         <windSpeedTopic>${wind_speed_topic}</windSpeedTopic>
         <commandTopic>${command_topic}</commandTopic>
-        <parentFrameId>${parent_frame_id}</parentFrameId>
-        <mass>${mass}</mass>
-        <linear_mu>${linear_mu}</linear_mu>
+        <parentFrameId>${parent_frame_id}</parentFrameId
+>        <linear_mu>${linear_mu}</linear_mu>
         <angular_mu>${angular_mu}</angular_mu>
         <ground_effect_a>${ground_effect_a}</ground_effect_a>
