Commit message: improved namespacing

File: fcu_sim/urdf/mikey/mikey_base.xacro (robot description, xacro)
@@ -44,10 +44,10 @@
   </gazebo>
   <!-- ************************* ROTOR DYNAMICS ********************** -->
-  <!-- ROSflight_SIL -->
+  <!-- ROSflight_SIL
   <xacro:include filename="$(find fcu_sim_plugins)/xacro/ROSflight_SIL.xacro"/>
-  <xacro:mikey_ROSflight_SIL namespace="${namespace}" parent_link="${namespace}/base_link" command_topic="command"/>
+  <xacro:mikey_ROSflight_SIL namespace="${namespace}" parent_link="${namespace}/base_link" command_topic="command"/> -->
   <!-- Simplified Dynamics -->
   <xacro:include filename="$(find fcu_sim_plugins)/xacro/multirotor_forces_and_moments.xacro"/>
-  <!-- <xacro:mikey_forces_and_moments namespace="${namespace}" parent_link="${namespace}/base_link" command_topic="command"/> -->
+  <xacro:mikey_forces_and_moments namespace="${namespace}" parent_link="${namespace}/base_link" command_topic="command"/>
   <!-- ***************** SENSORS ******************* -->
   <!-- Ground Truth -->

File: fcu_sim_plugins/xacro/rgbd.xacro (robot description, xacro)
@@ -1,4 +1,5 @@
 <?xml version="1.0"?>
 <robot xmlns:xacro="http://ros.org/wiki/xacro">
+  <xacro:property name="pi" value="3.14159265359" />
   <!-- XTION -->
   <xacro:macro
