Commit message: moved urdf folder to agents folder, added global parameters for MAV types, using ROS parameter server instead of SDF parameter server (which makes a lot more sense to me)

File: fcu_sim/agents/mikey/mikey.xacro (robot description, xacro)
@@ -45,9 +45,9 @@
   <!-- ************************* ROTOR DYNAMICS ********************** -->
   <!-- ROSflight_SIL -->
-  <xacro:include filename="$(find fcu_sim_plugins)/xacro/ROSflight_SIL.xacro"/>
-  <xacro:mikey_ROSflight_SIL namespace="${namespace}" parent_link="${namespace}/base_link" command_topic="command"/>
+  <!-- <xacro:include filename="$(find fcu_sim_plugins)/xacro/ROSflight_SIL.xacro"/> -->
+  <!-- <xacro:mikey_ROSflight_SIL namespace="${namespace}" parent_link="${namespace}/base_link" command_topic="command"/> -->
   <!-- Simplified Dynamics -->
   <xacro:include filename="$(find fcu_sim_plugins)/xacro/multirotor_forces_and_moments.xacro"/>
-  <!-- <xacro:mikey_forces_and_moments namespace="${namespace}" parent_link="${namespace}/base_link" command_topic="command"/> -->
+  <xacro:multirotor namespace="${namespace}" parent_link="${namespace}/base_link" command_topic="command"/>
   <!-- ***************** SENSORS ******************* -->
   <!-- Ground Truth -->

File: fcu_sim_plugins/xacro/ROSflight_SIL.xacro (robot description, xacro)
@@ -51,4 +51,5 @@
       name="mikey_ROSflight_SIL"
       params="namespace parent_link command_topic">
+      <xacro:property name="filename" value="$(find fcu_sim_plugins)/xacro/mikey_rotor_configuration.yaml"/>
       <xacro:ROSflight_sil_plugin
         namespace="${namespace}"
@@ -57,59 +58,10 @@
         command_topic="${command_topic}"
         parent_frame_id="${parent_link}"
-        linear_mu="1"
-        angular_mu="0.3"
-        ground_effect_a="-55.3516"
-        ground_effect_b="181.8265"
-        ground_effect_c="-203.9874"
-        ground_effect_d="85.3735"
-        ground_effect_e="-7.6619"
-        rotor_max_thrust="14.961"
-        rotor_F1="1.5e-5"
-        rotor_F2="-0.024451"
-        rotor_F3="9.00225"
-        rotor_T1="-2.22e-7"
-        rotor_T2="3.51e-4"
-        rotor_T3="-0.12531"
-        rotor_tau_down="0.1644"
-        rotor_tau_up="0.2164"
-        num_rotors="4"
-        rotor1_distance="0.28"
-        rotor1_angle="2.3201"
-        rotor1_direction="1"
-        rotor2_distance="0.30"
-        rotor2_angle="0.8736"
-        rotor2_direction="-1"
-        rotor3_distance="0.28"
-        rotor3_angle="-2.3201"
-        rotor3_direction="-1"
-        rotor4_distance="0.30"
-        rotor4_angle="-0.8736"
-        rotor4_direction="1"
-        rotor5_distance="0"
-        rotor5_angle="0"
-        rotor5_direction="1"
-        rotor6_distance="0"
-        rotor6_angle="0"
-        rotor6_direction="1"
-        rotor7_distance="0"
-        rotor7_angle="0"
-        rotor7_direction="1"
-        rotor8_distance="0"
-        rotor8_angle="0"
-        rotor8_direction="1"/>
+        rotor_config_file="${filename}"/>
     </xacro:macro>
   <!-- Macro to add a generic multirotor forces and moments plugin. -->
   <xacro:macro name="ROSflight_sil_plugin"
     params="
-        namespace parent_link wind_speed_topic command_topic parent_frame_id
-        linear_mu angular_mu
-        ground_effect_a ground_effect_b ground_effect_c ground_effect_d ground_effect_e
-        num_rotors rotor_max_thrust rotor_F1 rotor_F2 rotor_F3 rotor_T1 rotor_T2 rotor_T3
-        rotor_tau_down rotor_tau_up  rotor1_distance rotor1_angle
-        rotor1_direction rotor2_distance rotor2_angle rotor2_direction
-        rotor3_distance rotor3_angle rotor3_direction rotor4_distance rotor4_angle
-        rotor4_direction rotor5_distance rotor5_angle rotor5_direction rotor6_distance
-        rotor6_angle rotor6_direction rotor7_distance rotor7_angle  rotor7_direction
-        rotor8_distance rotor8_angle  rotor8_direction">
+        namespace parent_link wind_speed_topic command_topic parent_frame_id rotor_config_file">
     <!-- plugin -->
     <gazebo>
@@ -119,46 +71,6 @@
         <windSpeedTopic>${wind_speed_topic}</windSpeedTopic>
         <commandTopic>${command_topic}</commandTopic>
-        <parentFrameId>${parent_frame_id}</parentFrameId
->        <linear_mu>${linear_mu}</linear_mu>
-        <angular_mu>${angular_mu}</angular_mu>
-        <ground_effect_a>${ground_effect_a}</ground_effect_a>
-        <ground_effect_b>${ground_effect_b}</ground_effect_b>
-        <ground_effect_c>${ground_effect_c}</ground_effect_c>
-        <ground_effect_d>${ground_effect_d}</ground_effect_d>
-        <ground_effect_e>${ground_effect_e}</ground_effect_e>
-        <numRotors>${num_rotors}</numRotors>
-        <rotorMaxThrust>${rotor_max_thrust}</rotorMaxThrust>
-        <rotorF1>${rotor_F1}</rotorF1>
-        <rotorF2>${rotor_F2}</rotorF2>
-        <rotorF3>${rotor_F3}</rotorF3>
-        <rotorT1>${rotor_T1}</rotorT1>
-        <rotorT2>${rotor_T2}</rotorT2>
-        <rotorT3>${rotor_T3}</rotorT3>
-        <rotorTauDown>${rotor_tau_down}</rotorTauDown>
-        <rotorTauUp>${rotor_tau_up}</rotorTauUp>
-        <rotor1Distance>${rotor1_distance}</rotor1Distance>
-        <rotor1Angle>${rotor1_angle}</rotor1Angle>
-        <rotor1Direction>${rotor1_direction}</rotor1Direction>
-        <rotor2Distance>${rotor2_distance}</rotor2Distance>
-        <rotor2Angle>${rotor2_angle}</rotor2Angle>
-        <rotor2Direction>${rotor2_direction}</rotor2Direction>
-        <rotor3Distance>${rotor3_distance}</rotor3Distance>
-        <rotor3Angle>${rotor3_angle}</rotor3Angle>
-        <rotor3Direction>${rotor3_direction}</rotor3Direction>
-        <rotor4Distance>${rotor4_distance}</rotor4Distance>
-        <rotor4Angle>${rotor4_angle}</rotor4Angle>
-        <rotor4Direction>${rotor4_direction}</rotor4Direction>
-        <rotor5Distance>${rotor5_distance}</rotor5Distance>
-        <rotor5Angle>${rotor5_angle}</rotor5Angle>
-        <rotor5Direction>${rotor5_direction}</rotor5Direction>
-        <rotor6Distance>${rotor6_distance}</rotor6Distance>
-        <rotor6Angle>${rotor6_angle}</rotor6Angle>
-        <rotor6Direction>${rotor6_direction}</rotor6Direction>
-        <rotor7Distance>${rotor7_distance}</rotor7Distance>
-        <rotor7Angle>${rotor7_angle}</rotor7Angle>
-        <rotor7Direction>${rotor7_direction}</rotor7Direction>
-        <rotor8Distance>${rotor8_distance}</rotor8Distance>
-        <rotor8Angle>${rotor8_angle}</rotor8Angle>
-        <rotor8Direction>${rotor8_direction}</rotor8Direction>
+        <parentFrameId>${parent_frame_id}</parentFrameId>
+        <configFilename>${rotor_config_file}</configFilename>
       </plugin>
     </gazebo>

File: fcu_sim_plugins/xacro/aircraft_forces_and_moments.xacro (robot description, xacro)
@@ -10,92 +10,10 @@
         wind_speed_topic="gazebo/wind_speed"
         command_topic="${command_topic}"
-        parent_frame_id="${namespace}/base_link"
-        mass="1.5"
-        Jx="0.8244"
-        Jy="1.135"
-        Jz="1.759"
-        Jxz=".1204"
-        rho="1.2682"
-        wing_s="0.55"
-        wing_b="2.8956"
-        wing_c="0.18994"
-        wing_M="0.55"
-        wing_epsilon="2.8956"
-        wing_alpha0="0.18994"
-        k_motor="80.0"
-        k_T_P="0.0"
-        k_Omega="0.0"
-        prop_e="0.9"
-        prop_S="0.202"
-        prop_C="1.0"
-        C_L_O="0.28"
-        C_L_alpha="3.45"
-        C_L_beta="0.0"
-        C_L_p="0.0"
-        C_L_q="0.0"
-        C_L_r="0.0"
-        C_L_delta_a="0.0"
-        C_L_delta_e="-0.36"
-        C_L_delta_r="0.0"
-        C_D_O="0.03"
-        C_D_alpha="0.30"
-        C_D_beta="0.0"
-        C_D_p="0.0437"
-        C_D_q="0.0"
-        C_D_r="0.0"
-        C_D_delta_a="0.0"
-        C_D_delta_e="0.0"
-        C_D_delta_r="0.0"
-        C_ell_O="0.0"
-        C_ell_alpha="0.00"
-        C_ell_beta="-0.12"
-        C_ell_p="-0.26"
-        C_ell_q="0.0"
-        C_ell_r="0.14"
-        C_ell_delta_a="0.08"
-        C_ell_delta_e="0.0"
-        C_ell_delta_r="0.105"
-        C_m_O="-0.02338"
-        C_m_alpha="-0.38"
-        C_m_beta="0.0"
-        C_m_p="0.0"
-        C_m_q="-3.6"
-        C_m_r="0.0"
-        C_m_delta_a="0.0"
-        C_m_delta_e="-0.5"
-        C_m_delta_r="0.0"
-        C_n_O="0.0"
-        C_n_alpha="0.0"
-        C_n_beta="0.25"
-        C_n_p="0.022"
-        C_n_q="0.0"
-        C_n_r="-0.35"
-        C_n_delta_a="0.06"
-        C_n_delta_e="0.0"
-        C_n_delta_r="-0.032"
-        C_Y_O="0.0"
-        C_Y_alpha="0.00"
-        C_Y_beta="-0.98"
-        C_Y_p="0.0"
-        C_Y_q="0.0"
-        C_Y_r="0.0"
-        C_Y_delta_a="0.0"
-        C_Y_delta_e="0.0"
-        C_Y_delta_r="-0.017">
+        parent_frame_id="${namespace}/base_link">
       </xacro:aircraft_forces_and_moments_macro>
     </xacro:macro>
   <!-- Macro to add a generic odometry sensor. -->
   <xacro:macro name="aircraft_forces_and_moments_macro"
-    params="
-        namespace  parent_link wind_speed_topic command_topic parent_frame_id
-        mass Jx Jy Jz Jxz rho wing_s wing_b wing_c wing_M wing_epsilon
-        wing_alpha0 k_motor k_T_P k_Omega prop_e prop_S prop_C C_L_O C_L_alpha
-        C_L_beta C_L_p C_L_q C_L_r C_L_delta_a C_L_delta_e C_L_delta_r C_D_O
-        C_D_alpha C_D_beta C_D_p C_D_q C_D_r C_D_delta_a C_D_delta_e C_D_delta_r
-        C_ell_O C_ell_alpha C_ell_beta C_ell_p C_ell_q C_ell_r C_ell_delta_a
-        C_ell_delta_e C_ell_delta_r C_m_O C_m_alpha C_m_beta C_m_p C_m_q C_m_r
-        C_m_delta_a C_m_delta_e C_m_delta_r C_n_O C_n_alpha C_n_beta C_n_p C_n_q
-        C_n_r C_n_delta_a C_n_delta_e C_n_delta_r C_Y_O C_Y_alpha C_Y_beta C_Y_p
-        C_Y_q C_Y_r C_Y_delta_a C_Y_delta_e C_Y_delta_r">
+    params="namespace  parent_link wind_speed_topic command_topic parent_frame_id">
     <gazebo>
       <plugin
@@ -107,76 +25,4 @@
         <commandTopic>${command_topic}</commandTopic>
         <parentFrameId>${parent_frame_id}</parentFrameId>
-        <mass>${mass}</mass>
-        <Jx>${Jx}</Jx>
-        <Jy>${Jy}</Jy>
-        <Jz>${Jz}</Jz>
-        <Jxz>${Jxz}</Jxz>
-        <rho>${rho}</rho>
-        <wing_s>${wing_s}</wing_s>
-        <wing_b>${wing_b}</wing_b>
-        <wing_c>${wing_c}</wing_c>
-        <wing_M>${wing_M}</wing_M>
-        <wing_epsilon>${wing_epsilon}</wing_epsilon>
-        <wing_alpha0>${wing_alpha0}</wing_alpha0>
-        <k_motor>${k_motor}</k_motor>
-        <k_T_P>${k_T_P}</k_T_P>
-        <k_Omega>${k_Omega}</k_Omega>
-        <prop_e>${prop_e}</prop_e>
-        <prop_S>${prop_S}</prop_S>
-        <prop_C>${prop_C}</prop_C>
-        <C_L_O>${C_L_O}</C_L_O>
-        <C_L_alpha>${C_L_alpha}</C_L_alpha>
-        <C_L_beta>${C_L_beta}</C_L_beta>
-        <C_L_p>${C_L_p}</C_L_p>
-        <C_L_q>${C_L_q}</C_L_q>
-        <C_L_r>${C_L_r}</C_L_r>
-        <C_L_delta_a>${C_L_delta_a}</C_L_delta_a>
-        <C_L_delta_e>${C_L_delta_e}</C_L_delta_e>
-        <C_L_delta_r>${C_L_delta_r}</C_L_delta_r>
-        <C_D_O>${C_D_O}</C_D_O>
-        <C_D_alpha>${C_D_alpha}</C_D_alpha>
-        <C_D_beta>${C_D_beta}</C_D_beta>
-        <C_D_p>${C_D_p}</C_D_p>
-        <C_D_q>${C_D_q}</C_D_q>
-        <C_D_r>${C_D_r}</C_D_r>
-        <C_D_delta_a>${C_D_delta_a}</C_D_delta_a>
-        <C_D_delta_e>${C_D_delta_e}</C_D_delta_e>
-        <C_D_delta_r>${C_D_delta_r}</C_D_delta_r>
-        <C_ell_O>${C_ell_O}</C_ell_O>
-        <C_ell_alpha>${C_ell_alpha}</C_ell_alpha>
-        <C_ell_beta>${C_ell_beta}</C_ell_beta>
-        <C_ell_p>${C_ell_p}</C_ell_p>
-        <C_ell_q>${C_ell_q}</C_ell_q>
-        <C_ell_r>${C_ell_r}</C_ell_r>
-        <C_ell_delta_a>${C_ell_delta_a}</C_ell_delta_a>
-        <C_ell_delta_e>${C_ell_delta_e}</C_ell_delta_e>
-        <C_ell_delta_r>${C_ell_delta_r}</C_ell_delta_r>
-        <C_m_O>${C_m_O}</C_m_O>
-        <C_m_alpha>${C_m_alpha}</C_m_alpha>
-        <C_m_beta>${C_m_beta}</C_m_beta>
-        <C_m_p>${C_m_p}</C_m_p>
-        <C_m_q>${C_m_q}</C_m_q>
-        <C_m_r>${C_m_r}</C_m_r>
-        <C_m_delta_a>${C_m_delta_a}</C_m_delta_a>
-        <C_m_delta_e>${C_m_delta_e}</C_m_delta_e>
-        <C_m_delta_r>${C_m_delta_r}</C_m_delta_r>
-        <C_n_O>${C_n_O}</C_n_O>
-        <C_n_alpha>${C_n_alpha}</C_n_alpha>
-        <C_n_beta>${C_n_beta}</C_n_beta>
-        <C_n_p>${C_n_p}</C_n_p>
-        <C_n_q>${C_n_q}</C_n_q>
-        <C_n_r>${C_n_r}</C_n_r>
-        <C_n_delta_a>${C_n_delta_a}</C_n_delta_a>
-        <C_n_delta_e>${C_n_delta_e}</C_n_delta_e>
-        <C_n_delta_r>${C_n_delta_r}</C_n_delta_r>
-        <C_Y_O>${C_Y_O}</C_Y_O>
-        <C_Y_alpha>${C_Y_alpha}</C_Y_alpha>
-        <C_Y_beta>${C_Y_beta}</C_Y_beta>
-        <C_Y_p>${C_Y_p}</C_Y_p>
-        <C_Y_q>${C_Y_q}</C_Y_q>
-        <C_Y_r>${C_Y_r}</C_Y_r>
-        <C_Y_delta_a>${C_Y_delta_a}</C_Y_delta_a>
-        <C_Y_delta_e>${C_Y_delta_e}</C_Y_delta_e>
-        <C_Y_delta_r>${C_Y_delta_r}</C_Y_delta_r>
       </plugin>
     </gazebo>

File: fcu_sim_plugins/xacro/multirotor_forces_and_moments.xacro (robot description, xacro)
@@ -3,5 +3,5 @@
     <!-- Forces And Moments Plugin -->
     <xacro:macro
-      name="shredder_forces_and_moments"
+      name="multirotor"
       params="namespace parent_link command_topic">
       <xacro:multirotor_forces_and_moments_macro
@@ -10,75 +10,10 @@
         wind_speed_topic="gazebo/wind_speed"
         command_topic="${command_topic}"
-        parent_frame_id="${parent_link}"
-        mass="3.81"
-        mu="0.01"
-        max_l="12.542"
-        max_m="12.542"
-        max_n="0.4505"
-        max_F="109.86"
-        tau_up_l="0.1972"
-        tau_up_m="0.1972"
-        tau_up_n="0.1766"
-        tau_up_F="0.1766"
-        tau_down_l="0.1972"
-        tau_down_m="0.1972"
-        tau_down_n="0.2179"
-        tau_down_F="0.2179"
-        roll_P="25.0"
-        roll_I="0.0"
-        roll_D="8.0"
-        pitch_P="25.0"
-        pitch_I="0.0"
-        pitch_D="8.0"
-        yaw_P="90"
-        yaw_I="0.0"
-        yaw_D="0.0"
-        alt_P="16.0"
-        alt_I="5.0"
-        alt_D="32.0"/>
-    </xacro:macro>
-    <xacro:macro
-      name="mikey_forces_and_moments"
-      params="namespace parent_link command_topic">
-      <xacro:multirotor_forces_and_moments_macro
-        namespace="${namespace}"
-        parent_link="${namespace}/base_link"
-        wind_speed_topic="gazebo/wind_speed"
-        command_topic="${command_topic}"
-        parent_frame_id="${parent_link}"
-        mass="3.856"
-        mu="1"
-        max_l="6.5080"
-        max_m="5.087"
-        max_n="0.099828"
-        max_F="59.844"
-        tau_up_l="0.1904"
-        tau_up_m="0.1904"
-        tau_up_n="0.1644"
-        tau_up_F="0.1644"
-        tau_down_l="0.1904"
-        tau_down_m="0.1904"
-        tau_down_n="0.2164"
-        tau_down_F="0.2164"
-        roll_P="25.0"
-        roll_I="0.0"
-        roll_D="8.0"
-        pitch_P="25.0"
-        pitch_I="0.0"
-        pitch_D="8.0"
-        yaw_P="10"
-        yaw_I="0.0"
-        yaw_D="0.0"
-        alt_P="16.0"
-        alt_I="5.0"
-        alt_D="32.0"/>
+        parent_frame_id="${parent_link}"/>
     </xacro:macro>
   <!-- Macro to add a generic multirotor forces and moments plugin. -->
   <xacro:macro name="multirotor_forces_and_moments_macro"
     params="
-        namespace parent_link wind_speed_topic command_topic parent_frame_id mass
-        mu max_l max_m max_n max_F tau_up_l tau_up_m tau_up_n tau_up_F tau_down_l tau_down_m
-        tau_down_n tau_down_F roll_P roll_I roll_D pitch_P pitch_I pitch_D yaw_P yaw_I yaw_D alt_P
-        alt_I alt_D">
+        namespace parent_link wind_speed_topic command_topic parent_frame_id">
     <!-- plugin -->
     <gazebo>
@@ -89,30 +24,4 @@
         <commandTopic>${command_topic}</commandTopic>
         <parentFrameId>${parent_frame_id}</parentFrameId>
-        <mass>${mass}</mass>
-        <mu>${mu}</mu>
-        <max_l>${max_l}</max_l>
-        <max_m>${max_m}</max_m>
-        <max_n>${max_n}</max_n>
-        <max_F>${max_F}</max_F>
-        <tau_up_l>${tau_up_l}</tau_up_l>
-        <tau_up_m>${tau_up_m}</tau_up_m>
-        <tau_up_n>${tau_up_n}</tau_up_n>
-        <tau_up_F>${tau_up_F}</tau_up_F>
-        <tau_down_l>${tau_down_l}</tau_down_l>
-        <tau_down_m>${tau_down_m}</tau_down_m>
-        <tau_down_n>${tau_down_n}</tau_down_n>
-        <tau_down_F>${tau_down_F}</tau_down_F>
-        <roll_P>${roll_P}</roll_P>
-        <roll_I>${roll_I}</roll_I>
-        <roll_D>${roll_D}</roll_D>
-        <pitch_P>${pitch_P}</pitch_P>
-        <pitch_I>${pitch_I}</pitch_I>
-        <pitch_D>${pitch_D}</pitch_D>
-        <yaw_P>${yaw_P}</yaw_P>
-        <yaw_I>${yaw_I}</yaw_I>
-        <yaw_D>${yaw_D}</yaw_D>
-        <alt_P>${alt_P}</alt_P>
-        <alt_I>${alt_I}</alt_I>
-        <alt_D>${alt_D}</alt_D>
       </plugin>
     </gazebo>

Commit message: cleaned up commented code in odometry, got rid of initialization lists that were confusing qtcreator

File: fcu_sim/agents/mikey/mikey.xacro (robot description, xacro)
@@ -9,5 +9,5 @@
   <xacro:property name="use_mesh_file" value="true" />
   <xacro:property name="mesh_file" value="package://fcu_sim/meshes/firefly.dae" />
-  <xacro:property name="mass" value="3.562" />
+  <xacro:property name="mass" value="2.856" />
   <xacro:property name="body_width" value="0.505" />
   <xacro:property name="body_height" value="0.1" />

Commit message: cleaned up laser scanner a bit, also added Reset to IMU, didn't solve the break on reset problem

File: fcu_sim/agents/mikey/mikey.xacro (robot description, xacro)
@@ -55,9 +55,10 @@
   <xacro:ground_truth namespace="${namespace}" parent_link="${namespace}/base_link" />
   <!-- Mount an IMU -->
-  <xacro:include filename="$(find fcu_sim_plugins)/xacro/imu.xacro"/>
+<!--   <xacro:include filename="$(find fcu_sim_plugins)/xacro/imu.xacro"/>
   <xacro:IMU_MPU6050
     namespace="${namespace}"
     parent_link="${namespace}/base_link"
     imu_topic="imu/data"/>
+ -->
   <!--Enable Wind -->
   <!-- <xacro:include filename="$(find fcu_sim_plugins)/xacro/wind.xacro"/>
@@ -78,9 +79,11 @@
     parent_link="${namespace}/base_link"/>
   <!-- Laser Scanner -->
-  <!-- <xacro:include filename="$(find fcu_sim_plugins)/xacro/laser_scanner.xacro"/>
-  <xacro:hokuyo_UTM-30LX
+  <xacro:include filename="$(find fcu_sim_plugins)/xacro/laser_scanner.xacro"/>
+  <xacro:RPLIDAR-A2
     namespace="${namespace}"
     parent_link="${namespace}/base_link"
-    visualize="false"/> -->
+    visualize="false">
+    <origin xyz="0.0 0.0 0.2" rpy="0 0 0" />
+  </xacro:RPLIDAR-A2>
     <!-- Collision Sensor -->
     <!-- TODO  http://gazebosim.org/tutorials?tut=contact_sensor-->

File: fcu_sim_plugins/xacro/laser_scanner.xacro (robot description, xacro)
@@ -19,4 +19,25 @@
       update_rate="40">
       <origin xyz="0.09525 0 -0.0127" rpy="0 0 0" />
+    </xacro:laser_scanner>
+  </xacro:macro>
+    <!-- RPLIDAR-A2 -->
+  <xacro:macro
+    name="RPLIDAR-A2"
+    params="namespace
+            parent_link
+            visualize
+            *origin">
+    <xacro:laser_scanner
+      namespace="${namespace}"
+      parent_link="${parent_link}"
+      num_samples="400"
+      visualize="${visualize}"
+      min_range="0.15"
+      max_range="6"
+      res_range="0.01"
+      min_angle="-3.14159"
+      max_angle="3.14159"
+      update_rate="10">
+      <xacro:insert_block name="origin"/>
     </xacro:laser_scanner>
   </xacro:macro>
@@ -64,6 +85,6 @@
             <samples>720</samples>
             <resolution>1</resolution>
-            <min_angle>-1.570796</min_angle>
-            <max_angle>1.570796</max_angle>
+            <min_angle>${min_angle}</min_angle>
+            <max_angle>${max_angle}</max_angle>
           </horizontal>
         </scan>
@@ -80,6 +101,6 @@
       </ray>
       <plugin name="${namespace}_laser" filename="libgazebo_ros_laser.so">
-        <topicName>scan</topicName>
-        <frameName>laser_link</frameName>
+        <topicName>${namespace}/scan</topicName>
+        <frameName>${namespace}/base_laser_link</frameName>
       </plugin>
     </sensor>
