Commit message: got ROSflight_SIL working

File: fcu_sim/agents/mikey/mikey.xacro (robot description, xacro)
@@ -44,10 +44,11 @@
   </gazebo>
   <!-- ************************* ROTOR DYNAMICS ********************** -->
-  <!-- ROSflight_SIL
+  <!-- ROSflight_SIL -->
   <xacro:include filename="$(find fcu_sim_plugins)/xacro/ROSflight_SIL.xacro"/>
-  <xacro:mikey_ROSflight_SIL namespace="${namespace}" parent_link="${namespace}/base_link" command_topic="command"/> -->
+  <xacro:mikey_ROSflight_SIL namespace="${namespace}" parent_link="${namespace}/base_link" command_topic="command"/>
   <!-- Simplified Dynamics -->
-  <xacro:include filename="$(find fcu_sim_plugins)/xacro/multirotor_forces_and_moments.xacro"/>
+<!--   <xacro:include filename="$(find fcu_sim_plugins)/xacro/multirotor_forces_and_moments.xacro"/>
   <xacro:multirotor namespace="${namespace}" parent_link="${namespace}/base_link" command_topic="command"/>
+ -->
   <!-- ***************** SENSORS ******************* -->
   <!-- Ground Truth -->
@@ -55,10 +56,9 @@
   <xacro:ground_truth namespace="${namespace}" parent_link="${namespace}/base_link" />
   <!-- Mount an IMU -->
-<!--   <xacro:include filename="$(find fcu_sim_plugins)/xacro/imu.xacro"/>
+  <xacro:include filename="$(find fcu_sim_plugins)/xacro/imu.xacro"/>
   <xacro:IMU_MPU6050
     namespace="${namespace}"
     parent_link="${namespace}/base_link"
     imu_topic="imu/data"/>
- -->
   <!--Enable Wind -->
   <!-- <xacro:include filename="$(find fcu_sim_plugins)/xacro/wind.xacro"/>

File: fcu_sim_plugins/xacro/ROSflight_SIL.xacro (robot description, xacro)
@@ -10,46 +10,9 @@
         wind_speed_topic="gazebo/wind_speed"
         command_topic="${command_topic}"
-        parent_frame_id="${parent_link}"
-        linear_mu="1"
-        angular_mu="0.3"
-        rotor_max_thrust="14.961"
-        rotor_F1="1.5e-5"
-        rotor_F2="-0.024451"
-        rotor_F3="9.00225"
-        rotor_T1="-2.22e-7"
-        rotor_T2="3.51e-4"
-        rotor_T3="-0.12531"
-        rotor_tau_down="0.1644"
-        rotor_tau_up="0.2164"
-        num_rotors="4"
-        rotor1_distance="0.30"
-        rotor1_angle="2.35619449019"
-        rotor1_direction="-1"
-        rotor2_distance="0.30"
-        rotor2_angle="0.78539816339"
-        rotor2_direction="1"
-        rotor3_distance="0.30"
-        rotor3_angle="-2.35619449019"
-        rotor3_direction="1"
-        rotor4_distance="0.30"
-        rotor4_angle="-0.78539816339"
-        rotor4_direction="-1"
-        rotor5_distance="0"
-        rotor5_angle="0"
-        rotor5_direction="1"
-        rotor6_distance="0"
-        rotor6_angle="0"
-        rotor6_direction="1"
-        rotor7_distance="0"
-        rotor7_angle="0"
-        rotor7_direction="1"
-        rotor8_distance="0"
-        rotor8_angle="0"
-        rotor8_direction="1"/>
+        parent_frame_id="${parent_link}"/>
     </xacro:macro>
     <xacro:macro
       name="mikey_ROSflight_SIL"
       params="namespace parent_link command_topic">
-      <xacro:property name="filename" value="$(find fcu_sim_plugins)/xacro/mikey_rotor_configuration.yaml"/>
       <xacro:ROSflight_sil_plugin
         namespace="${namespace}"
@@ -57,11 +20,10 @@
         wind_speed_topic="gazebo/wind_speed"
         command_topic="${command_topic}"
-        parent_frame_id="${parent_link}"
-        rotor_config_file="${filename}"/>
+        parent_frame_id="${parent_link}"/>
     </xacro:macro>
   <!-- Macro to add a generic multirotor forces and moments plugin. -->
   <xacro:macro name="ROSflight_sil_plugin"
     params="
-        namespace parent_link wind_speed_topic command_topic parent_frame_id rotor_config_file">
+        namespace parent_link wind_speed_topic command_topic parent_frame_id">
     <!-- plugin -->
     <gazebo>
@@ -72,5 +34,4 @@
         <commandTopic>${command_topic}</commandTopic>
         <parentFrameId>${parent_frame_id}</parentFrameId>
-        <configFilename>${rotor_config_file}</configFilename>
       </plugin>
     </gazebo>

Commit message: tested and working, removed debug and added some comments

File: fcu_sim/agents/mikey/mikey.xacro (robot description, xacro)
@@ -1,5 +1,5 @@
 <?xml version="1.0"?>
 <!--
-Gazebo Shredder Definition File
+Gazebo Multirotor Definition File
 Author: James Jackson
 -->
@@ -13,5 +13,5 @@
   <xacro:property name="body_height" value="0.1" />
   <xacro:property name="body_inertia">
-    <inertia ixx="0.0347563" ixy="0.0" ixz="0.0" iyy="0.0458929" iyz="0.0" izz="0.0977" />
+    <inertia ixx="0.07" ixy="0.0" ixz="0.0" iyy="0.08" iyz="0.0" izz="0.12" />
   </xacro:property>
   <!-- *********************** GAZEBO ROBOT DEFINITION ******************* -->
@@ -43,5 +43,5 @@
     <material>Gazebo/$(arg color)</material>
   </gazebo>
-  <!-- ************************* ROTOR DYNAMICS ********************** -->
+  <!-- ************************* FORCES AND MOMENTS ********************** -->
   <!-- ROSflight_SIL -->
   <xacro:include filename="$(find fcu_sim_plugins)/xacro/ROSflight_SIL.xacro"/>
@@ -49,6 +49,5 @@
   <!-- Simplified Dynamics -->
 <!--   <xacro:include filename="$(find fcu_sim_plugins)/xacro/multirotor_forces_and_moments.xacro"/>
-  <xacro:multirotor namespace="${namespace}" parent_link="${namespace}/base_link" command_topic="command"/>
- -->
+  <xacro:multirotor namespace="${namespace}" parent_link="${namespace}/base_link" command_topic="command"/> -->
   <!-- ***************** SENSORS ******************* -->
   <!-- Ground Truth -->
@@ -57,20 +56,20 @@
   <!-- Mount an IMU -->
   <xacro:include filename="$(find fcu_sim_plugins)/xacro/imu.xacro"/>
-  <xacro:IMU_MPU6050
+  <xacro:perfect_IMU
     namespace="${namespace}"
     parent_link="${namespace}/base_link"
     imu_topic="imu/data"/>
   <!--Enable Wind -->
-  <!-- <xacro:include filename="$(find fcu_sim_plugins)/xacro/wind.xacro"/>
+  <xacro:include filename="$(find fcu_sim_plugins)/xacro/wind.xacro"/>
   <xacro:wind_param
     namespace="${namespace}"
     link_name="${namespace}/base_link"
-    wind_pub_topic="wind"/> -->
+    wind_pub_topic="wind"/>
   <!-- Mount an Altimeter -->
-  <!-- <xacro:include filename="$(find fcu_sim_plugins)/xacro/altimeter.xacro"/>
+  <xacro:include filename="$(find fcu_sim_plugins)/xacro/altimeter.xacro"/>
   <xacro:Sonar_MB1030
     namespace="${namespace}"
     parent_link="${namespace}/base_link"
-    altimeter_topic="altimeter"/> -->
+    altimeter_topic="altimeter"/>
   <!-- Mount an RGBD Camera -->
   <xacro:include filename="$(find fcu_sim_plugins)/xacro/rgbd.xacro"/>

Commit message: fixed sonar

File: fcu_sim/agents/mikey/mikey.xacro (robot description, xacro)
@@ -46,8 +46,8 @@
   <!-- ROSflight_SIL -->
   <xacro:include filename="$(find fcu_sim_plugins)/xacro/ROSflight_SIL.xacro"/>
-  <xacro:mikey_ROSflight_SIL namespace="${namespace}" parent_link="${namespace}/base_link" command_topic="command"/>
+  <!-- <xacro:mikey_ROSflight_SIL namespace="${namespace}" parent_link="${namespace}/base_link" command_topic="command"/> -->
   <!-- Simplified Dynamics -->
-<!--   <xacro:include filename="$(find fcu_sim_plugins)/xacro/multirotor_forces_and_moments.xacro"/>
-  <xacro:multirotor namespace="${namespace}" parent_link="${namespace}/base_link" command_topic="command"/> -->
+  <xacro:include filename="$(find fcu_sim_plugins)/xacro/multirotor_forces_and_moments.xacro"/>
+  <xacro:multirotor namespace="${namespace}" parent_link="${namespace}/base_link" command_topic="command"/>
   <!-- ***************** SENSORS ******************* -->
   <!-- Ground Truth -->
@@ -67,9 +67,11 @@
     wind_pub_topic="wind"/>
   <!-- Mount an Altimeter -->
-  <xacro:include filename="$(find fcu_sim_plugins)/xacro/altimeter.xacro"/>
+  <xacro:include filename="$(find fcu_sim_plugins)/xacro/sonar.xacro"/>
   <xacro:Sonar_MB1030
     namespace="${namespace}"
     parent_link="${namespace}/base_link"
-    altimeter_topic="altimeter"/>
+    sonar_topic="alt">
+    <origin xyz="0.4 0.1 -0.21" rpy="0 0 0" />
+  </xacro:Sonar_MB1030>
   <!-- Mount an RGBD Camera -->
   <xacro:include filename="$(find fcu_sim_plugins)/xacro/rgbd.xacro"/>

Commit message: fixed sonar sensor

File: fcu_sim/agents/mikey/mikey.xacro (robot description, xacro)
@@ -72,5 +72,5 @@
     parent_link="${namespace}/base_link"
     sonar_topic="alt">
-    <origin xyz="0.4 0.1 -0.21" rpy="0 0 0" />
+    <origin xyz="0 0 0" rpy="0 1.57 0" />
   </xacro:Sonar_MB1030>
   <!-- Mount an RGBD Camera -->

File: fcu_sim_plugins/xacro/sonar.xacro (robot description, xacro)
@@ -15,7 +15,6 @@
     resolution="0.10"
     field_of_view="0.2618"
-    publish_rate="40">
+    update_rate="40">
     <inertia ixx="0.00001" ixy="0.0" ixz="0.0" iyy="0.00001" iyz="0.0" izz="0.00001" />
-    <origin xyz="0 0 0" rpy="0 0 0" />
     <xacro:insert_block name="origin"/>
   </xacro:sonar_plugin_macro>
@@ -38,5 +37,4 @@
     <inertia ixx="0.00001" ixy="0.0" ixz="0.0" iyy="0.00001" iyz="0.0" izz="0.00001" />
     <xacro:insert_block name="origin"/>
-    <!-- <origin xyz="0 0 0" rpy="0 0 0"/> -->
   </xacro:sonar_plugin_macro>
 </xacro:macro>
@@ -60,49 +58,52 @@
   <link name="${namespace}/sonar_link">
     <inertial>
-      <xacro:insert_block name="inertia" />
-      <mass value="${mass}" />
+      <mass value="${mass}"/>
       <xacro:insert_block name="origin"/>
+      <xacro:insert_block name="inertia"/>
     </inertial>
-  <sensor type="ray" name="sonar">
-     <update_rate>${update_rate}</update_rate>
-     <ray>
-       <scan>
-         <horizontal>
-           <samples>10</samples>
-           <resolution>${resolution}</resolution>
-           <min_angle>${-field_of_view / 2.0}</min_angle>
-           <max_angle>${field_of_view / 2.0}</max_angle>
-         </horizontal>
-         <vertical>
-           <samples>10</samples>
-           <resolution>${resolution}</resolution>
-           <min_angle>${-field_of_view / 2.0}</min_angle>
-           <max_angle>${field_of_view / 2.0}</max_angle>
-         </vertical>
-       </scan>
-       <range>
-         <min>${min_range}</min>
-         <max>${max_range}</max>
-         <resolution>${resolution}</resolution>
-       </range>
-     </ray>
-     <plugin filename="libgazebo_ros_range.so" name="gazebo_ros_range">
-       <gaussianNoise>${noise}</gaussianNoise>
-       <alwaysOn>true</alwaysOn>
-       <updateRate>${update_rate}</updateRate>
-       <topicName>{sonar_topic}</topicName>
-       <frameName>sonar_link</frameName>
-       <fov>${field_of_view}</fov>
-       <radiation>ultrasound</radiation>
-     </plugin>
-   </sensor>
- </link>
+  </link>
   <!-- sonar joint -->
-  <joint name="${namespace}/sonar_joint" type="revolute">
-    <xacro:insert_block name="origin" />
-    <parent link="${parent_link}" />
-    <child link="${namespace}/sonar_link" />
-    <limit upper="0" lower="0" effort="0" velocity="0" />
+  <joint name="${namespace}/sonar_joint" type="fixed">
+    <xacro:insert_block name="origin"/>
+    <parent link="${parent_link}"/>
+    <child link="${namespace}/sonar_link"/>
+    <limit upper="0" lower="0" effort="0" velocity="0"/>
   </joint>
+  <!-- attach a sonar -->
+  <gazebo reference="${namespace}/sonar_link">
+    <sensor type="ray" name="${namespace}/sonar">
+      <ray>
+        <scan>
+          <horizontal>
+            <samples>10</samples>
+            <resolution>${resolution}</resolution>
+            <min_angle>${-field_of_view / 2.0}</min_angle>
+            <max_angle>${field_of_view / 2.0}</max_angle>
+          </horizontal>
+          <vertical>
+            <samples>10</samples>
+            <resolution>${resolution}</resolution>
+            <min_angle>${-field_of_view / 2.0}</min_angle>
+            <max_angle>${field_of_view / 2.0}</max_angle>
+          </vertical>
+        </scan>
+        <range>
+          <min>${min_range}</min>
+          <max>${max_range}</max>
+          <resolution>${resolution}</resolution>
+        </range>
+      </ray>
+      <!-- load range plugin -->
+      <plugin filename="libgazebo_ros_range.so" name="${namespace}_sonar">
+        <robotNamespace>${namespace}</robotNamespace>
+        <gaussianNoise>${noise}</gaussianNoise>
+        <updateRate>${update_rate}</updateRate>
+        <topicName>${sonar_topic}</topicName>
+        <frameName>/sonar_link</frameName>
+        <fov>${field_of_view}</fov>
+        <radiation>ultrasound</radiation>
+      </plugin>
+    </sensor>
+  </gazebo>
 </xacro:macro>
 </robot>
