Commit message: Working for handoff sim

File: fcu_sim/agents/junker/junker.xacro (robot description, xacro)
@@ -2,5 +2,5 @@
 <robot name="junker" xmlns:xacro="http://ros.org/wiki/xacro">
   <!-- Properties -->
-  <xacro:property name="namespace" value="junker"/>
+  <xacro:property name="namespace" value="$(arg namespace)"/>
   <xacro:property name="wind_speed_topic" value="gazebo/wind_speed"/>
   <xacro:property name="command_topic" value="/command"/>
@@ -77,5 +77,5 @@
   <!-- Color -->
   <gazebo reference="${namespace}/base_link">
-    <material>Gazebo/Blue</material>
+    <material>Gazebo/$(arg color)</material>
   </gazebo>
   <!-- Sensors -->

Commit message: working on getting a new IMU working

File: fcu_sim/agents/junker/junker.xacro (robot description, xacro)
@@ -6,5 +6,5 @@
   <xacro:property name="command_topic" value="/command"/>
   <xacro:property name="use_mesh_file" value="true" />
-  <xacro:property name="mesh_file" value="package://fcu_sim/meshes/ju-87.dae"/>
+  <xacro:property name="mesh_file" value="model://zephyr_delta_wing/meshes/wing.dae"/>
   <xacro:property name="body_width" value="1.4"/>
   <xacro:property name="body_height" value="1.0" />
@@ -27,8 +27,8 @@
     </inertial>
     <visual name="plane_visual">
-      <origin xyz="0 0 0" rpy="1.570796 0 1.570796" />
+      <origin xyz="0 0 0" rpy="0 0 1.5707" />
       <geometry>
         <xacro:if value="${use_mesh_file}">
-          <mesh filename="${mesh_file}" scale="0.002 0.002 0.002" />
+          <mesh filename="${mesh_file}" scale="5 5 5"/>
         </xacro:if>
         <xacro:unless value="${use_mesh_file}">
@@ -38,5 +38,5 @@
     </visual>
     <collision name="plane_collision">
-      <origin xyz="0 0 0" rpy="1.570796 0 1.570796" />
+      <origin xyz="0 0 0" rpy="1.570796-1.570796 1.570796" />
       <geometry>
         <box size="${body_width} ${body_height} ${body_length}" />

File: fcu_sim_plugins/xacro/imu.xacro (robot description, xacro)
@@ -1,5 +1,5 @@
 <?xml version="1.0"?>
 <robot xmlns:xacro="http://ros.org/wiki/xacro">
-    <!-- Configure IMU -->
+      <!-- Perfect IMU -->
     <xacro:macro
       name="perfect_IMU"
@@ -8,88 +8,48 @@
       namespace="${namespace}"
       parent_link="${parent_link}"
+      update_rate="${update_rate}"
       imu_topic="${imu_topic}"
-      update_rate="${update_rate}"
-      gyroscope_noise_density="0.0"
-      gyroscopoe_random_walk="0.0"
-      gyroscope_bias_correlation_time="1000.0"
-      gyroscope_turn_on_bias_sigma="0.000"
-      accelerometer_noise_density="0.000"
-      accelerometer_random_walk="0.000"
-      accelerometer_bias_correlation_time="300.0"
-      accelerometer_turn_on_bias_sigma="0.0"
-      perfect_imu="true">
-      <inertia ixx="0.00001" ixy="0.0" ixz="0.0" iyy="0.00001" iyz="0.0" izz="0.00001" />
-      <origin xyz="0 0 0" rpy="0 0 0" />
-    </xacro:imu_plugin_macro>
+      gyro_stdev="0.0"
+      gyro_bias_range="0.00"
+      gyro_bias_walk_stdev="0.000"
+      acc_stdev="0.0"
+      acc_bias_range="0.0"
+      acc_bias_walk_stdev="0.000" />
   </xacro:macro>
+  <!-- MPU6050 (Naze) on a multirotor -->
     <xacro:macro
-      name="IMU_ADIS16448"
+      name="IMU_MPU6050_multirotor"
       params="namespace parent_link imu_topic update_rate">
     <xacro:imu_plugin_macro
       namespace="${namespace}"
       parent_link="${parent_link}"
+      update_rate="${update_rate}"
       imu_topic="${imu_topic}"
-      update_rate="${update_rate}"
-      gyroscope_noise_density="0.0003394"
-      gyroscopoe_random_walk="0.000038785"
-      gyroscope_bias_correlation_time="1000.0"
-      gyroscope_turn_on_bias_sigma="0.0.008"
-      accelerometer_noise_density="0.004"
-      accelerometer_random_walk="0.006"
-      accelerometer_bias_correlation_time="300.0"
-      accelerometer_turn_on_bias_sigma="0.1960"
-      perfect_imu="false">
-      <inertia ixx="0.00001" ixy="0.0" ixz="0.0" iyy="0.00001" iyz="0.0" izz="0.00001" />
-      <origin xyz="0 0 0" rpy="0 0 0" />
-    </xacro:imu_plugin_macro>
-  </xacro:macro>
-  <!-- Configure IMU -->
-    <xacro:macro
-      name="IMU_MPU6050"
-      params="namespace parent_link imu_topic update_rate">
-    <xacro:imu_plugin_macro
-      namespace="${namespace}"
-      parent_link="${parent_link}"
-      imu_topic="${imu_topic}"
-      update_rate="${update_rate}"
-      gyroscope_noise_density="0.0008726646"
-      gyroscopoe_random_walk="0.000038785"
-      gyroscope_bias_correlation_time="1000.0"
-      gyroscope_turn_on_bias_sigma="0.0087"
-      accelerometer_noise_density="0.008"
-      accelerometer_random_walk="0.006"
-      accelerometer_bias_correlation_time="300.0"
-      accelerometer_turn_on_bias_sigma="0.1960"
-      perfect_imu="false">
-      <inertia ixx="0.00001" ixy="0.0" ixz="0.0" iyy="0.00001" iyz="0.0" izz="0.00001" />
-      <origin xyz="0 0 0" rpy="0 0 0" />
-    </xacro:imu_plugin_macro>
+      gyro_stdev="0.13"
+      gyro_bias_range="0.08"
+      gyro_bias_walk_stdev="0.00001"
+      acc_stdev="1.15"
+      acc_bias_range="0.25"
+      acc_bias_walk_stdev="0.00001" />
   </xacro:macro>
     <!-- Macro to add an IMU. -->
   <xacro:macro name="imu_plugin_macro"
-    params="namespace parent_link imu_topic update_rate
-      gyroscope_noise_density gyroscopoe_random_walk
-      gyroscope_bias_correlation_time gyroscope_turn_on_bias_sigma
-      accelerometer_noise_density accelerometer_random_walk
-      accelerometer_bias_correlation_time accelerometer_turn_on_bias_sigma
-      perfect_imu
-      *inertia *origin">
+    params="namespace parent_link update_rate imu_topic
+            gyro_stdev gyro_bias_range gyro_bias_walk_stdev acc_stdev acc_bias_range
+            acc_bias_walk_stdev">
     <gazebo>
       <plugin filename="libimu_plugin.so" name="${namespace}_imu_plugin">
-      <!-- A good description of the IMU parameters can be found in the kalibr documentation:
-           https://github.com/ethz-asl/kalibr/wiki/IMU-Noise-Model-and-Intrinsics -->
-        <robotNamespace>${namespace}</robotNamespace> <!-- (string, required): ros namespace in which the messages are published -->
-        <linkName>${parent_link}</linkName> <!-- (string, required): name of the body which holds the IMU sensor -->
-        <imuTopic>${imu_topic}</imuTopic> <!-- (string): name of the sensor output topic and prefix of service names (defaults to imu) -->
-	<updateRate>${update_rate}</updateRate>
-	<gyroscopeNoiseDensity>${gyroscope_noise_density}</gyroscopeNoiseDensity> <!-- Gyroscope noise density (two-sided spectrum) [rad/s/sqrt(Hz)] -->
-        <gyroscopeRandomWalk>${gyroscopoe_random_walk}</gyroscopeRandomWalk> <!-- Gyroscope bias random walk [rad/s/s/sqrt(Hz)] -->
-        <gyroscopeBiasCorrelationTime>${gyroscope_bias_correlation_time}</gyroscopeBiasCorrelationTime> <!-- Gyroscope bias correlation time constant [s] -->
-        <gyroscopeTurnOnBiasSigma>${gyroscope_turn_on_bias_sigma}</gyroscopeTurnOnBiasSigma> <!-- Gyroscope turn on bias standard deviation [rad/s] -->
-        <accelerometerNoiseDensity>${accelerometer_noise_density}</accelerometerNoiseDensity> <!-- Accelerometer noise density (two-sided spectrum) [m/s^2/sqrt(Hz)] -->
-        <accelerometerRandomWalk>${accelerometer_random_walk}</accelerometerRandomWalk> <!-- Accelerometer bias random walk. [m/s^2/s/sqrt(Hz)] -->
-        <accelerometerBiasCorrelationTime>${accelerometer_bias_correlation_time}</accelerometerBiasCorrelationTime> <!-- Accelerometer bias correlation time constant [s] -->
-        <accelerometerTurnOnBiasSigma>${accelerometer_turn_on_bias_sigma}</accelerometerTurnOnBiasSigma> <!-- Accelerometer turn on bias standard deviation [m/s^2] -->
-        <perfectIMU>${perfect_imu}</perfectIMU>
+        <namespace>${namespace}</namespace>
+        <link_name>${parent_link}</link_name>
+        <update_rate>${update_rate}</update_rate>
+        <imu_topic>${imu_topic}/data</imu_topic>
+        <acc_bias_topic>${imu_topic}/acc_bias</acc_bias_topic>
+        <gyro_bias_topic>${imu_topic}/gyro_bias</gyro_bias_topic>
+        <gyro_stdev>${gyro_stdev}</gyro_stdev>
+        <gyro_bias_range>${gyro_bias_range}</gyro_bias_range>
+        <gyro_bias_walk_stdev>${gyro_bias_walk_stdev}</gyro_bias_walk_stdev>
+        <acc_stdev>${acc_stdev}</acc_stdev>
+        <acc_bias_range>${acc_bias_range}</acc_bias_range>
+        <acc_bias_walk_stdev>${acc_bias_walk_stdev}</acc_bias_walk_stdev>
       </plugin>
     </gazebo>

File: fcu_sim_plugins/xacro/odometry_sensor.xacro (robot description, xacro)
@@ -7,62 +7,21 @@
       <xacro:odometry_plugin_macro
         namespace="${namespace}/ground_truth"
-        parent_link="${namespace}/base_link"
-        pose_topic="pose"
-        pose_with_covariance_topic="pose_with_covariance"
-        position_topic="position"
+        parent_link="${parent_link}"
         transform_topic="transform"
         odometry_topic="odometry"
-        parent_frame_id="world"
-        measurement_divisor="1"
-        measurement_delay="0"
-        unknown_delay="0.0"
-        noise_normal_position="0 0 0"
-        noise_normal_quaternion="0 0 0"
-        noise_normal_linear_velocity="0 0 0"
-        noise_normal_angular_velocity="0 0 0"
-        noise_uniform_position="0 0 0"
-        noise_uniform_quaternion="0 0 0"
-        noise_uniform_linear_velocity="0 0 0"
-        noise_uniform_angular_velocity="0 0 0"
-        enable_odometry_map="false"
-        odometry_map=""
-        image_scale=""/>
+        parent_frame_id="world"/>
     </xacro:macro>
   <!-- Macro to add a generic odometry sensor. -->
   <xacro:macro name="odometry_plugin_macro"
     params="
-      namespace parent_link pose_topic pose_with_covariance_topic
-      position_topic transform_topic odometry_topic parent_frame_id
-      measurement_divisor measurement_delay unknown_delay
-      noise_normal_position noise_normal_quaternion noise_normal_linear_velocity
-      noise_normal_angular_velocity noise_uniform_position
-      noise_uniform_quaternion noise_uniform_linear_velocity
-      noise_uniform_angular_velocity enable_odometry_map odometry_map
-      image_scale">
+      namespace parent_link transform_topic
+      odometry_topic parent_frame_id">
     <gazebo>
       <plugin filename="libodometry_plugin.so" name="${namespace}_odometry_sensor">
-        <linkName>${parent_link}</linkName>
-        <robotNamespace>${namespace}</robotNamespace>
-        <poseTopic>${pose_topic}</poseTopic>
-        <poseWithCovarianceTopic>${pose_with_covariance_topic}</poseWithCovarianceTopic>
-        <positionTopic>${position_topic}</positionTopic>
-        <transformTopic>${transform_topic}</transformTopic>
-        <odometryTopic>${odometry_topic}</odometryTopic>
-        <parentFrameId>${parent_frame_id}</parentFrameId> <!-- Use the scoped link name here. e.g. Model::link. -->
-        <measurementDivisor>${measurement_divisor}</measurementDivisor> <!-- only every (seq % measurementDivisor) == 0 measurement is published [int] -->
-        <measurementDelay>${measurement_delay}</measurementDelay> <!-- time that measurement gets held back before it's published in [simulation cycles (int)] -->
-        <unknownDelay>${unknown_delay}</unknownDelay> <!-- additional delay, that just gets added to the timestamp [s] -->
-        <noiseNormalPosition>${noise_normal_position}</noiseNormalPosition> <!-- standard deviation of additive white gaussian noise [m] -->
-        <noiseNormalQuaternion>${noise_normal_quaternion}</noiseNormalQuaternion> <!-- standard deviation white gaussian noise [rad]: q_m = q*quaternionFromSmallAngleApproximation(noiseNormalQ) -->
-        <noiseNormalLinearVelocity>${noise_normal_linear_velocity}</noiseNormalLinearVelocity> <!-- standard deviation of additive white gaussian noise [m/s] -->
-        <noiseNormalAngularVelocity>${noise_normal_angular_velocity}</noiseNormalAngularVelocity> <!-- standard deviation of additive white gaussian noise [rad/s] -->
-        <noiseUniformPosition>${noise_uniform_position}</noiseUniformPosition> <!-- symmetric bounds of uniform noise [m] -->
-        <noiseUniformQuaternion>${noise_uniform_quaternion}</noiseUniformQuaternion> <!-- symmetric bounds of uniform noise [rad], computation see above -->
-        <noiseUniformLinearVelocity>${noise_uniform_linear_velocity}</noiseUniformLinearVelocity> <!-- symmetric bounds of uniform noise [m/s] -->
-        <noiseUniformAngularVelocity>${noise_uniform_angular_velocity}</noiseUniformAngularVelocity> <!-- symmetric bounds of uniform noise [rad/s] -->
-        <xacro:if value="${enable_odometry_map}">
-          <covarianceImage>package://fcu_sim/resource/${odometry_map}</covarianceImage> <!-- a bitmap image describing where the sensor works (white), and where not (black) -->
-          <covarianceImageScale>${image_scale}</covarianceImageScale> <!-- the scale of the image in the gazebo world, if set to 1.0, 1 pixel in the image corresponds to 1 meter in the world -->
-        </xacro:if>
+        <parent_link>${parent_link}</parent_link>
+        <namespace>${namespace}</namespace>
+        <frame_id>${parent_frame_id}</frame_id>
+        <odometry_topic>${odometry_topic}</odometry_topic>
+        <transform_topic>${transform_topic}</transform_topic>
       </plugin>
     </gazebo>
